File: eagle/Gearnode/H-bro_gear.sch (EAGLE design)
At the start: 17 parts, among them IC1 LM4558N, IC2 74AC08D, IC3 4070D, Q1 IRF512, Q2 IRF512, Q3 IRF512, Q4 IRF512

Commit message: finalized v1 of board
Parts:
- removed F1: (no value), fuse:PICOFUSE
- removed IC1: LM4558N, linear:LM4558N
- removed Q1, Q2, Q3, Q4: IRF512, transistor-power:IRF512
- added C5, C6: (no value), rcl:CPOL-EUE15-5AXIAL
- added IC4: 7805T, linear:7805T
- added IC6: TL074P, linear:TL074P
- added LED1, LED2: (no value), adafruit:LED5MM
- added R2, R3, R4, R6, R7: (no value), rcl:R-EU_0204/7
- added R5: (no value), pot:TRIM_EU-RJ9W
- added U$3, U$4, U$5, U$6: STU95N5, Brushless-motor-controller:STU95N5
- added U$7: LITTE_FUSE, unicorn_v2:LITTE_FUSE
- added X1, X2: (no value), con-wago-500:W237-102
- added X3: 22-23-2031, con-molex:22-23-2031
- added X4: 22-23-2041, con-molex:22-23-2041
- C1, C2, C3, C4: device resistor:C-EU025-025X050 -> rcl:C-EU050-025X075
Connections:
- removed net IN0: IC2A.I0, IC3B.I0
- removed net IN1: IC2B.I1, IC3B.I1
- new net ADC0: IC6A.+IN, IC6D.OUT, R2.2, X4-2.S
- new net INA: IC2D.I0, X4-4.S
- new net INB: IC2C.I1, X4-3.S
- new net N$16: IC2A.I0, IC2D.O, IC3D.I0
- new net N$17: IC2B.I1, IC2C.O, IC3D.I1
- new net N$18: IC6A.-IN, R4.1, R5.E, R5.S
- new net N$19: LED1.A, R6.2
- new net N$20: IC6B.+IN, X3-2.S
- new net N$21: IC6D.-IN, R2.1, R3.2
- new net N$22: LED2.A, R7.1
- new net OPC: IC2C.I0, IC2D.I1, IC6A.OUT, R7.2
- new net POSPOT: IC6B.-IN, IC6B.OUT, X4-1.S
- net +12V: now also C6.+, IC4.VI, U$7.PIN1, X2-1.KL; no longer F1.2
- net +5V: now also C5.+, IC4.VO, IC6P.V+, R4.2, X3-3.S; no longer IC1P.V+
- net GND: now also C5.-, C6.-, IC4.GND, IC6P.V-, LED1.C, LED2.C, R3.1, R5.A, X2-2.KL, X3-1.S; no longer IC1P.V-
- net N$1: now also U$3.G; no longer Q1.G
- net N$11: now also IC6D.+IN, U$4.S, U$5.S; no longer Q3.S, Q4.S
- net N$15: now also IC3D.O; no longer IC3B.O
- net N$2: now also U$4.G; no longer Q3.G
- net N$3: now also U$6.G; no longer Q2.G
- net N$4: now also U$5.G; no longer Q4.G
- net N$6: now also U$3.S, U$4.D, U$4.TAB, X1-2.KL; no longer Q1.S, Q3.D
- net N$7: now also U$5.D, U$5.TAB, U$6.S, X1-1.KL; no longer Q2.S, Q4.D
- net N$9: now also R6.1, U$3.D, U$3.TAB, U$6.D, U$6.TAB, U$7.PIN2; no longer F1.1, Q1.D, Q2.D
Other:
- moved on the sheet: R1
