File: STM32F407 era/Processor board/processor board.sch (EAGLE design)
At the start: 0 parts

Commit message: Added peripfial ports to processor port
added connections for CAN. USB. JTAG; I2C, SPI.
Added crystal, and decoupling circuitry
Parts:
- added C1, C2: 2u2, microbuilder:CAP_CERAMIC_0402MP
- added C10, C12, C3, C5, C6, C7, C8, C9: 100n, microbuilder:CAP_CERAMIC_0402MP
- added C11: (no value), microbuilder:CAP_CERAMIC_0402MP
- added C13, C4: 1u, microbuilder:CAP_CERAMIC_0402MP
- added C14, C15: 22p, microbuilder:CAP_CERAMIC_0402MP
- added C16: 4u7, microbuilder:CAP_CERAMIC_0603MP
- added JTAG1: JTAG-ARM, microbuilder:JTAG-ARM
- added Q1: 8 MHz, special:XTAL/S
- added R1, R2: 500, microbuilder:RESISTOR_0402MP
- added R3, R4, R5: 1k8, microbuilder:RESISTOR_0402MP
- added S1: RESET, SparkFun-Electromechanical:SWITCH-MOMENTARY-2SMD-1101NE
- added S2: BOOT, SparkFun-Electromechanical:SWITCH-MOMENTARY-2SMD-1101NE
- added U1: (no value), apbteam_stm32:STM32F4-100
- added X1: MINI-USB-SCHIELD-32005-201, con-cypressindustries:MINI-USB-SCHIELD-32005-201
Connections:
- new net 3.3V: C10.P$1, C11.P$1, C12.P$1, C13.P$1, C3.P$1, C4.P$1, C5.P$1, C6.P$1, C7.P$1, C8.P$1, C9.P$1, JTAG1.1, JTAG1.2, R2.1, R3.1, R4.1, S2.2, U1G$1.VDD, U1G$1.VDD@1, U1G$1.VDD@2, U1G$1.VDD@3, U1G$1.VDD@4, U1G$1.VDD@5, U1G$1.VDDA, U1G$1.VREF+
- new net CAN_RX: U1G$3.PB8
- new net CAN_TX: U1G$3.PB9
- new net GND: C1.P$2, C10.P$2, C11.P$2, C12.P$2, C13.P$2, C14.P$1, C15.P$2, C16.P$2, C2.P$2, C3.P$2, C4.P$2, C5.P$2, C6.P$2, C7.P$2, C8.P$2, C9.P$2, JTAG1.10, JTAG1.12, JTAG1.14, JTAG1.16, JTAG1.18, JTAG1.20, JTAG1.3, JTAG1.4, JTAG1.6, JTAG1.8, R1.2, R5.2, S1.2, U1G$1.VSS, U1G$1.VSS@1, U1G$1.VSS@2, U1G$1.VSS@3, U1G$1.VSSA, U1G$3.PB2/BOOT1, X1G$1.5, X1S.S1, X1S.S2, X1S.S3, X1S.S4
- new net JTAG_TCK: JTAG1.9, U1G$2.PA14
- new net JTAG_TDI: JTAG1.5, U1G$2.PA15
- new net JTAG_TDO: JTAG1.13, U1G$3.PB3
- new net JTAG_TMS: JTAG1.7, U1G$2.PA13
- new net N$1: C15.P$1, Q1.2, U1G$7.PH0
- new net N$11: C14.P$2, Q1.1, U1G$7.PH1
- new net N$2: C1.P$1, U1G$1.VCAP2
- new net N$3: C2.P$1, U1G$1.VCAP1
- new net N$4: R1.1, S2.1, U1G$7.BOOT0
- new net N$5: R2.2, S1.1, U1G$7.NRST
- new net RESET: JTAG1.15
- new net SCL: R3.2, U1G$3.PB6
- new net SDA: R4.2, U1G$3.PB7
- new net SPI_MISO: U1G$3.PB14
- new net SPI_MOSI: U1G$3.PB15
- new net SPI_SCK: R5.1, U1G$3.PB13
- new net USB_DM: U1G$2.PA11, X1G$1.2
- new net USB_DP: U1G$2.PA12, X1G$1.3
- new net USB_ID: U1G$2.PA10, X1G$1.4
- new net USB_VBUS: C16.P$1, U1G$2.PA9, X1G$1.1
