File: STM32F407 era/Processor board/processor board.sch (EAGLE design)
At the start: 42 parts, among them IC1 REG1117, U2 MAX13052ESA+, X1 MINI-USB-SCHIELD-32005-201, X2 057-010-1, Y1 25 MHz, Y2 32.768KHz

Commit message: small updates for etching
Parts:
- added PTC1: (no value), microbuilder:PTC1206
Changed lines of the file:
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@@
 <part name="U$11" library="microbuilder" deviceset="GND" device=""/>
 <part name="U$12" library="microbuilder" deviceset="GND" device=""/>
+<part name="PTC1" library="microbuilder" deviceset="PTC" device="1206"/>
 </parts>
 <sheets>
@@
 <instance part="U$11" gate="G$1" x="215.9" y="25.4" rot="MR0"/>
 <instance part="U$12" gate="G$1" x="203.2" y="25.4" rot="MR0"/>
+<instance part="PTC1" gate="G$1" x="144.78" y="121.92"/>
 </instances>
 <busses>
