File: STM32F407 era/Development board/development board.brd (EAGLE design)
At the start: 160 x 100 mm, 75 parts, among them IC1 74HC595N, IC2 74HC595N, IC3 317T, IC4 317T, U1 MAX13052ESA+, X1 K375M, X2 HD44780LCD-1602, X3 SDBMF, X4 057-006-1, X8 057-006-1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

Commit message: updates to the layout and done routing (maybe)
Parts:
- added JP3: (no value), pinhead:2X11
- added LED10, LED9: (no value), led:LED3MM
- added R29: 150, microbuilder:_0603
- added R30: 100, microbuilder:_0603
- added SV5: (no value), con-lstb:MA03-2
- moved ISP1 0.64 mm to (59.1, 89.5)
- moved R11 0.64 mm to (50.8, 20.3)
- moved R12 0.64 mm to (57.8, 20.3)
- moved R13 0.64 mm to (64.8, 20.3)
- moved R14 0.64 mm to (71.8, 20.3)
- moved R15 0.64 mm to (78.7, 20.3)
- moved R16 0.64 mm to (85.7, 20.3)
- moved R17 0.64 mm to (92.7, 20.3)
- moved R18 0.64 mm to (99.7, 20.3)
- moved S1 0.64 mm to (50.8, 20.3)
- moved S2 0.64 mm to (57.8, 20.3)
- moved S3 0.64 mm to (64.8, 20.3)
- moved S4 0.64 mm to (71.8, 20.3)
- moved S5 0.64 mm to (78.7, 20.3)
- moved S6 0.64 mm to (85.7, 20.3)
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Connections:
- new net N$20: LED10.A, R30.1
- new net N$31: LED9.A, R29.1
- new net PA0: JP3.4, U$1.P$75
- new net PA1: JP3.3, U$1.P$76
- new net PA2: JP3.2, U$1.P$77
- new net PA9: JP3.1, U$1.P$40
- new net PB4: JP3.18, U$1.P$54
- new net PB9: JP3.17, U$1.P$59
- new net PC0: JP3.8, U$1.P$71
- new net PC1: JP3.7, U$1.P$72
- new net PC13: JP3.9, U$1.P$68
- new net PC2: JP3.6, U$1.P$73
- new net PC3: JP3.5, U$1.P$74
- new net PD4: JP3.20, U$1.P$50
- new net PD7: JP3.19, U$1.P$53
- new net PE0: JP3.16, U$1.P$60
- new net PE1: JP3.15, U$1.P$61
- new net PE2: JP3.14, U$1.P$63
- new net PE3: JP3.13, U$1.P$64
- new net PE4: JP3.12, U$1.P$65
- new net PE5: JP3.11, U$1.P$66
- new net PE6: JP3.10, U$1.P$67
- net 3.3V: now also R30.2, SV5.2
- net 5.0V: now also R29.2
- net GND: now also JP3.21, JP3.22, LED10.K, LED9.K, SV5.6
- net SPI_MISO: now also SV5.1
- net SPI_MOSI: now also SV5.4
- net SPI_SCK: now also SV5.3
Routing:
- net PA9: track 0.00 -> 115.8 mm, vias 0 -> 2
- net PD4: track 0.00 -> 74.0 mm, vias 0 -> 2
- net SDIO_D0: track 27.3 -> 99.7 mm, vias 0 -> 1
- net PB4: track 0.00 -> 71.1 mm, vias 0 -> 2
- net SDIO_D1: track 23.1 -> 89.6 mm, vias 0 -> 1
- net PE0: track 0.00 -> 65.6 mm
- net PD7: track 0.00 -> 64.9 mm, vias 0 -> 2
- net PA2: track 0.00 -> 63.3 mm
- net PC13: track 0.00 -> 63.2 mm
- net PA1: track 0.00 -> 62.9 mm
- net PE6: track 0.00 -> 62.8 mm
- net PA0: track 0.00 -> 62.5 mm
- net PE5: track 0.00 -> 62.5 mm
- net PC3: track 0.00 -> 62.1 mm
- net PE4: track 0.00 -> 62.1 mm
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Other:
- board text added: "3,3V"
- board text added: "CAN2"
- board text added: "Charecter LCD"
- board text added: "I2C1 <G|C|D>"
- board text added: "PA2 PA0 PC2 PC0 PE6 PE4 PE2 PE0 PB4 PD4"
- board text added: "PA9 PA1 PC3 PC1 PC13 PE5 PE3 PE1 PB9 PD7"
- board text added: "SPI1"
- board text added: "USART2 <G|R|T>"
- board text added: "USART3 <G|R|T>"
- board text removed: "Charecter LCD port"

Commit message: updates to layout
Parts:
- moved R11 0.64 mm to (50.8, 19.7)
- moved R12 0.64 mm to (57.8, 19.7)
- moved R13 0.64 mm to (64.8, 19.7)
- moved R14 0.64 mm to (71.8, 19.7)
- moved R15 0.64 mm to (78.7, 19.7)
- moved R16 0.64 mm to (85.7, 19.7)
- moved R17 0.64 mm to (92.7, 19.7)
- moved R18 0.64 mm to (99.7, 19.7)
- moved SV1 0.63 mm to (75.6, 53.3)
Routing:
- net N$33: track 0.00 -> 64.1 mm
- net N$35: track 0.00 -> 16.2 mm
- net 3.3V: track 392.2 -> 393.1 mm
- net LED7: track 106.9 -> 106.3 mm
- net N$29: track 4.33 -> 3.70 mm
- net N$28: track 4.33 -> 3.70 mm
- net N$27: track 4.33 -> 3.70 mm
- net N$26: track 4.33 -> 3.70 mm
- net N$25: track 4.33 -> 3.70 mm
- net N$23: track 4.33 -> 3.70 mm
- net N$21: track 4.33 -> 3.70 mm
- net N$19: track 4.33 -> 3.70 mm
- net LED6: track 55.8 -> 55.2 mm
- net LED5: track 54.2 -> 53.5 mm
- net LED4: track 43.3 -> 42.7 mm
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Other:
- board text added: "GND"
- board text added: "MISO"
- board text added: "MOSI"
- board text added: "PA3"
- board text added: "PA8"
- board text added: "PB0"
- board text added: "PB1"
- board text added: "PB12"
- board text added: "PC4"
- board text added: "PC5"
- board text added: "PE10"
- board text added: "PE11"
- board text added: "PE12"
- board text added: "PE13"
- board text added: "PE14"
- board text added: "PE15"
- board text added: "PE7"
- board text added: "PE8"
- board text added: "PE9"
- board text added: "RST"
- board text added: "SCK"
- board text added: "VCC"

Commit message: updates to layout
Routing:
- net N$47: track 0.00 -> 156.8 mm
- net N$39: track 0.00 -> 120.0 mm
- net N$33: track 64.1 -> 124.5 mm
- net N$37: track 0.00 -> 52.7 mm
- net N$46: track 0.00 -> 41.6 mm
- net N$41: track 0.00 -> 14.9 mm
- net N$43: track 0.00 -> 12.7 mm
Other:
- board text added: "IC1"
- board text added: "N.C."
- board text added: "PA5"
- board text added: "PA6"
- board text added: "PA7"
- board text added: "PB10"
- board text added: "PB11"
- board text added: "PB5"
- board text added: "PB6"
- board text added: "PB7"
- board text added: "PB8"
- board text added: "PD5"
- board text added: "PD6"
- board text added: "RX"
- board text added: "SCL"
- board text added: "SDA"
- board text added: "TX"
- board text added: "USART"
- board text added: "USART2"
- board text added: "USART3"
