File: STM32F407 era/CAN 5-way/can-5-way.brd (EAGLE design)
At the start: 160 x 100 mm, 5 parts

Commit message: updates to the layout and done routing (maybe)
Changed lines of the file:
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@@
 <wire x1="51.975" y1="35.56" x2="52.07" y2="35.655" width="0.4064" layer="1"/>
 <wire x1="52.07" y1="35.655" x2="52.07" y2="39.91" width="0.4064" layer="1"/>
-<wire x1="50.26" y1="45.72" x2="50.26" y2="45.18" width="0.4064" layer="1"/>
-<wire x1="50.26" y1="45.18" x2="47.625" y2="42.545" width="0.4064" layer="1"/>
-<wire x1="47.625" y1="42.545" x2="45.815" y2="42.545" width="0.4064" layer="1"/>
+<wire x1="48.895" y1="42.545" x2="45.815" y2="42.545" width="0.4064" layer="1"/>
 <wire x1="45.815" y1="42.545" x2="45.72" y2="42.64" width="0.4064" layer="1"/>
-<wire x1="52.07" y1="39.91" x2="50.26" y2="39.91" width="0.4064" layer="1"/>
-<wire x1="50.26" y1="39.91" x2="47.625" y2="42.545" width="0.4064" layer="1"/>
 <wire x1="42.7675" y1="35.56" x2="42.7675" y2="36.1" width="0.4064" layer="1"/>
 <wire x1="42.7675" y1="36.1" x2="44.1325" y2="37.465" width="0.4064" layer="1"/>
-<wire x1="44.1325" y1="37.465" x2="47.815" y2="37.465" width="0.4064" layer="1"/>
-<wire x1="47.815" y1="37.465" x2="50.26" y2="39.91" width="0.4064" layer="1"/>
+<wire x1="50.26" y1="45.72" x2="50.26" y2="44.545" width="0.4064" layer="1"/>
+<wire x1="50.26" y1="44.545" x2="48.895" y2="43.18" width="0.4064" layer="1"/>
+<wire x1="48.895" y1="43.18" x2="48.895" y2="42.545" width="0.4064" layer="1"/>
+<wire x1="44.1325" y1="37.465" x2="47.3075" y2="37.465" width="0.4064" layer="1"/>
+<wire x1="47.3075" y1="37.465" x2="48.895" y2="39.0525" width="0.4064" layer="1"/>
+<wire x1="48.895" y1="39.0525" x2="48.895" y2="40.005" width="0.4064" layer="1"/>
+<wire x1="48.895" y1="40.005" x2="48.895" y2="42.545" width="0.4064" layer="1"/>
+<wire x1="52.07" y1="39.91" x2="48.99" y2="39.91" width="0.4064" layer="1"/>
+<wire x1="48.99" y1="39.91" x2="48.895" y2="40.005" width="0.4064" layer="1"/>
 </signal>
 <signal name="N$2">
@@
 <contactref element="U$3" pad="PIN2"/>
 <contactref element="U$2" pad="PIN2"/>
-<wire x1="52.07" y1="42.91" x2="50.53" y2="42.91" width="0.4064" layer="16"/>
-<wire x1="50.53" y1="42.91" x2="50.165" y2="42.545" width="0.4064" layer="16"/>
-<wire x1="50.165" y1="42.545" x2="47.26" y2="39.64" width="0.4064" layer="16"/>
-<wire x1="47.26" y1="39.64" x2="45.72" y2="39.64" width="0.4064" layer="16"/>
+<wire x1="47.5775" y1="39.64" x2="45.72" y2="39.64" width="0.4064" layer="16"/>
 <wire x1="45.72" y1="39.64" x2="45.7675" y2="39.5925" width="0.4064" layer="16"/>
 <wire x1="45.7675" y1="39.5925" x2="45.7675" y2="37.465" width="0.4064" layer="16"/>
@@
 <wire x1="54.975" y1="36.7825" x2="54.2925" y2="37.465" width="0.4064" layer="16"/>
 <wire x1="54.2925" y1="37.465" x2="45.7675" y2="37.465" width="0.4064" layer="16"/>
-<wire x1="47.26" y1="45.72" x2="47.26" y2="45.45" width="0.4064" layer="16"/>
-<wire x1="47.26" y1="45.45" x2="50.165" y2="42.545" width="0.4064" layer="16"/>
+<wire x1="47.5775" y1="39.64" x2="48.895" y2="40.9575" width="0.4064" layer="16"/>
+<wire x1="48.895" y1="40.9575" x2="48.895" y2="42.8625" width="0.4064" layer="16"/>
+<wire x1="48.895" y1="42.8625" x2="48.895" y2="44.085" width="0.4064" layer="16"/>
+<wire x1="48.895" y1="44.085" x2="47.26" y2="45.72" width="0.4064" layer="16"/>
+<wire x1="52.07" y1="42.91" x2="48.9425" y2="42.91" width="0.4064" layer="16"/>
+<wire x1="48.9425" y1="42.91" x2="48.895" y2="42.8625" width="0.4064" layer="16"/>
 </signal>
 <signal name="GND">
@@
 <polygon width="0.4064" layer="1">
 <vertex x="33.9725" y="23.8125"/>
-<vertex x="64.135" y="23.8125"/>
-<vertex x="64.135" y="45.4025"/>
-<vertex x="51.1175" y="58.42"/>
-<vertex x="46.0375" y="58.42"/>
+<vertex x="63.8175" y="23.8125"/>
+<vertex x="63.8175" y="45.4025"/>
+<vertex x="51.7525" y="57.4675"/>
+<vertex x="46.0375" y="57.4675"/>
 <vertex x="33.9725" y="45.4025"/>
 </polygon>

Commit message: small updates for etching
Parts:
- added H1, H2, H3, H4: MOUNT-HOLE3.0, holes:3,0
- added U$7: MICROFIT4, unicorn:MICROFIT4SOCK
- moved U$2 51.8 mm to (14.6, 1.91)
- moved U$4 50.8 mm to (4.45, 24.1), turned to 270 degrees
- moved U$1 45.7 mm to (4.45, 14.0), turned to 270 degrees
- moved U$3 34.3 mm to (24.1, 14.0), turned to 90 degrees
- moved U$5 32.4 mm to (24.1, 24.1), turned to 90 degrees
Connections:
- net GND: now also U$7.PIN3, U$7.PIN4
- net N$1: now also U$7.PIN1
- net N$2: now also U$7.PIN2
Routing:
- net N$1: track 25.9 -> 29.5 mm
- net N$2: track 27.2 -> 30.1 mm
Other:
- outline, holes or cut-outs redrawn
- board text added: "bund"
