File: STM32F407 era/CAN 5-way/can-5-way.sch (EAGLE design)
At the start: 5 parts

Commit message: small updates for etching
Parts:
- added H1, H2, H3, H4: MOUNT-HOLE3.0, holes:MOUNT-HOLE3.0
- added U$7: MICROFIT4, unicorn:MICROFIT4
Connections:
- net GND: now also U$7.PIN3, U$7.PIN4
- net N$1: now also U$7.PIN1
- net N$2: now also U$7.PIN2
Changed lines of the file:
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@@
 <part name="U$5" library="unicorn" deviceset="MICROFIT4" device=""/>
 <part name="U$6" library="microbuilder" deviceset="GND" device=""/>
+<part name="U$7" library="unicorn" deviceset="MICROFIT4" device=""/>
+<part name="H1" library="holes" deviceset="MOUNT-HOLE" device="3.0"/>
+<part name="H2" library="holes" deviceset="MOUNT-HOLE" device="3.0"/>
+<part name="H3" library="holes" deviceset="MOUNT-HOLE" device="3.0"/>
+<part name="H4" library="holes" deviceset="MOUNT-HOLE" device="3.0"/>
 </parts>
 <sheets>
@@
 <instance part="U$4" gate="G$1" x="48.26" y="38.1"/>
 <instance part="U$5" gate="G$1" x="48.26" y="22.86"/>
-<instance part="U$6" gate="G$1" x="33.02" y="15.24"/>
+<instance part="U$6" gate="G$1" x="33.02" y="0"/>
+<instance part="U$7" gate="G$1" x="48.26" y="7.62"/>
+<instance part="H1" gate="G$1" x="12.7" y="48.26"/>
+<instance part="H2" gate="G$1" x="12.7" y="40.64"/>
+<instance part="H3" gate="G$1" x="12.7" y="33.02"/>
+<instance part="H4" gate="G$1" x="12.7" y="25.4"/>
 </instances>
 <busses>
@@
 <wire x1="40.64" y1="73.66" x2="38.1" y2="73.66" width="0.1524" layer="91"/>
 <junction x="38.1" y="73.66"/>
+<pinref part="U$7" gate="G$1" pin="PIN1"/>
+<wire x1="40.64" y1="12.7" x2="38.1" y2="12.7" width="0.1524" layer="91"/>
+<wire x1="38.1" y1="12.7" x2="38.1" y2="27.94" width="0.1524" layer="91"/>
+<junction x="38.1" y="27.94"/>
 </segment>
 </net>
@@
 <wire x1="40.64" y1="71.12" x2="35.56" y2="71.12" width="0.1524" layer="91"/>
 <junction x="35.56" y="71.12"/>
+<pinref part="U$7" gate="G$1" pin="PIN2"/>
+<wire x1="40.64" y1="10.16" x2="35.56" y2="10.16" width="0.1524" layer="91"/>
+<wire x1="35.56" y1="10.16" x2="35.56" y2="25.4" width="0.1524" layer="91"/>
+<junction x="35.56" y="25.4"/>
 </segment>
 </net>
@@
 <wire x1="33.02" y1="35.56" x2="33.02" y2="22.86" width="0.1524" layer="91"/>
 <wire x1="33.02" y1="22.86" x2="33.02" y2="20.32" width="0.1524" layer="91"/>
-<wire x1="33.02" y1="20.32" x2="33.02" y2="17.78" width="0.1524" layer="91"/>
+<wire x1="33.02" y1="20.32" x2="33.02" y2="7.62" width="0.1524" layer="91"/>
+<wire x1="33.02" y1="7.62" x2="33.02" y2="5.08" width="0.1524" layer="91"/>
+<wire x1="33.02" y1="5.08" x2="33.02" y2="2.54" width="0.1524" layer="91"/>
 <wire x1="40.64" y1="81.28" x2="33.02" y2="81.28" width="0.1524" layer="91"/>
 <junction x="33.02" y="81.28"/>
@@
 <wire x1="40.64" y1="20.32" x2="33.02" y2="20.32" width="0.1524" layer="91"/>
 <junction x="33.02" y="20.32"/>
+<pinref part="U$7" gate="G$1" pin="PIN3"/>
+<wire x1="40.64" y1="7.62" x2="33.02" y2="7.62" width="0.1524" layer="91"/>
+<junction x="33.02" y="7.62"/>
+<pinref part="U$7" gate="G$1" pin="PIN4"/>
+<wire x1="40.64" y1="5.08" x2="33.02" y2="5.08" width="0.1524" layer="91"/>
+<junction x="33.02" y="5.08"/>
 </segment>
 </net>
