File: STM32F407 era/Telemetry external unit/Battery holder/battery holder.brd (EAGLE design)
At the start: 115.8 x 68.7 mm, 11 parts

Commit message: layout updates
Routing:
- net 12V: track 95.0 -> 99.7 mm, vias 0 -> 1
Other:
- board size 115.8 x 68.7 mm -> 108.2 x 68.7 mm
Changed lines of the file:
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@@
 <board>
 <plain>
-<wire x1="-25.4" y1="-9.7" x2="-22.4" y2="-12.7" width="0" layer="20" curve="90"/>
-<wire x1="-22.4" y1="-12.7" x2="87.4" y2="-12.7" width="0" layer="20"/>
+<wire x1="-17.78" y1="-9.7" x2="-14.78" y2="-12.7" width="0" layer="20" curve="90"/>
+<wire x1="-14.78" y1="-12.7" x2="87.4" y2="-12.7" width="0" layer="20"/>
 <wire x1="87.4" y1="-12.7" x2="90.4" y2="-9.7" width="0" layer="20" curve="90"/>
 <wire x1="90.4" y1="-9.7" x2="90.4" y2="53" width="0" layer="20"/>
 <wire x1="90.4" y1="53" x2="87.4" y2="56" width="0" layer="20" curve="90"/>
-<wire x1="87.4" y1="56" x2="-22.4" y2="56" width="0" layer="20"/>
-<wire x1="-22.4" y1="56" x2="-25.4" y2="53" width="0" layer="20" curve="90"/>
+<wire x1="87.4" y1="56" x2="-14.78" y2="56" width="0" layer="20"/>
+<wire x1="-14.78" y1="56" x2="-17.78" y2="53" width="0" layer="20" curve="90"/>
 <hole x="3.5" y="3.5" drill="2.8"/>
 <hole x="3.5" y="52.5" drill="2.8"/>
@@
 <circle x="3.485" y="21.5975" radius="1.55" width="3.1" layer="42"/>
 <circle x="3.485" y="21.5975" radius="1.55" width="3.1" layer="41"/>
-<wire x1="-25.4" y1="53" x2="-25.4" y2="-9.7" width="0" layer="20"/>
-<hole x="-21.28" y="21.5975" drill="2.8"/>
-<circle x="-21.28" y="21.5975" radius="1.55" width="3.1" layer="41"/>
-<circle x="-21.28" y="21.5975" radius="1.55" width="3.1" layer="42"/>
-<circle x="-21.28" y="21.5975" radius="1.55" width="3.1" layer="41"/>
+<wire x1="-17.78" y1="53" x2="-17.78" y2="-9.7" width="0" layer="20"/>
 </plain>
 <attributes>
@@
 <signal name="GND">
 <polygon width="0.254" layer="16">
-<vertex x="-25.4" y="-9.7" curve="90"/>
-<vertex x="-22.4" y="-12.7"/>
+<vertex x="-17.78" y="-9.7" curve="90"/>
+<vertex x="-14.78" y="-12.7"/>
 <vertex x="87.4" y="-12.7" curve="90"/>
 <vertex x="90.4" y="-9.7"/>
 <vertex x="90.4" y="53" curve="90"/>
-<vertex x="87.4" y="56"/>
-<vertex x="-22.4" y="56" curve="90"/>
-<vertex x="-25.4" y="53"/>
+<vertex x="87.4" y="56.3175"/>
+<vertex x="-14.78" y="56.3175" curve="90"/>
+<vertex x="-17.78" y="53"/>
 </polygon>
 <polygon width="0.254" layer="1">
-<vertex x="-25.4" y="-9.7" curve="90"/>
-<vertex x="-22.4" y="-12.7"/>
+<vertex x="-17.78" y="-9.7" curve="90"/>
+<vertex x="-14.78" y="-12.7"/>
 <vertex x="87.4" y="-12.7" curve="90"/>
 <vertex x="90.4" y="-9.7"/>
 <vertex x="90.4" y="53" curve="90"/>
-<vertex x="87.4" y="56"/>
-<vertex x="-22.4" y="56" curve="90"/>
-<vertex x="-25.4" y="53"/>
+<vertex x="87.4" y="56.3175"/>
+<vertex x="-14.78" y="56.3175" curve="90"/>
+<vertex x="-17.78" y="53"/>
 </polygon>
 <contactref element="CN1" pad="2"/>
@@
 <wire x1="57.277" y1="31.115" x2="57.4675" y2="31.115" width="0.6096" layer="1"/>
 <wire x1="57.4675" y1="31.115" x2="59.69" y2="31.115" width="0.6096" layer="1"/>
-<wire x1="85.09" y1="1.905" x2="78.4225" y2="1.905" width="0.8128" layer="16"/>
-<wire x1="78.4225" y1="1.905" x2="73.67" y2="6.6575" width="0.8128" layer="16"/>
-<wire x1="73.67" y1="6.6575" x2="73.67" y2="52.218" width="0.8128" layer="16"/>
 <wire x1="73.67" y1="52.218" x2="69.6805" y2="52.218" width="0.6096" layer="1"/>
 <wire x1="69.6805" y1="52.218" x2="56.515" y2="39.0525" width="0.6096" layer="1"/>
 <wire x1="56.515" y1="39.0525" x2="56.515" y2="32.0675" width="0.6096" layer="1"/>
 <wire x1="56.515" y1="32.0675" x2="57.4675" y2="31.115" width="0.6096" layer="1"/>
+<wire x1="73.67" y1="52.218" x2="83.037" y2="52.218" width="0.6096" layer="1"/>
+<wire x1="83.037" y1="52.218" x2="85.09" y2="50.165" width="0.6096" layer="1"/>
+<via x="85.09" y="50.165" extent="1-16" drill="0.9" shape="octagon"/>
+<wire x1="85.09" y1="50.165" x2="85.09" y2="28.2575" width="0.6096" layer="16"/>
+<wire x1="85.09" y1="28.2575" x2="81.28" y2="24.4475" width="0.6096" layer="16"/>
+<wire x1="81.28" y1="24.4475" x2="81.28" y2="11.7475" width="0.6096" layer="16"/>
+<wire x1="81.28" y1="11.7475" x2="85.09" y2="7.9375" width="0.6096" layer="16"/>
+<wire x1="85.09" y1="7.9375" x2="85.09" y2="1.905" width="0.6096" layer="16"/>
 </signal>
 <signal name="N$6">
@@
 <wire x1="64.77" y1="32.385" x2="63.9975" y2="32.385" width="0.6096" layer="1"/>
 </signal>
+<signal name="N$5">
+<via x="3.4925" y="21.59" extent="1-16" drill="0.6"/>
+</signal>
+<signal name="N$7">
+<via x="17.145" y="21.59" extent="1-16" drill="0.6"/>
+</signal>
+<signal name="N$8">
+<via x="3.4925" y="3.4925" extent="1-16" drill="0.6"/>
+</signal>
+<signal name="N$9">
+<via x="61.2775" y="21.59" extent="1-16" drill="0.6"/>
+</signal>
+<signal name="N$10">
+<via x="85.725" y="21.59" extent="1-16" drill="0.6"/>
+</signal>
+<signal name="N$11">
+<via x="61.595" y="3.4925" extent="1-16" drill="0.6"/>
+</signal>
+<signal name="N$12">
+<via x="61.595" y="52.3875" extent="1-16" drill="0.6"/>
+</signal>
+<signal name="N$13">
+<via x="3.4925" y="52.3875" extent="1-16" drill="0.6"/>
+</signal>
 </signals>
