File: AT90CAN128 era and older/Gearnode/H-bro_gear.sch (EAGLE design)
At the start: 32 parts, among them IC2 74AC08D, IC3 4070D, IC4 7805T, IC6 TL074P, X3 22-23-2031, X4 22-23-2041

Commit message: redid power circuitry to accomondate oversight
forget the laser needed 5V DOH!
Changed lines of the file:
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@@
 <instance part="X1" gate="-1" x="45.72" y="53.34"/>
 <instance part="X1" gate="-2" x="40.64" y="53.34" rot="R180"/>
-<instance part="IC3" gate="A" x="162.56" y="76.2"/>
-<instance part="IC3" gate="C" x="160.02" y="88.9"/>
 <instance part="IC3" gate="D" x="-10.16" y="30.48"/>
 <instance part="IC2" gate="C" x="-35.56" y="22.86"/>
