File: STM32F407 era/Com-node/Schematic.sch (EAGLE design)
At the start: 2 parts, among them X1 SDBMF

Commit message: update
Parts:
- added C1, C2, C4: 100nF, resistor:C-EU050-024X044
- added C3: 4.7uF, rcl:CPOL-EUE15-5AXIAL
- added C5: 100uF, rcl:CPOL-EUE15-5AXIAL
- added C6: xuF, rcl:CPOL-EUE15-5AXIAL
- added LED1, LED2, LED3, LED4, LED5: (no value), led:LED3MM
- added LM2575-ADJ: LM2596S, national-semiconductor:LM2596S
- added R1, R2, R8, R9: (no value), resistor:R-EU_0207/10
- added R10, R11: X, resistor:R-EU_0207/10
- added R3, R4, R5, R6: 47k, resistor:R-EU_0207/10
- added R7: 500, resistor:R-EU_0207/10
- added U$1: CPU-BOARD, unicorn_v2:CPU-BOARD
- added XB2: XBEE-PRO, maxstream:XBEE-PRO
- XB1: device microbuilder:XBEE-PRO -> maxstream:XBEE-PRO
Connections:
- new net +3.3V: C4.1, XB2.!RESET, XB2.VCC
- new net +3V3: C1.1, C2.1, C3.+, LED3.A, LM2575-ADJ.OUT, R10.2, R3.1, R4.1, R5.1, U$1G$2.VCC1, X1.4, XB1.!RESET, XB1.VCC
- new net 12V: C5.+, LM2575-ADJ.VIN
- new net N$1: LED1.C, R2.2
- new net N$13: LM2575-ADJ.FB, R10.1, R11.2
- new net N$2: LED1.A, XB1.PWM0/RSSI
- new net N$3: LED4.C, R9.2
- new net N$4: LED4.A, XB2.PWM0/RSSI
- new net N$5: LED2.A, XB1.ASSOC/AD5/DIO5
- new net N$6: LED2.C, R1.2
- new net N$7: LED5.A, XB2.ASSOC/AD5/DIO5
- new net N$8: LED5.C, R8.2
- new net N$9: LED3.C, R7.2
- new net PE: C1.2, C2.2, C3.-, C4.2, C5.-, LM2575-ADJ.!ON!/OFF, LM2575-ADJ.GND, R1.1, R11.1, R2.1, R6.1, R8.1, R9.1, X1.3, X1.6, XB1.GND, XB2.GND
- new net RX-XBEE: U$1G$4.PA1, XB1.DOUT, XB2.DOUT
- new net SD-CS: R3.2, R7.1, U$1G$1.PA4, X1.1
- new net SD-MISO: R5.2, U$1G$1.PA6, X1.7
- new net SD-MOSI: R4.2, U$1G$1.PA7, X1.2
- new net SD-SCK: R6.2, U$1G$1.PA5, X1.5
- new net TX-XBEE: U$1G$4.PA0, XB1.DIN/!CONFIG
Other:
- moved on the sheet: X1, XB1

Commit message: Update
Parts:
- removed R1, R2: (no value), resistor:R-EU_0207/10
- added D1: 1N5638, diode:1N5638
- added L1: 220µH, SparkFun-Passives:INDUCTORPWR
- R10: value X -> 1K69; device resistor:R-EU_0207/10 -> microbuilder:RESISTOR_0603
- R11: value X -> 1K; device resistor:R-EU_0207/10 -> microbuilder:RESISTOR_0603
- R3, R4, R5, R6, R7, R8, R9: device resistor:R-EU_0207/10 -> microbuilder:RESISTOR_0603
Connections:
- net N$1: no longer R2.2
- net N$6: no longer R1.2
- net PE: no longer R1.1, R2.1

Commit message: Updated
Parts:
- C6: value xuF -> 220uF
Connections:
- new net N$10: D1.C, L1.1, LM2575-ADJ.OUT
- net +3V3: now also C6.+, L1.2; no longer LM2575-ADJ.OUT
- net PE: now also C6.-, D1.A
Other:
- moved on the sheet: D1, L1
Changed lines of the file:
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@@
 <part name="C5" library="rcl" deviceset="CPOL-EU" device="E15-5AXIAL" value="100uF"/>
 <part name="SUPPLY3" library="supply2" deviceset="PE" device=""/>
-<part name="C6" library="rcl" deviceset="CPOL-EU" device="E15-5AXIAL" value="xuF"/>
+<part name="C6" library="rcl" deviceset="CPOL-EU" device="E15-5AXIAL" value="220uF"/>
 <part name="R10" library="microbuilder" deviceset="RESISTOR" device="_0603" value="1K69"/>
 <part name="R11" library="microbuilder" deviceset="RESISTOR" device="_0603" value="1K"/>
@@
 <instance part="R11" gate="G$1" x="-101.6" y="-27.94" rot="R90"/>
 <instance part="P+2" gate="G$1" x="-101.6" y="-5.08"/>
-<instance part="L1" gate="G$1" x="-132.08" y="-45.72"/>
-<instance part="D1" gate="1" x="-157.48" y="-45.72"/>
+<instance part="L1" gate="G$1" x="-124.46" y="-7.62" rot="R90"/>
+<instance part="D1" gate="1" x="-132.08" y="-25.4" rot="R90"/>
 </instances>
 <busses>
@@
 <junction x="-182.88" y="-15.24"/>
 <pinref part="R11" gate="G$1" pin="1"/>
-<wire x1="-101.6" y1="-33.02" x2="-170.18" y2="-33.02" width="0.1524" layer="91"/>
+<wire x1="-101.6" y1="-33.02" x2="-114.3" y2="-33.02" width="0.1524" layer="91"/>
+<wire x1="-114.3" y1="-33.02" x2="-132.08" y2="-33.02" width="0.1524" layer="91"/>
+<wire x1="-132.08" y1="-33.02" x2="-170.18" y2="-33.02" width="0.1524" layer="91"/>
 <wire x1="-170.18" y1="-33.02" x2="-170.18" y2="-17.78" width="0.1524" layer="91"/>
 <junction x="-170.18" y="-17.78"/>
+<pinref part="D1" gate="1" pin="A"/>
+<wire x1="-132.08" y1="-27.94" x2="-132.08" y2="-33.02" width="0.1524" layer="91"/>
+<junction x="-132.08" y="-33.02"/>
+<pinref part="C6" gate="G$1" pin="-"/>
+<wire x1="-114.3" y1="-17.78" x2="-114.3" y2="-33.02" width="0.1524" layer="91"/>
+<junction x="-114.3" y="-33.02"/>
 </segment>
 </net>
@@
 <pinref part="P+4" gate="G$1" pin="+3V3"/>
 <wire x1="-76.2" y1="2.54" x2="-76.2" y2="7.62" width="0.1524" layer="91"/>
-</segment>
-<segment>
-<pinref part="LM2575-ADJ" gate="G$1" pin="OUT"/>
-<wire x1="-142.24" y1="-10.16" x2="-139.7" y2="-10.16" width="0.1524" layer="91"/>
+<label x="-101.6" y="-7.62" size="1.27" layer="95" xref="yes"/>
+</segment>
+<segment>
 <pinref part="R10" gate="G$1" pin="2"/>
-<wire x1="-101.6" y1="-7.62" x2="-139.7" y2="-7.62" width="0.1524" layer="91"/>
-<wire x1="-139.7" y1="-7.62" x2="-139.7" y2="-10.16" width="0.1524" layer="91"/>
 <pinref part="P+2" gate="G$1" pin="+3V3"/>
+<pinref part="L1" gate="G$1" pin="2"/>
+<wire x1="-116.84" y1="-7.62" x2="-114.3" y2="-7.62" width="0.1524" layer="91"/>
 <junction x="-101.6" y="-7.62"/>
-<label x="-101.6" y="-7.62" size="1.27" layer="95" xref="yes"/>
+<pinref part="C6" gate="G$1" pin="+"/>
+<wire x1="-114.3" y1="-7.62" x2="-101.6" y2="-7.62" width="0.1524" layer="91"/>
+<wire x1="-114.3" y1="-10.16" x2="-114.3" y2="-7.62" width="0.1524" layer="91"/>
+<junction x="-114.3" y="-7.62"/>
 </segment>
 <segment>
@@
 </segment>
 </net>
+<net name="N$10" class="0">
+<segment>
+<pinref part="LM2575-ADJ" gate="G$1" pin="OUT"/>
+<wire x1="-142.24" y1="-10.16" x2="-139.7" y2="-10.16" width="0.1524" layer="91"/>
+<wire x1="-139.7" y1="-7.62" x2="-139.7" y2="-10.16" width="0.1524" layer="91"/>
+<pinref part="L1" gate="G$1" pin="1"/>
+<wire x1="-139.7" y1="-7.62" x2="-132.08" y2="-7.62" width="0.1524" layer="91"/>
+<pinref part="D1" gate="1" pin="C"/>
+<wire x1="-132.08" y1="-22.86" x2="-132.08" y2="-7.62" width="0.1524" layer="91"/>
+<junction x="-132.08" y="-7.62"/>
+</segment>
+</net>

Commit message: Update
Connections:
- net 12V renamed 14.2V
Changed lines of the file:
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@@
 <grid distance="0.1" unitdist="inch" unit="inch" style="lines" multiple="1" display="no" altdistance="0.01" altunitdist="inch" altunit="inch"/>
 <layers>
-<layer number="1" name="Top" color="4" fill="1" visible="yes" active="no"/>
-<layer number="2" name="Route2" color="1" fill="3" visible="yes" active="no"/>
-<layer number="3" name="Route3" color="4" fill="3" visible="yes" active="no"/>
-<layer number="4" name="Route4" color="1" fill="4" visible="yes" active="no"/>
-<layer number="5" name="Route5" color="4" fill="4" visible="yes" active="no"/>
-<layer number="6" name="Route6" color="1" fill="8" visible="yes" active="no"/>
-<layer number="7" name="Route7" color="4" fill="8" visible="yes" active="no"/>
-<layer number="8" name="Route8" color="1" fill="2" visible="yes" active="no"/>
-<layer number="9" name="Route9" color="4" fill="2" visible="yes" active="no"/>
-<layer number="10" name="Route10" color="1" fill="7" visible="yes" active="no"/>
-<layer number="11" name="Route11" color="4" fill="7" visible="yes" active="no"/>
-<layer number="12" name="Route12" color="1" fill="5" visible="yes" active="no"/>
-<layer number="13" name="Route13" color="4" fill="5" visible="yes" active="no"/>
-<layer number="14" name="Route14" color="1" fill="6" visible="yes" active="no"/>
-<layer number="15" name="Route15" color="4" fill="6" visible="yes" active="no"/>
-<layer number="16" name="Bottom" color="1" fill="1" visible="yes" active="no"/>
-<layer number="17" name="Pads" color="2" fill="1" visible="yes" active="no"/>
-<layer number="18" name="Vias" color="2" fill="1" visible="yes" active="no"/>
-<layer number="19" name="Unrouted" color="6" fill="1" visible="yes" active="no"/>
-<layer number="20" name="Dimension" color="15" fill="1" visible="yes" active="no"/>
-<layer number="21" name="tPlace" color="16" fill="1" visible="yes" active="no"/>
-<layer number="22" name="bPlace" color="14" fill="1" visible="yes" active="no"/>
-<layer number="23" name="tOrigins" color="15" fill="1" visible="yes" active="no"/>
-<layer number="24" name="bOrigins" color="15" fill="1" visible="yes" active="no"/>
-<layer number="25" name="tNames" color="7" fill="1" visible="yes" active="no"/>
-<layer number="26" name="bNames" color="7" fill="1" visible="yes" active="no"/>
-<layer number="27" name="tValues" color="7" fill="1" visible="yes" active="no"/>
-<layer number="28" name="bValues" color="7" fill="1" visible="yes" active="no"/>
+<layer number="1" name="Top" color="4" fill="1" visible="no" active="no"/>
+<layer number="2" name="Route2" color="1" fill="3" visible="no" active="no"/>
+<layer number="3" name="Route3" color="4" fill="3" visible="no" active="no"/>
+<layer number="4" name="Route4" color="1" fill="4" visible="no" active="no"/>
+<layer number="5" name="Route5" color="4" fill="4" visible="no" active="no"/>
+<layer number="6" name="Route6" color="1" fill="8" visible="no" active="no"/>
+<layer number="7" name="Route7" color="4" fill="8" visible="no" active="no"/>
+<layer number="8" name="Route8" color="1" fill="2" visible="no" active="no"/>
+<layer number="9" name="Route9" color="4" fill="2" visible="no" active="no"/>
+<layer number="10" name="Route10" color="1" fill="7" visible="no" active="no"/>
+<layer number="11" name="Route11" color="4" fill="7" visible="no" active="no"/>
+<layer number="12" name="Route12" color="1" fill="5" visible="no" active="no"/>
+<layer number="13" name="Route13" color="4" fill="5" visible="no" active="no"/>
+<layer number="14" name="Route14" color="1" fill="6" visible="no" active="no"/>
+<layer number="15" name="Route15" color="4" fill="6" visible="no" active="no"/>
+<layer number="16" name="Bottom" color="1" fill="1" visible="no" active="no"/>
+<layer number="17" name="Pads" color="2" fill="1" visible="no" active="no"/>
+<layer number="18" name="Vias" color="2" fill="1" visible="no" active="no"/>
+<layer number="19" name="Unrouted" color="6" fill="1" visible="no" active="no"/>
+<layer number="20" name="Dimension" color="15" fill="1" visible="no" active="no"/>
+<layer number="21" name="tPlace" color="16" fill="1" visible="no" active="no"/>
+<layer number="22" name="bPlace" color="14" fill="1" visible="no" active="no"/>
+<layer number="23" name="tOrigins" color="15" fill="1" visible="no" active="no"/>
+<layer number="24" name="bOrigins" color="15" fill="1" visible="no" active="no"/>
+<layer number="25" name="tNames" color="7" fill="1" visible="no" active="no"/>
+<layer number="26" name="bNames" color="7" fill="1" visible="no" active="no"/>
+<layer number="27" name="tValues" color="7" fill="1" visible="no" active="no"/>
+<layer number="28" name="bValues" color="7" fill="1" visible="no" active="no"/>
 <layer number="29" name="tStop" color="7" fill="3" visible="no" active="no"/>
 <layer number="30" name="bStop" color="7" fill="6" visible="no" active="no"/>
@@
 <layer number="35" name="tGlue" color="7" fill="4" visible="no" active="no"/>
 <layer number="36" name="bGlue" color="7" fill="5" visible="no" active="no"/>
-<layer number="37" name="tTest" color="7" fill="1" visible="yes" active="no"/>
-<layer number="38" name="bTest" color="7" fill="1" visible="yes" active="no"/>
+<layer number="37" name="tTest" color="7" fill="1" visible="no" active="no"/>
+<layer number="38" name="bTest" color="7" fill="1" visible="no" active="no"/>
 <layer number="39" name="tKeepout" color="4" fill="11" visible="no" active="no"/>
 <layer number="40" name="bKeepout" color="1" fill="11" visible="no" active="no"/>
@@
 <layer number="44" name="Drills" color="7" fill="1" visible="no" active="no"/>
 <layer number="45" name="Holes" color="7" fill="1" visible="no" active="no"/>
-<layer number="46" name="Milling" color="3" fill="1" visible="yes" active="no"/>
-<layer number="47" name="Measures" color="7" fill="1" visible="yes" active="no"/>
-<layer number="48" name="Document" color="7" fill="1" visible="yes" active="no"/>
-<layer number="49" name="Reference" color="7" fill="1" visible="yes" active="no"/>
-<layer number="50" name="dxf" color="7" fill="1" visible="yes" active="no"/>
-<layer number="51" name="tDocu" color="6" fill="1" visible="yes" active="no"/>
-<layer number="52" name="bDocu" color="7" fill="1" visible="yes" active="no"/>
-<layer number="53" name="tGND_GNDA" color="7" fill="9" visible="yes" active="no"/>
-<layer number="54" name="bGND_GNDA" color="1" fill="9" visible="yes" active="no"/>
-<layer number="56" name="wert" color="7" fill="1" visible="yes" active="no"/>
+<layer number="46" name="Milling" color="3" fill="1" visible="no" active="no"/>
+<layer number="47" name="Measures" color="7" fill="1" visible="no" active="no"/>
+<layer number="48" name="Document" color="7" fill="1" visible="no" active="no"/>
+<layer number="49" name="Reference" color="7" fill="1" visible="no" active="no"/>
+<layer number="50" name="dxf" color="7" fill="1" visible="no" active="no"/>
+<layer number="51" name="tDocu" color="6" fill="1" visible="no" active="no"/>
+<layer number="52" name="bDocu" color="7" fill="1" visible="no" active="no"/>
+<layer number="53" name="tGND_GNDA" color="7" fill="9" visible="no" active="no"/>
+<layer number="54" name="bGND_GNDA" color="1" fill="9" visible="no" active="no"/>
+<layer number="56" name="wert" color="7" fill="1" visible="no" active="no"/>
 <layer number="91" name="Nets" color="2" fill="1" visible="yes" active="yes"/>
 <layer number="92" name="Busses" color="1" fill="1" visible="yes" active="yes"/>
@@
 </segment>
 </net>
-<net name="12V" class="0">
+<net name="14.2V" class="0">
 <segment>
 <pinref part="LM2575-ADJ" gate="G$1" pin="VIN"/>

Commit message: Update
Parts:
- removed LED1, LED4, LED5: (no value), led:LED3MM
- removed R9: (no value), microbuilder:RESISTOR_0603
- removed XB2: XBEE-PRO, maxstream:XBEE-PRO
- added C7: 1uF, rcl:CPOL-EUE15-5AXIAL
- added Q1: (no value), microbuilder:TRANSISTOR_NPNWIDE
- added R1: 850, microbuilder:RESISTOR_0603
Connections:
- removed net N$3: LED4.C, R9.2
- removed net N$4: LED4.A, XB2.PWM0/RSSI
- removed net N$7: LED5.A, XB2.ASSOC/AD5/DIO5
- new net CTS-XBEE: U$1G$4.PA2, XB1.!CTS!/DIO7
- new net RTS-XBEE: U$1G$4.PC3, XB1.!RTS!/AD6/DIO6
- new net SS-XBEE: U$1G$1.PA3
- new net V-SENSE: Q1.E, U$1G$2.PA8
- net +3.3V: no longer XB2.!RESET, XB2.VCC
- net +3V3: now also Q1.C
- net 14.2V: now also Q1.B
- net N$1: now also C7.+, R1.2; no longer LED1.C
- net N$2: now also R1.1; no longer LED1.A
- net N$8: no longer LED5.C
- net PE: now also C7.-; no longer C1.2, R9.1, XB2.GND
- net RX-XBEE: no longer XB2.DOUT
Other:
- moved on the sheet: C1, C2, C3, C4, LED2, LED3, R3, R4, R5, R6, R7, R8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

Commit message: Updates
Parts:
- added C8: SUPERCAP, unicorn_v2:SUPERCAP
- added LED1, LED4: (no value), led:LEDCHIPLED_1206
- added R2, R9: 500, microbuilder:RESISTOR_0603
- added X2: 057-006-1, con-panduit:057-006-1
Connections:
- new net DEBUG-LED1: R9.2
- new net DEBUG-LED2: R2.2
- new net N$11: U$1G$4.PE3
- new net N$12: U$1G$4.PE5
- new net N$3: LED1.A, R2.1
- new net N$7: LED4.A, R9.1
- new net UART3-RX: U$1G$1.PB11
- new net UART3-TX: U$1G$1.PB10, X2-1.S
- new net UART4-RX: U$1G$3.PC11
- new net UART4-TX: U$1G$3.PC10
- net PE: now also LED1.C, LED4.C, X2-4.S

Commit message: First schematic revision for com-node done
Parts:
- added R12: 20K, microbuilder:RESISTOR_0603
- added R13: 1K8, microbuilder:RESISTOR_0603
- added U1: MAX13052ESA+, Maxim_By_element14_Batch_1:MAX13052ESA+
- added X3: 22-23-2041, con-molex:22-23-2041
Connections:
- removed net 14.2V: C5.+, LM2575-ADJ.VIN, Q1.B
- new net +14V2: C5.+, LM2575-ADJ.VIN, R12.1, X3-3.S
- new net ECU_CAN_H: R13.1, U1.CANH, X3-1.S
- new net ECU_CAN_L: R13.2, U1.CANL, X3-2.S
- new net ECU_CAN_RX: U$1G$2.PB12, U1.RXD
- new net ECU_CAN_TX: U$1G$2.PB13, U1.TXD
- new net N$14: Q1.B, R12.2
- net +3V3: now also U1.VCC
- net PE: now also U1.GND, U1.RS, X3-4.S
Other:
- moved on the sheet: Q1
Changed lines of the file:
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@@
 <part name="X2" library="con-panduit" deviceset="057-006-" device="1"/>
 <part name="SUPPLY8" library="supply2" deviceset="PE" device=""/>
+<part name="R12" library="microbuilder" deviceset="RESISTOR" device="_0603" value="20K"/>
+<part name="U1" library="Maxim_By_element14_Batch_1" deviceset="MAX13052ESA+" device=""/>
+<part name="SUPPLY10" library="supply2" deviceset="PE" device=""/>
+<part name="SUPPLY11" library="supply2" deviceset="PE" device=""/>
+<part name="R13" library="microbuilder" deviceset="RESISTOR" device="_0603" value="1K8"/>
+<part name="X3" library="con-molex" deviceset="22-23-2041" device=""/>
 </parts>
 <sheets>
@@
 <instance part="R1" gate="G$1" x="-5.08" y="-7.62" rot="R180"/>
 <instance part="C7" gate="G$1" x="-20.32" y="-12.7"/>
-<instance part="Q1" gate="G$1" x="-172.72" y="7.62" rot="R90"/>
+<instance part="Q1" gate="G$1" x="-172.72" y="12.7" rot="R90"/>
 <instance part="LED1" gate="G$1" x="114.3" y="40.64"/>
 <instance part="LED4" gate="G$1" x="129.54" y="40.64"/>
@@
 <instance part="X2" gate="-6" x="-132.08" y="-76.2"/>
 <instance part="SUPPLY8" gate="PE" x="-144.78" y="-83.82"/>
+<instance part="R12" gate="G$1" x="-172.72" y="0" rot="R90"/>
+<instance part="U1" gate="A" x="60.96" y="-109.22"/>
+<instance part="SUPPLY10" gate="PE" x="38.1" y="-127"/>
+<instance part="SUPPLY11" gate="PE" x="-43.18" y="-109.22"/>
+<instance part="R13" gate="G$1" x="-58.42" y="-101.6" rot="R270"/>
+<instance part="X3" gate="-1" x="-38.1" y="-96.52"/>
+<instance part="X3" gate="-2" x="-38.1" y="-99.06"/>
+<instance part="X3" gate="-3" x="-38.1" y="-101.6"/>
+<instance part="X3" gate="-4" x="-38.1" y="-104.14"/>
 </instances>
 <busses>
@@
 <wire x1="-144.78" y1="-81.28" x2="-144.78" y2="-71.12" width="0.1524" layer="91"/>
 </segment>
+<segment>
+<pinref part="U1" gate="A" pin="GND"/>
+<wire x1="43.18" y1="-121.92" x2="38.1" y2="-121.92" width="0.1524" layer="91"/>
+<wire x1="38.1" y1="-121.92" x2="38.1" y2="-124.46" width="0.1524" layer="91"/>
+<pinref part="U1" gate="A" pin="RS"/>
+<wire x1="43.18" y1="-109.22" x2="38.1" y2="-109.22" width="0.1524" layer="91"/>
+<wire x1="38.1" y1="-109.22" x2="38.1" y2="-121.92" width="0.1524" layer="91"/>
+<junction x="38.1" y="-121.92"/>
+<pinref part="SUPPLY10" gate="PE" pin="PE"/>
+</segment>
+<segment>
+<pinref part="SUPPLY11" gate="PE" pin="PE"/>
+<wire x1="-43.18" y1="-104.14" x2="-43.18" y2="-106.68" width="0.1524" layer="91"/>
+<wire x1="-40.64" y1="-104.14" x2="-43.18" y2="-104.14" width="0.1524" layer="91"/>
+<pinref part="X3" gate="-4" pin="S"/>
+</segment>
 </net>
 <net name="SD-SCK" class="0">
@@
 <segment>
 <pinref part="Q1" gate="G$1" pin="C"/>
-<wire x1="-177.8" y1="7.62" x2="-180.34" y2="7.62" width="0.1524" layer="91"/>
-<label x="-180.34" y="7.62" size="1.27" layer="95" rot="R180" xref="yes"/>
-</segment>
-</net>
-<net name="14.2V" class="0">
+<wire x1="-177.8" y1="12.7" x2="-180.34" y2="12.7" width="0.1524" layer="91"/>
+<label x="-180.34" y="12.7" size="1.27" layer="95" rot="R180" xref="yes"/>
+</segment>
+<segment>
+<pinref part="U1" gate="A" pin="VCC"/>
+<wire x1="43.18" y1="-101.6" x2="40.64" y2="-101.6" width="0.1524" layer="91"/>
+<label x="40.64" y="-101.6" size="1.27" layer="95" rot="R180" xref="yes"/>
+</segment>
+</net>
+<net name="+14V2" class="0">
 <segment>
 <pinref part="LM2575-ADJ" gate="G$1" pin="VIN"/>
 <pinref part="C5" gate="G$1" pin="+"/>
+<label x="-182.88" y="-7.62" size="1.27" layer="95" rot="R180" xref="yes"/>
 <wire x1="-167.64" y1="-7.62" x2="-172.72" y2="-7.62" width="0.1524" layer="91"/>
-<label x="-182.88" y="-7.62" size="1.27" layer="95" rot="R180" xref="yes"/>
-<pinref part="Q1" gate="G$1" pin="B"/>
+<pinref part="R12" gate="G$1" pin="1"/>
 <wire x1="-172.72" y1="-7.62" x2="-182.88" y2="-7.62" width="0.1524" layer="91"/>
-<wire x1="-172.72" y1="2.54" x2="-172.72" y2="-7.62" width="0.1524" layer="91"/>
+<wire x1="-172.72" y1="-7.62" x2="-172.72" y2="-5.08" width="0.1524" layer="91"/>
 <junction x="-172.72" y="-7.62"/>
+</segment>
+<segment>
+<pinref part="X3" gate="-3" pin="S"/>
+<wire x1="-40.64" y1="-101.6" x2="-48.26" y2="-101.6" width="0.1524" layer="91"/>
+<wire x1="-48.26" y1="-101.6" x2="-48.26" y2="-111.76" width="0.1524" layer="91"/>
+<wire x1="-48.26" y1="-111.76" x2="-50.8" y2="-111.76" width="0.1524" layer="91"/>
+<label x="-50.8" y="-111.76" size="1.27" layer="95" rot="R180" xref="yes"/>
 </segment>
 </net>
@@
 <segment>
 <pinref part="Q1" gate="G$1" pin="E"/>
-<wire x1="-167.64" y1="7.62" x2="-165.1" y2="7.62" width="0.1524" layer="91"/>
-<label x="-165.1" y="7.62" size="1.27" layer="95" xref="yes"/>
+<wire x1="-167.64" y1="12.7" x2="-162.56" y2="12.7" width="0.1524" layer="91"/>
+<label x="-162.56" y="12.7" size="1.27" layer="95" xref="yes"/>
 </segment>
 <segment>
@@
 </segment>
 </net>
+<net name="N$14" class="0">
+<segment>
+<pinref part="Q1" gate="G$1" pin="B"/>
+<pinref part="R12" gate="G$1" pin="2"/>
+<wire x1="-172.72" y1="7.62" x2="-172.72" y2="5.08" width="0.1524" layer="91"/>
+</segment>
+</net>
+<net name="ECU_CAN_TX" class="0">
+<segment>
+<pinref part="U$1" gate="G$2" pin="PB13"/>
+<wire x1="-55.88" y1="60.96" x2="-53.34" y2="60.96" width="0.1524" layer="91"/>
+<label x="-53.34" y="60.96" size="1.27" layer="95" xref="yes"/>
+</segment>
+<segment>
+<pinref part="U1" gate="A" pin="TXD"/>
+<wire x1="43.18" y1="-106.68" x2="35.56" y2="-106.68" width="0.1524" layer="91"/>
+<label x="35.56" y="-106.68" size="1.27" layer="95" rot="R180" xref="yes"/>
+</segment>
+</net>
+<net name="ECU_CAN_H" class="0">
+<segment>
+<pinref part="U1" gate="A" pin="CANH"/>
+<wire x1="43.18" y1="-116.84" x2="33.02" y2="-116.84" width="0.1524" layer="91"/>
+<label x="33.02" y="-116.84" size="1.27" layer="95" rot="R180" xref="yes"/>
+</segment>
+<segment>
+<pinref part="R13" gate="G$1" pin="1"/>
+<wire x1="-40.64" y1="-96.52" x2="-58.42" y2="-96.52" width="0.1524" layer="91"/>
+<wire x1="-58.42" y1="-96.52" x2="-63.5" y2="-96.52" width="0.1524" layer="91"/>
+<junction x="-58.42" y="-96.52"/>
+<label x="-63.5" y="-96.52" size="1.27" layer="95" rot="R180" xref="yes"/>
+<pinref part="X3" gate="-1" pin="S"/>
+</segment>
+</net>
+<net name="ECU_CAN_L" class="0">
+<segment>
+<pinref part="U1" gate="A" pin="CANL"/>
+<wire x1="43.18" y1="-114.3" x2="33.02" y2="-114.3" width="0.1524" layer="91"/>
+<label x="33.02" y="-114.3" size="1.27" layer="95" rot="R180" xref="yes"/>
+</segment>
+<segment>
+<pinref part="R13" gate="G$1" pin="2"/>
+<wire x1="-58.42" y1="-106.68" x2="-53.34" y2="-106.68" width="0.1524" layer="91"/>
+<wire x1="-53.34" y1="-106.68" x2="-53.34" y2="-99.06" width="0.1524" layer="91"/>
+<wire x1="-53.34" y1="-99.06" x2="-40.64" y2="-99.06" width="0.1524" layer="91"/>
+<wire x1="-58.42" y1="-106.68" x2="-63.5" y2="-106.68" width="0.1524" layer="91"/>
+<junction x="-58.42" y="-106.68"/>
+<label x="-63.5" y="-106.68" size="1.27" layer="95" rot="R180" xref="yes"/>
+<pinref part="X3" gate="-2" pin="S"/>
+</segment>
+</net>
+<net name="ECU_CAN_RX" class="0">
+<segment>
+<pinref part="U$1" gate="G$2" pin="PB12"/>
+<wire x1="-78.74" y1="60.96" x2="-81.28" y2="60.96" width="0.1524" layer="91"/>
+<label x="-81.28" y="60.96" size="1.27" layer="95" rot="R180" xref="yes"/>
+</segment>
+<segment>
+<pinref part="U1" gate="A" pin="RXD"/>
+<wire x1="78.74" y1="-101.6" x2="81.28" y2="-101.6" width="0.1524" layer="91"/>
+<label x="81.28" y="-101.6" size="1.27" layer="95" xref="yes"/>
+</segment>
+</net>
