File: STM32F407 era/Com-node/Schematic.sch (EAGLE design)
At the start: 35 parts, among them U1 MAX13052ESA+, X1 SDBMF, X2 057-006-1, X3 22-23-2041

Commit message: Update on board
Still some ERC warnings to solve
Parts:
- removed C3: 4.7uF, rcl:CPOL-EUE15-5AXIAL
- removed C4: 100nF, resistor:C-EU050-024X044
- removed LED3: (no value), led:LED3MM
- removed R13: 1K8, microbuilder:RESISTOR_0603
- removed X3: 22-23-2041, con-molex:22-23-2041
- added R14: XXXXX, microbuilder:RESISTOR_0603
- added R15, R16: 60, microbuilder:RESISTOR_0603
- added X4: (no value), con-molex:22-23-2061
- C2: value 100nF -> 4n7; device resistor:C-EU050-024X044 -> microbuilder:CAP_CERAMIC0603
- R7: value 500 -> 47k
- R8: value (none) -> 500
Connections:
- net UART3-RX renamed UART3_RX
- removed net +3.3V: C4.1
- removed net N$1 (its old number): C7.+, R1.2
- removed net N$9: LED3.C, R7.2
- removed net SD-CS: R3.2, R7.1, U$1G$1.PA4, X1.1
- removed net SD-MISO: R5.2, U$1G$1.PA6, X1.7
- removed net SD-MOSI: R4.2, U$1G$1.PA7, X1.2
- removed net SD-SCK: R6.2, U$1G$1.PA5, X1.5
- removed net UART3-TX: U$1G$1.PB10, X2-1.S
- removed net UART4-RX: U$1G$3.PC11
- removed net UART4-TX: U$1G$3.PC10
- new net N$15: X4-2.S
- new net N$16: R3.1, R4.1, R5.1, R6.1, R7.1
- new net N$19: X2-3.S, X2-4.S
- new net N$21: C2.P$1, R15.1, R16.1, U1.SPLIT
- new net N$4: X4-1.S
- new net SDIO_CMD: R3.2, U$1G$3.PD2, X1.2
- new net SDIO_D0: R4.2, U$1G$2.PC8, X1.7
- new net SDIO_D1: R6.2, U$1G$2.PA9, X1.8
- new net SDIO_D2: R7.2, U$1G$3.PC10, X1.9
- new net SDIO_D3: R5.2, U$1G$3.PC11, X1.1
- new net SDIO_SCK: U$1G$3.PC12, X1.5
- new net SD_IN: U$1G$3.PD3, X1.SW1
- new net UART3_TX: U$1G$1.PB10, X2-1.S, X2-2.S
- new net USART1_RX: U$1G$3.PB7
- new net USART1_TX: U$1G$3.PB6
- net +14V2: now also X4-5.S; no longer X3-3.S
- net +3V3: no longer C2.1, C3.+, LED3.A, R3.1, R4.1, R5.1
- net ECU_CAN_H: now also R15.2, X4-3.S; no longer R13.1, X3-1.S
- net ECU_CAN_L: now also R16.2, X4-4.S; no longer R13.2, X3-2.S
- net N$14: now also R14.2
- net N$6: now also R8.2
- net N$8: now also X1.SW3; no longer R8.2
- net PE: now also C1.2, C2.P$2, R14.1, X2-5.S, X2-6.S, X4-6.S; no longer C2.2, C3.-, C4.2, R6.1, X2-4.S, X3-4.S
- net RX-XBEE: no longer XB1.DOUT
- net SS-XBEE: now also C7.+, R1.2
Other:
- moved on the sheet: C2, R3, R4, R5, R6, R7
