File: STM32F407 era/Com-node/Schematic.brd (EAGLE design)
At the start: 76.2 x 66 mm, 27 parts, among them X1 SDBMF

Commit message: Update
Parts:
- removed R1, R2: (no value), resistor:0207/10
- added D1: 1N5638, diode:DO13M
- added L1: 220µH, SparkFun-Passives:CDRH125
- R10: value X -> 1K69; device resistor:0207/10 -> microbuilder:_0603
- R11: value X -> 1K; device resistor:0207/10 -> microbuilder:_0603
- R3, R4, R5, R6, R7, R8, R9: device resistor:0207/10 -> microbuilder:_0603
Connections:
- net N$1: no longer R2.2
- net N$6: no longer R1.2
- net PE: no longer R1.1, R2.1
Routing:
- net SD-CS: track 77.6 -> 90.6 mm
- net SD-MOSI: track 57.3 -> 66.0 mm
- net SD-MISO: track 43.4 -> 49.1 mm
- net N$6: track 4.95 -> 0.00 mm
- net N$9: track 6.81 -> 11.1 mm
- net SD-SCK: track 50.4 -> 52.9 mm
- net N$1: track 2.29 -> 0.00 mm
- net PE: track 52.9 -> 53.8 mm

Commit message: Updated
Parts:
- C6: value xuF -> 220uF
Connections:
- new net N$10: D1.C, L1.1, LM2575-ADJ.2
- net +3V3: now also C6.+, L1.2; no longer LM2575-ADJ.2
- net PE: now also C6.-, D1.A
Changed lines of the file:
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@@
 </element>
 <element name="C5" library="rcl" package="E15-5" value="100uF" x="-6.35" y="-96.52"/>
-<element name="C6" library="rcl" package="E15-5" value="xuF" x="-6.35" y="-106.68"/>
+<element name="C6" library="rcl" package="E15-5" value="220uF" x="-6.35" y="-106.68"/>
 <element name="R10" library="microbuilder" package="_0603" value="1K69" x="-8.89" y="-115.57"/>
 <element name="R11" library="microbuilder" package="_0603" value="1K" x="-8.89" y="-120.65"/>
@@
 <contactref element="C5" pad="-"/>
 <contactref element="R11" pad="1"/>
-<wire x1="1.27" y1="-96.52" x2="-9.652" y2="-120.65" width="0" layer="19" extent="1-1"/>
+<contactref element="D1" pad="A"/>
+<contactref element="C6" pad="-"/>
+<wire x1="-9.652" y1="-120.65" x2="-6.35" y2="-128.27" width="0" layer="19" extent="1-1"/>
+<wire x1="1.27" y1="-106.68" x2="-9.652" y2="-120.65" width="0" layer="19" extent="1-1"/>
+<wire x1="1.27" y1="-96.52" x2="1.27" y2="-106.68" width="0" layer="19" extent="1-1"/>
 <wire x1="-5.4864" y1="-89.6112" x2="1.27" y2="-96.52" width="0" layer="19" extent="1-1"/>
 <wire x1="-8.89" y1="-89.6112" x2="-5.4864" y2="-89.6112" width="0" layer="19" extent="1-1"/>
@@
 <wire x1="28.575" y1="13.589" x2="33.909" y2="9.271" width="0" layer="19" extent="1-1"/>
 <wire x1="30.184" y1="22.521" x2="28.575" y2="13.589" width="0" layer="19" extent="1-1"/>
-<wire x1="12.241" y1="40.53" x2="32.893" y2="24.13" width="0" layer="19" extent="1-1"/>
+<wire x1="12.241" y1="40.53" x2="30.184" y2="22.521" width="0" layer="19" extent="1-1"/>
 <wire x1="17.018" y1="52.832" x2="12.241" y2="40.53" width="0" layer="19" extent="1-1"/>
 </signal>
@@
 <contactref element="XB1" pad="5"/>
 <contactref element="C1" pad="1"/>
-<contactref element="LM2575-ADJ" pad="2"/>
 <contactref element="R10" pad="2"/>
 <contactref element="U$1" pad="P$43"/>
@@
 <vertex x="0" y="66.04"/>
 </polygon>
-<wire x1="-10.5918" y1="-89.6112" x2="-8.128" y2="-115.57" width="0" layer="19" extent="1-1"/>
-<wire x1="29.11475" y1="-49.94275" x2="-10.5918" y2="-89.6112" width="0" layer="19" extent="1-1"/>
+<contactref element="L1" pad="2"/>
+<contactref element="C6" pad="+"/>
+<wire x1="-8.128" y1="-115.57" x2="-22.86" y2="-119.2" width="0" layer="19" extent="1-1"/>
+<wire x1="-13.97" y1="-106.68" x2="-8.128" y2="-115.57" width="0" layer="19" extent="1-1"/>
+<wire x1="29.11475" y1="-49.94275" x2="-13.97" y2="-106.68" width="0" layer="19" extent="1-1"/>
 <wire x1="18.669" y1="9.271" x2="29.11475" y2="-49.94275" width="0" layer="19" extent="1-1"/>
 <wire x1="23.495" y1="13.589" x2="18.669" y2="9.271" width="0" layer="19" extent="1-1"/>
 <wire x1="32.893" y1="20.32" x2="23.495" y2="13.589" width="0" layer="19" extent="1-1"/>
-<wire x1="32.893" y1="27.94" x2="32.893" y2="20.32" width="0" layer="19" extent="1-1"/>
-<wire x1="34.29" y1="27.94" x2="32.893" y2="27.94" width="0" layer="19" extent="1-1"/>
+<wire x1="35.941" y1="26.289" x2="32.893" y2="20.32" width="0" layer="19" extent="1-1"/>
+<wire x1="32.893" y1="27.94" x2="34.29" y2="27.94" width="0" layer="19" extent="1-1"/>
 <wire x1="32.893" y1="35.433" x2="32.893" y2="27.94" width="0" layer="19" extent="1-1"/>
 <wire x1="20.701" y1="28.194" x2="32.893" y2="27.94" width="0" layer="19" extent="1-1"/>
-<wire x1="12.241" y1="50.53" x2="32.893" y2="35.433" width="0" layer="19" extent="1-1"/>
+<wire x1="12.241" y1="50.53" x2="20.701" y2="28.194" width="0" layer="19" extent="1-1"/>
 <wire x1="12.241" y1="58.53" x2="12.241" y2="50.53" width="0" layer="19" extent="1-1"/>
 <wire x1="17.018" y1="57.912" x2="12.241" y2="58.53" width="0" layer="19" extent="1-1"/>
@@
 <wire x1="-7.1882" y1="-89.6112" x2="-9.652" y2="-115.57" width="0" layer="19" extent="1-1"/>
 </signal>
+<signal name="N$10">
+<contactref element="LM2575-ADJ" pad="2"/>
+<contactref element="L1" pad="1"/>
+<contactref element="D1" pad="C"/>
+<wire x1="-22.86" y1="-109.4" x2="-26.67" y2="-128.27" width="0" layer="19" extent="1-1"/>
+<wire x1="-10.5918" y1="-89.6112" x2="-22.86" y2="-109.4" width="0" layer="19" extent="1-1"/>
+</signal>
 </signals>

Commit message: Update
Connections:
- net 12V renamed 14.2V
Changed lines of the file:
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@@
 <wire x1="17.018" y1="57.912" x2="12.241" y2="58.53" width="0" layer="19" extent="1-1"/>
 </signal>
-<signal name="12V">
+<signal name="14.2V">
 <contactref element="LM2575-ADJ" pad="1"/>
 <contactref element="C5" pad="+"/>

Commit message: Update
Parts:
- removed LED1, LED4, LED5: (no value), led:LED3MM
- removed R9: (no value), microbuilder:_0603
- removed XB2: XBEE-PRO, maxstream:XBEE-PRO
- added C7: 1uF, rcl:E15-5
- added Q1: (no value), microbuilder:SOT23-WIDE
- added R1: 850, microbuilder:_0603
- moved R8 63.3 mm to (45.7, 8.89), turned to 90 degrees
- moved X1 23.0 mm to (68.2, 51.2)
- moved C3 14.5 mm to (12.3, 5.46)
- moved C2 13.7 mm to (13.3, 18.7)
- moved C4 8.52 mm to (33.0, 3.81)
- moved XB1 7.73 mm to (15.6, 50.8)
- moved R4 5.08 mm to (28.6, 27.9)
- moved LED3 4.02 mm to (18.2, 26.9)
Connections:
- removed net N$3: LED4.K, R9.2
- removed net N$4: LED4.A, XB2.6
- removed net N$7: LED5.A, XB2.15
- new net CTS-XBEE: U$1.P$77, XB1.12
- new net RTS-XBEE: U$1.P$74, XB1.16
- new net SS-XBEE: U$1.P$1
- new net V-SENSE: Q1.2, U$1.P$39
- net +3.3V: no longer XB2.1, XB2.5
- net +3V3: now also Q1.3
- net 14.2V: now also Q1.1
- net N$1: now also C7.+, R1.2; no longer LED1.K
- net N$2: now also R1.1; no longer LED1.A
- net N$8: no longer LED5.K
- net PE: now also C7.-; no longer C1.2, R9.1, XB2.10
- net RX-XBEE: no longer XB2.2
Routing:
- net SD-CS: track 90.6 -> 0.00 mm
- net SD-MOSI: track 66.0 -> 0.00 mm
- net PE: track 53.8 -> 0.00 mm
- net SD-SCK: track 52.9 -> 0.00 mm
- net SD-MISO: track 49.1 -> 0.00 mm
- net RX-XBEE: track 44.0 -> 0.00 mm
- net +3V3: track 27.2 -> 0.00 mm
- net N$2: track 14.2 -> 0.00 mm
- net N$5: track 12.5 -> 0.00 mm
- net N$9: track 11.1 -> 0.00 mm
Other:
- board size 76.2 x 66 mm -> 118.1 x 66 mm
- board text removed: "Unicorn node1 v2.0"

Commit message: Updates
Parts:
- added C8: SUPERCAP, unicorn_v2:SUPERCAP
- added LED1, LED4: (no value), led:CHIPLED_1206
- added R2, R9: 500, microbuilder:_0603
- added X2: 057-006-1, con-panduit:057-006-1
Connections:
- new net DEBUG-LED1: R9.2
- new net DEBUG-LED2: R2.2
- new net N$11: U$1.P$64
- new net N$12: U$1.P$66
- new net N$3: LED1.A, R2.1
- new net N$7: LED4.A, R9.1
- new net UART3-RX: U$1.P$20
- new net UART3-TX: U$1.P$19, X2.1
- new net UART4-RX: U$1.P$46
- new net UART4-TX: U$1.P$45
- net PE: now also LED1.C, LED4.C, X2.4
Changed lines of the file:
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@@
 <element name="C7" library="rcl" package="E15-5" value="1uF" x="-19.05" y="-142.24"/>
 <element name="Q1" library="microbuilder" package="SOT23-WIDE" value="" x="-39.37" y="-149.86"/>
+<element name="LED1" library="led" package="CHIPLED_1206" value="" x="-45.72" y="-148.59"/>
+<element name="LED4" library="led" package="CHIPLED_1206" value="" x="-52.07" y="-148.59"/>
+<element name="R2" library="microbuilder" package="_0603" value="500" x="-58.42" y="-154.94"/>
+<element name="R9" library="microbuilder" package="_0603" value="500" x="-58.42" y="-160.02"/>
+<element name="C8" library="unicorn_v2" package="SUPERCAP" value="SUPERCAP" x="-48.26" y="-172.72"/>
+<element name="X2" library="con-panduit" package="057-006-1" value="057-006-1" x="-52.07" y="-190.5">
+<attribute name="OC_NEWARK" value="unknown" x="-52.07" y="-190.5" size="1.778" layer="27" display="off"/>
+<attribute name="MPN" value="" x="-52.07" y="-190.5" size="1.778" layer="27" display="off"/>
+<attribute name="MF" value="" x="-52.07" y="-190.5" size="1.778" layer="27" display="off"/>
+<attribute name="OC_FARNELL" value="unknown" x="-52.07" y="-190.5" size="1.778" layer="27" display="off"/>
+</element>
 </elements>
 <signals>
@@
 <contactref element="C6" pad="-"/>
 <contactref element="C7" pad="-"/>
+<contactref element="LED4" pad="C"/>
+<contactref element="LED1" pad="C"/>
+<contactref element="X2" pad="4"/>
+<wire x1="-52.07" y1="-146.84" x2="-52.07" y2="-189.23" width="0" layer="19" extent="1-1"/>
+<wire x1="-45.72" y1="-146.84" x2="-52.07" y2="-146.84" width="0" layer="19" extent="1-1"/>
+<wire x1="-11.43" y1="-142.24" x2="-45.72" y2="-146.84" width="0" layer="19" extent="1-1"/>
 <wire x1="-6.35" y1="-128.27" x2="-11.43" y2="-142.24" width="0" layer="19" extent="1-1"/>
 <wire x1="-9.652" y1="-120.65" x2="-6.35" y2="-128.27" width="0" layer="19" extent="1-1"/>
@@
 <wire x1="-5.4864" y1="-89.6112" x2="1.27" y2="-96.52" width="0" layer="19" extent="1-1"/>
 <wire x1="-8.89" y1="-89.6112" x2="-5.4864" y2="-89.6112" width="0" layer="19" extent="1-1"/>
-<wire x1="45.72" y1="8.128" x2="-5.4864" y2="-89.6112" width="0" layer="19" extent="1-1"/>
-<wire x1="35.56" y1="3.81" x2="45.72" y2="8.128" width="0" layer="19" extent="1-1"/>
-<wire x1="19.939" y1="5.461" x2="35.56" y2="3.81" width="0" layer="19" extent="1-1"/>
+<wire x1="19.939" y1="5.461" x2="-5.4864" y2="-89.6112" width="0" layer="19" extent="1-1"/>
 <wire x1="15.875" y1="18.669" x2="19.939" y2="5.461" width="0" layer="19" extent="1-1"/>
+<wire x1="35.56" y1="3.81" x2="19.939" y2="5.461" width="0" layer="19" extent="1-1"/>
+<wire x1="45.72" y1="8.128" x2="35.56" y2="3.81" width="0" layer="19" extent="1-1"/>
 <wire x1="32.893" y1="24.13" x2="15.875" y2="18.669" width="0" layer="19" extent="1-1"/>
-<wire x1="4.621" y1="41.8" x2="32.893" y2="24.13" width="0" layer="19" extent="1-1"/>
+<wire x1="4.621" y1="41.8" x2="15.875" y2="18.669" width="0" layer="19" extent="1-1"/>
 <wire x1="62.874" y1="45.381" x2="32.893" y2="24.13" width="0" layer="19" extent="1-1"/>
 <wire x1="62.874" y1="52.881" x2="62.874" y2="45.381" width="0" layer="19" extent="1-1"/>
@@
 <wire x1="34.19475" y1="-49.94275" x2="-38.42" y2="-150.86" width="0" layer="19" extent="1-1"/>
 </signal>
+<signal name="UART3-RX">
+<contactref element="U$1" pad="P$20"/>
+</signal>
+<signal name="N$3">
+<contactref element="R2" pad="1"/>
+<contactref element="LED1" pad="A"/>
+<wire x1="-45.72" y1="-150.34" x2="-59.182" y2="-154.94" width="0" layer="19" extent="1-1"/>
+</signal>
+<signal name="N$7">
+<contactref element="R9" pad="1"/>
+<contactref element="LED4" pad="A"/>
+<wire x1="-52.07" y1="-150.34" x2="-59.182" y2="-160.02" width="0" layer="19" extent="1-1"/>
+</signal>
+<signal name="DEBUG-LED2">
+<contactref element="R2" pad="2"/>
+</signal>
+<signal name="DEBUG-LED1">
+<contactref element="R9" pad="2"/>
+</signal>
+<signal name="N$11">
+<contactref element="U$1" pad="P$64"/>
+</signal>
+<signal name="N$12">
+<contactref element="U$1" pad="P$66"/>
+</signal>
+<signal name="UART3-TX">
+<contactref element="X2" pad="1"/>
+<contactref element="U$1" pad="P$19"/>
+<wire x1="59.69" y1="-58.42" x2="-54.61" y2="-191.77" width="0" layer="19" extent="1-1"/>
+</signal>
+<signal name="UART4-TX">
+<contactref element="U$1" pad="P$45"/>
+</signal>
+<signal name="UART4-RX">
+<contactref element="U$1" pad="P$46"/>
+</signal>
 </signals>

Commit message: First schematic revision for com-node done
Parts:
- added R12: 20K, microbuilder:_0603
- added R13: 1K8, microbuilder:_0603
- added U1: MAX13052ESA+, Maxim_By_element14_Batch_1:SOIC127P600X175-8N
- added X3: 22-23-2041, con-molex:22-23-2041
Connections:
- removed net 14.2V: C5.+, LM2575-ADJ.1, Q1.1
- new net +14V2: C5.+, LM2575-ADJ.1, R12.1, X3.3
- new net ECU_CAN_H: R13.1, U1.7, X3.1
- new net ECU_CAN_L: R13.2, U1.6, X3.2
- new net ECU_CAN_RX: U$1.P$23, U1.4
- new net ECU_CAN_TX: U$1.P$24, U1.1
- new net N$14: Q1.1, R12.2
- net +3V3: now also U1.3
- net PE: now also U1.2, U1.8, X3.4
Changed lines of the file:
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@@
 <attribute name="OC_FARNELL" value="unknown" x="-52.07" y="-190.5" size="1.778" layer="27" display="off"/>
+</element>
+<element name="R12" library="microbuilder" package="_0603" value="20K" x="-58.42" y="-200.66"/>
+<element name="U1" library="Maxim_By_element14_Batch_1" package="SOIC127P600X175-8N" value="MAX13052ESA+" x="-69.85" y="-195.58">
+<attribute name="PACKAGE" value="SOIC-8" x="-69.85" y="-195.58" size="1.778" layer="27" display="off"/>
+<attribute name="OC_NEWARK" value="99K2875" x="-69.85" y="-195.58" size="1.778" layer="27" display="off"/>
+<attribute name="MPN" value="MAX13052ESA+" x="-69.85" y="-195.58" size="1.778" layer="27" display="off"/>
+<attribute name="SUPPLIER" value="Maxim" x="-69.85" y="-195.58" size="1.778" layer="27" display="off"/>
+<attribute name="OC_FARNELL" value="1600112" x="-69.85" y="-195.58" size="1.778" layer="27" display="off"/>
+</element>
+<element name="R13" library="microbuilder" package="_0603" value="1K8" x="-78.74" y="-205.74"/>
+<element name="X3" library="con-molex" package="22-23-2041" value="22-23-2041" x="-74.93" y="-213.36">
+<attribute name="OC_NEWARK" value="38C0355" x="-74.93" y="-213.36" size="1.778" layer="27" display="off"/>
+<attribute name="MPN" value="22-23-2041" x="-74.93" y="-213.36" size="1.778" layer="27" display="off"/>
+<attribute name="MF" value="MOLEX" x="-74.93" y="-213.36" size="1.778" layer="27" display="off"/>
+<attribute name="OC_FARNELL" value="1462920" x="-74.93" y="-213.36" size="1.778" layer="27" display="off"/>
 </element>
 </elements>
@@
 <contactref element="LED1" pad="C"/>
 <contactref element="X2" pad="4"/>
+<contactref element="U1" pad="2"/>
+<contactref element="U1" pad="8"/>
+<contactref element="X3" pad="4"/>
+<wire x1="-67.3862" y1="-193.675" x2="-52.07" y2="-189.23" width="0" layer="19" extent="1-1"/>
+<wire x1="-72.3138" y1="-194.945" x2="-67.3862" y2="-193.675" width="0" layer="19" extent="1-1"/>
+<wire x1="-71.12" y1="-213.36" x2="-72.3138" y2="-194.945" width="0" layer="19" extent="1-1"/>
 <wire x1="-52.07" y1="-146.84" x2="-52.07" y2="-189.23" width="0" layer="19" extent="1-1"/>
 <wire x1="-45.72" y1="-146.84" x2="-52.07" y2="-146.84" width="0" layer="19" extent="1-1"/>
@@
 <contactref element="C6" pad="+"/>
 <contactref element="Q1" pad="3"/>
+<contactref element="U1" pad="3"/>
 <wire x1="-22.86" y1="-119.2" x2="-39.37" y2="-148.86" width="0" layer="19" extent="1-1"/>
 <wire x1="-8.128" y1="-115.57" x2="-22.86" y2="-119.2" width="0" layer="19" extent="1-1"/>
 <wire x1="-13.97" y1="-106.68" x2="-8.128" y2="-115.57" width="0" layer="19" extent="1-1"/>
+<wire x1="-72.3138" y1="-196.215" x2="-39.37" y2="-148.86" width="0" layer="19" extent="1-1"/>
 <wire x1="29.11475" y1="-49.94275" x2="-13.97" y2="-106.68" width="0" layer="19" extent="1-1"/>
 <wire x1="4.699" y1="5.461" x2="29.11475" y2="-49.94275" width="0" layer="19" extent="1-1"/>
@@
 <wire x1="62.874" y1="50.381" x2="32.893" y2="35.433" width="0" layer="19" extent="1-1"/>
 </signal>
-<signal name="14.2V">
+<signal name="+14V2">
 <contactref element="LM2575-ADJ" pad="1"/>
 <contactref element="C5" pad="+"/>
-<contactref element="Q1" pad="1"/>
-<wire x1="-13.97" y1="-96.52" x2="-40.32" y2="-150.86" width="0" layer="19" extent="1-1"/>
+<contactref element="R12" pad="1"/>
+<contactref element="X3" pad="3"/>
 <wire x1="-12.2936" y1="-89.6112" x2="-13.97" y2="-96.52" width="0" layer="19" extent="1-1"/>
+<wire x1="-59.182" y1="-200.66" x2="-13.97" y2="-96.52" width="0" layer="19" extent="1-1"/>
+<wire x1="-73.66" y1="-213.36" x2="-59.182" y2="-200.66" width="0" layer="19" extent="1-1"/>
 </signal>
 <signal name="N$13">
@@
 <contactref element="U$1" pad="P$46"/>
 </signal>
+<signal name="N$14">
+<contactref element="Q1" pad="1"/>
+<contactref element="R12" pad="2"/>
+<wire x1="-57.658" y1="-200.66" x2="-40.32" y2="-150.86" width="0" layer="19" extent="1-1"/>
+</signal>
+<signal name="ECU_CAN_TX">
+<contactref element="U$1" pad="P$24"/>
+<contactref element="U1" pad="1"/>
+<wire x1="54.51475" y1="-52.48275" x2="-72.3138" y2="-193.675" width="0" layer="19" extent="1-1"/>
+</signal>
+<signal name="ECU_CAN_H">
+<contactref element="U1" pad="7"/>
+<contactref element="R13" pad="1"/>
+<contactref element="X3" pad="1"/>
+<wire x1="-79.502" y1="-205.74" x2="-78.74" y2="-213.36" width="0" layer="19" extent="1-1"/>
+<wire x1="-67.3862" y1="-194.945" x2="-79.502" y2="-205.74" width="0" layer="19" extent="1-1"/>
+</signal>
+<signal name="ECU_CAN_L">
+<contactref element="U1" pad="6"/>
+<contactref element="R13" pad="2"/>
+<contactref element="X3" pad="2"/>
+<wire x1="-77.978" y1="-205.74" x2="-76.2" y2="-213.36" width="0" layer="19" extent="1-1"/>
+<wire x1="-67.3862" y1="-196.215" x2="-77.978" y2="-205.74" width="0" layer="19" extent="1-1"/>
+</signal>
+<signal name="ECU_CAN_RX">
+<contactref element="U$1" pad="P$23"/>
+<contactref element="U1" pad="4"/>
+<wire x1="54.51475" y1="-49.94275" x2="-72.3138" y2="-197.485" width="0" layer="19" extent="1-1"/>
+</signal>
 </signals>

Commit message: Update on board
Still some ERC warnings to solve
Parts:
- removed C3: 4.7uF, rcl:E15-5
- removed C4: 100nF, resistor:C050-024X044
- removed LED3: (no value), led:LED3MM
- removed R13: 1K8, microbuilder:_0603
- removed X3: 22-23-2041, con-molex:22-23-2041
- added R14: XXXXX, microbuilder:_0603
- added R15, R16: 60, microbuilder:_0603
- added X4: (no value), con-molex:22-23-2061
- C2: value 100nF -> 4n7; device resistor:C050-024X044 -> microbuilder:0603
- R7: value 500 -> 47k
- R8: value (none) -> 500
- moved R7 296.5 mm to (-78.7, -242.6), turned to 0 degrees
- moved C2 289.0 mm to (-78.7, -255.3)
- moved R3 285.8 mm to (-78.7, -227.3)
- moved R6 284.7 mm to (-78.7, -237.5)
- moved R4 281.6 mm to (-78.7, -232.4)
Connections:
- net UART3-RX renamed UART3_RX
- removed net +3.3V: C4.1
- removed net N$1 (its old number): C7.+, R1.2
- removed net N$9: LED3.K, R7.2
- removed net SD-CS: R3.2, R7.1, U$1.P$2, X1.1
- removed net SD-MISO: R5.2, U$1.P$4, X1.7
- removed net SD-MOSI: R4.2, U$1.P$5, X1.2
- removed net SD-SCK: R6.2, U$1.P$3, X1.5
- removed net UART3-TX: U$1.P$19, X2.1
- removed net UART4-RX: U$1.P$46
- removed net UART4-TX: U$1.P$45
- new net N$15: X4.2
- new net N$16: R3.1, R4.1, R5.1, R6.1, R7.1
- new net N$19: X2.3, X2.4
- new net N$21: C2.1, R15.1, R16.1, U1.5
- new net N$4: X4.1
- new net SDIO_CMD: R3.2, U$1.P$48, X1.2
- new net SDIO_D0: R4.2, U$1.P$37, X1.7
- new net SDIO_D1: R6.2, U$1.P$40, X1.8
- new net SDIO_D2: R7.2, U$1.P$45, X1.9
- new net SDIO_D3: R5.2, U$1.P$46, X1.1
- new net SDIO_SCK: U$1.P$47, X1.5
- new net SD_IN: U$1.P$49, X1.SW1
- new net UART3_TX: U$1.P$19, X2.1, X2.2
- new net USART1_RX: U$1.P$57
- new net USART1_TX: U$1.P$56
- net +14V2: now also X4.5; no longer X3.3
- net +3V3: no longer C2.1, C3.+, LED3.A, R3.1, R4.1, R5.1
- net ECU_CAN_H: now also R15.2, X4.3; no longer R13.1, X3.1
- net ECU_CAN_L: now also R16.2, X4.4; no longer R13.2, X3.2
- net N$14: now also R14.2
- net N$6: now also R8.2
- net N$8: now also X1.SW3; no longer R8.2
- net PE: now also C1.2, R14.1, X2.5, X2.6, X4.6; no longer C3.-, C4.2, R6.1, X2.4, X3.4
- net RX-XBEE: no longer XB1.2
- net SS-XBEE: now also C7.+, R1.2
