File: STM32F407 era/Com-node/Schematic.brd (EAGLE design)
At the start: 118.1 x 66 mm, 34 parts, among them U1 MAX13052ESA+, X1 SDBMF, X2 057-006-1

Commit message: Can't get the last error removed...
Parts:
- moved XB1 18.2 mm to (11.8, 33.0)
Changed lines of the file:
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@@
 <setting verticaltext="up"/>
 </settings>
-<grid distance="0.05" unitdist="inch" unit="inch" style="lines" multiple="1" display="yes" altdistance="0.005" altunitdist="inch" altunit="inch"/>
+<grid distance="1" unitdist="mm" unit="mm" style="lines" multiple="1" display="yes" altdistance="0.005" altunitdist="inch" altunit="inch"/>
 <layers>
 <layer number="1" name="Top" color="4" fill="1" visible="yes" active="yes"/>
@@
 </autorouter>
 <elements>
-<element name="XB1" library="maxstream" package="XBEE-PRO" value="XBEE-PRO" x="15.621" y="50.8"/>
+<element name="XB1" library="maxstream" package="XBEE-PRO" value="XBEE-PRO" x="11.811" y="33.02"/>
 <element name="X1" library="farnell" package="SDBMF-009XXBXX2" value="SDBMF" x="68.199" y="51.181" rot="R90"/>
 <element name="LED2" library="led" package="LED3MM" value="" x="39.243" y="57.531" rot="R270"/>
@@
 <contactref element="X1" pad="6"/>
 <polygon width="0.6096" layer="16" isolate="0.3048">
-<vertex x="76.2" y="0"/>
-<vertex x="76.2" y="66.04"/>
-<vertex x="0" y="66.04"/>
+<vertex x="160.2" y="0.25"/>
+<vertex x="160.48" y="100.04"/>
+<vertex x="-0.45" y="100.04"/>
 <vertex x="0" y="0"/>
 </polygon>
@@
 <wire x1="62.874" y1="52.881" x2="62.874" y2="45.381" width="0" layer="19" extent="1-1"/>
 <wire x1="17.018" y1="52.832" x2="62.874" y2="52.881" width="0" layer="19" extent="1-1"/>
-<wire x1="4.621" y1="41.8" x2="17.018" y2="52.832" width="0" layer="19" extent="1-1"/>
+<wire x1="0.811" y1="24.02" x2="17.018" y2="52.832" width="0" layer="19" extent="1-1"/>
 </signal>
 <signal name="N$2">
 <contactref element="XB1" pad="6"/>
 <contactref element="R1" pad="1"/>
-<wire x1="4.621" y1="49.8" x2="62.738" y2="13.97" width="0" layer="19" extent="1-1"/>
+<wire x1="0.811" y1="32.02" x2="62.738" y2="13.97" width="0" layer="19" extent="1-1"/>
 </signal>
 <signal name="RX-XBEE">
@@
 <contactref element="U$1" pad="P$75"/>
 <contactref element="XB1" pad="3"/>
-<wire x1="49.545240625" y1="-89.603578125" x2="4.621" y2="55.8" width="0" layer="19" extent="1-1"/>
+<wire x1="49.545240625" y1="-89.603578125" x2="0.811" y2="38.02" width="0" layer="19" extent="1-1"/>
 </signal>
 <signal name="+3V3">
@@
 <polygon width="1.016" layer="1" isolate="0.3048">
 <vertex x="0" y="0"/>
-<vertex x="76.2" y="0"/>
-<vertex x="76.2" y="66.04"/>
-<vertex x="0" y="66.04"/>
+<vertex x="160.2" y="0.25"/>
+<vertex x="160.48" y="100.04"/>
+<vertex x="-0.45" y="100.04"/>
 </polygon>
 <contactref element="L1" pad="2"/>
@@
 <wire x1="-72.3138" y1="-196.215" x2="-39.37" y2="-148.86" width="0" layer="19" extent="1-1"/>
 <wire x1="29.11475" y1="-49.94275" x2="-13.97" y2="-106.68" width="0" layer="19" extent="1-1"/>
-<wire x1="4.621" y1="51.8" x2="29.11475" y2="-49.94275" width="0" layer="19" extent="1-1"/>
-<wire x1="4.621" y1="59.8" x2="4.621" y2="51.8" width="0" layer="19" extent="1-1"/>
-<wire x1="17.018" y1="57.912" x2="4.621" y2="59.8" width="0" layer="19" extent="1-1"/>
+<wire x1="0.811" y1="34.02" x2="29.11475" y2="-49.94275" width="0" layer="19" extent="1-1"/>
+<wire x1="0.811" y1="42.02" x2="0.811" y2="34.02" width="0" layer="19" extent="1-1"/>
+<wire x1="17.018" y1="57.912" x2="0.811" y2="42.02" width="0" layer="19" extent="1-1"/>
 <wire x1="62.874" y1="50.381" x2="17.018" y2="57.912" width="0" layer="19" extent="1-1"/>
 </signal>
@@
 <contactref element="XB1" pad="16"/>
 <contactref element="U$1" pad="P$74"/>
-<wire x1="47.005240625" y1="-87.063578125" x2="26.621" y2="51.8" width="0" layer="19" extent="1-1"/>
+<wire x1="47.005240625" y1="-87.063578125" x2="22.811" y2="34.02" width="0" layer="19" extent="1-1"/>
 </signal>
 <signal name="CTS-XBEE">
 <contactref element="XB1" pad="12"/>
 <contactref element="U$1" pad="P$77"/>
-<wire x1="52.085240625" y1="-89.603578125" x2="26.621" y2="43.8" width="0" layer="19" extent="1-1"/>
+<wire x1="52.085240625" y1="-89.603578125" x2="22.811" y2="26.02" width="0" layer="19" extent="1-1"/>
 </signal>
 <signal name="N$5">
 <contactref element="XB1" pad="15"/>
 <contactref element="LED2" pad="A"/>
-<wire x1="26.621" y1="49.8" x2="39.243" y2="58.801" width="0" layer="19" extent="1-1"/>
+<wire x1="22.811" y1="32.02" x2="39.243" y2="58.801" width="0" layer="19" extent="1-1"/>
 </signal>
 <signal name="SS-XBEE">
@@
 <signal name="DEBUG-LED1">
 <contactref element="R9" pad="2"/>
-</signal>
-<signal name="N$12">
-<contactref element="U$1" pad="P$66"/>
 </signal>
 <signal name="SDIO_D3">
@@
 <wire x1="-67.3862" y1="-197.485" x2="-79.59" y2="-255.27" width="0" layer="19" extent="1-1"/>
 </signal>
-<signal name="N$4">
-<contactref element="X4" pad="1"/>
-</signal>
-<signal name="N$15">
-<contactref element="X4" pad="2"/>
-</signal>
-<signal name="N$1">
-<contactref element="U$1" pad="P$64"/>
-</signal>
 <signal name="N$6">
 <contactref element="R8" pad="2"/>
@@
 <contactref element="X1" pad="SW3"/>
 </signal>
+<signal name="N$1">
+<contactref element="U$1" pad="P$64"/>
+</signal>
+<signal name="N$9">
+<contactref element="U$1" pad="P$66"/>
+</signal>
+<signal name="N$4">
+<contactref element="X4" pad="1"/>
+</signal>
+<signal name="N$11">
+<contactref element="X4" pad="2"/>
+</signal>
 </signals>
