File: STM32F407 era/Display/dashboard/LCD Version/dashboard.sch (EAGLE design)
At the start: 44 parts, among them U1 CAT4238TD-GT3

Commit message: startet working on seven segment version
Parts:
- added C6, C7: 2u, microbuilder:CAP_CERAMIC_0805
- added C8: 100n, microbuilder:CAP_CERAMIC_0603
- added LED16, LED17, LED18, LED19, LED20: (no value), microbuilder:LED_RGB_PLCC6CREE-CLV6A
- added R10, R11, R12, R13, R14: 500, microbuilder:RESISTOR_0805
- added R15: 931, microbuilder:RESISTOR_0603
- added R9: 10m, microbuilder:RESISTOR_0805
- added U$42: MICROFIT6, unicorn:MICROFIT6
- added U$51: TLC59116, tlc:TLC59116
- R7, R8: value 1k -> 500
Connections:
- new net BTN1: R10.1, U$1G$2.PB12, U$42.PIN2
- new net BTN2: R14.1, U$1G$2.PB13, U$42.PIN3
- new net BTN3: R13.1, U$1G$2.PB14, U$42.PIN4
- new net BTN4: R12.1, U$1G$2.PB15, U$42.PIN5
- new net BTN5: R11.1, U$1G$2.PD8, U$42.PIN6
- new net CD: U$10.CD, U$1G$1.PC4
- new net LCD_CLOCK: U$10.D0/SCK, U$1G$1.PA5
- new net LCD_CS: U$10.CS0/A2, U$1G$1.PC5
- new net LCD_DATA: U$10.D3/SDA, U$1G$1.PA7
- new net LCD_RESET: U$10.RST, U$1G$1.PB0
- new net N$54: LED16.RGND, U$51./OUT0
- new net N$57: C6.P$1, U$10.VB1-
- new net N$58: C7.P$1, U$10.VB0-
- new net N$59: C6.P$2, U$10.VB1+
- new net N$60: C7.P$2, U$10.VB0+
- new net N$61: C8.P$2, R9.2, U$10.VLCD
- new net N$62: LED16.GGND, U$51./OUT1
- new net N$63: LED16.BGND, U$51./OUT2
- new net N$64: LED17.RGND, U$51./OUT3
- new net N$65: LED17.GGND, U$51./OUT4
- new net N$66: LED17.BGND, U$51./OUT5
- new net N$67: LED18.RGND, U$51./OUT6
- new net N$68: LED18.GGND, U$51./OUT7
- new net N$69: LED18.BGND, U$51./OUT8
- new net N$70: LED19.RGND, U$51./OUT9
- new net N$71: LED19.GGND, U$51./OUT10
- new net N$72: LED19.BGND, U$51./OUT11
- new net N$73: LED20.RGND, U$51./OUT12
- new net N$74: LED20.GGND, U$51./OUT13
- new net N$75: LED20.BGND, U$51./OUT14
- new net N$76: R15.1, U$51.REXT
- net 3.3V: now also LED16.BLUE, LED16.GRN, LED16.RED, LED17.BLUE, LED17.GRN, LED17.RED, LED18.BLUE, LED18.GRN, LED18.RED, LED19.BLUE, LED19.GRN, LED19.RED, LED20.BLUE, LED20.GRN, LED20.RED, R10.2, R11.2, R12.2, R13.2, R14.2, U$10.D6, U$51.A0, U$51.A1, U$51.VCC
- net GND: now also C8.P$1, R15.2, R9.1, U$10.BM0, U$42.PIN1, U$51.A2, U$51.A3, U$51.GND@10, U$51.GND@19, U$51.GND@24
- net SCL: now also U$51.SCL
- net SDA: now also U$51.SDA
- net ~RESET: now also U$51./RESET
Other:
- moved on the sheet: C1, C2, C3, D1, L1, LED1, LED11, LED12, LED13, LED14, LED15, LED2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

Commit message: added dashboard control buttons
added buttons to add functionality to the LCD panel
Parts:
- added R16, R17, R18, R19: 500, microbuilder:RESISTOR_0805
- added S1, S2, S3, S4: (no value), switch-omron:10-XX
Connections:
- new net SW1: R16.1, S1.P, S1.P1, U$1G$1.PE8
- new net SW2: R17.1, S2.P, S2.P1, U$1G$1.PE10
- new net SW3: R18.1, S3.P, S3.P1, U$1G$1.PE12
- new net SW4: R19.1, S4.P, S4.P1, U$1G$1.PE14
- net 3.3V: now also R16.2, R17.2, R18.2, R19.2
- net GND: now also S1.S, S1.S1, S2.S, S2.S1, S3.S, S3.S1, S4.S, S4.S1
Changed lines of the file:
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@@
 <part name="R15" library="microbuilder" deviceset="RESISTOR" device="_0603" value="931"/>
 <part name="U$52" library="microbuilder" deviceset="3.3V" device=""/>
+<part name="S1" library="switch-omron" deviceset="10-XX" device=""/>
+<part name="S2" library="switch-omron" deviceset="10-XX" device=""/>
+<part name="S3" library="switch-omron" deviceset="10-XX" device=""/>
+<part name="S4" library="switch-omron" deviceset="10-XX" device=""/>
+<part name="U$53" library="microbuilder" deviceset="GND" device=""/>
+<part name="R16" library="microbuilder" deviceset="RESISTOR" device="_0805" value="500"/>
+<part name="R17" library="microbuilder" deviceset="RESISTOR" device="_0805" value="500"/>
+<part name="R18" library="microbuilder" deviceset="RESISTOR" device="_0805" value="500"/>
+<part name="R19" library="microbuilder" deviceset="RESISTOR" device="_0805" value="500"/>
+<part name="U$54" library="microbuilder" deviceset="3.3V" device=""/>
 </parts>
 <sheets>
@@
 <instance part="R15" gate="G$1" x="269.24" y="-142.24" rot="R270"/>
 <instance part="U$52" gate="G$1" x="355.6" y="-76.2"/>
+<instance part="S1" gate="1" x="-76.2" y="-38.1" rot="R270"/>
+<instance part="S2" gate="1" x="-76.2" y="-50.8" rot="R270"/>
+<instance part="S3" gate="1" x="-76.2" y="-63.5" rot="R270"/>
+<instance part="S4" gate="1" x="-76.2" y="-76.2" rot="R270"/>
+<instance part="U$53" gate="G$1" x="-68.58" y="-83.82"/>
+<instance part="R16" gate="G$1" x="-91.44" y="-33.02" rot="R180"/>
+<instance part="R17" gate="G$1" x="-91.44" y="-45.72" rot="R180"/>
+<instance part="R18" gate="G$1" x="-91.44" y="-58.42" rot="R180"/>
+<instance part="R19" gate="G$1" x="-91.44" y="-71.12" rot="R180"/>
+<instance part="U$54" gate="G$1" x="-99.06" y="-27.94"/>
 </instances>
 <busses>
@@
 <wire x1="274.32" y1="-149.86" x2="269.24" y2="-149.86" width="0.1524" layer="91"/>
 <wire x1="269.24" y1="-149.86" x2="269.24" y2="-147.32" width="0.1524" layer="91"/>
+</segment>
+<segment>
+<pinref part="S4" gate="1" pin="S1"/>
+<pinref part="U$53" gate="G$1" pin="GND"/>
+<wire x1="-71.12" y1="-78.74" x2="-68.58" y2="-78.74" width="0.1524" layer="91"/>
+<wire x1="-68.58" y1="-78.74" x2="-68.58" y2="-81.28" width="0.1524" layer="91"/>
+<pinref part="S4" gate="1" pin="S"/>
+<wire x1="-71.12" y1="-76.2" x2="-68.58" y2="-76.2" width="0.1524" layer="91"/>
+<wire x1="-68.58" y1="-76.2" x2="-68.58" y2="-78.74" width="0.1524" layer="91"/>
+<junction x="-68.58" y="-78.74"/>
+<pinref part="S3" gate="1" pin="S1"/>
+<wire x1="-71.12" y1="-66.04" x2="-68.58" y2="-66.04" width="0.1524" layer="91"/>
+<wire x1="-68.58" y1="-66.04" x2="-68.58" y2="-76.2" width="0.1524" layer="91"/>
+<junction x="-68.58" y="-76.2"/>
+<pinref part="S3" gate="1" pin="S"/>
+<wire x1="-71.12" y1="-63.5" x2="-68.58" y2="-63.5" width="0.1524" layer="91"/>
+<wire x1="-68.58" y1="-63.5" x2="-68.58" y2="-66.04" width="0.1524" layer="91"/>
+<junction x="-68.58" y="-66.04"/>
+<pinref part="S2" gate="1" pin="S1"/>
+<wire x1="-71.12" y1="-53.34" x2="-68.58" y2="-53.34" width="0.1524" layer="91"/>
+<wire x1="-68.58" y1="-53.34" x2="-68.58" y2="-63.5" width="0.1524" layer="91"/>
+<junction x="-68.58" y="-63.5"/>
+<pinref part="S2" gate="1" pin="S"/>
+<wire x1="-71.12" y1="-50.8" x2="-68.58" y2="-50.8" width="0.1524" layer="91"/>
+<wire x1="-68.58" y1="-50.8" x2="-68.58" y2="-53.34" width="0.1524" layer="91"/>
+<junction x="-68.58" y="-53.34"/>
+<pinref part="S1" gate="1" pin="S1"/>
+<wire x1="-71.12" y1="-40.64" x2="-68.58" y2="-40.64" width="0.1524" layer="91"/>
+<wire x1="-68.58" y1="-40.64" x2="-68.58" y2="-50.8" width="0.1524" layer="91"/>
+<junction x="-68.58" y="-50.8"/>
+<pinref part="S1" gate="1" pin="S"/>
+<wire x1="-71.12" y1="-38.1" x2="-68.58" y2="-38.1" width="0.1524" layer="91"/>
+<wire x1="-68.58" y1="-38.1" x2="-68.58" y2="-40.64" width="0.1524" layer="91"/>
+<junction x="-68.58" y="-40.64"/>
 </segment>
 </net>
@@
 <pinref part="LED20" gate="G$1" pin="BLUE"/>
 </segment>
+<segment>
+<pinref part="R19" gate="G$1" pin="2"/>
+<pinref part="U$54" gate="G$1" pin="3.3V"/>
+<wire x1="-96.52" y1="-71.12" x2="-99.06" y2="-71.12" width="0.1524" layer="91"/>
+<wire x1="-99.06" y1="-71.12" x2="-99.06" y2="-58.42" width="0.1524" layer="91"/>
+<pinref part="R18" gate="G$1" pin="2"/>
+<wire x1="-99.06" y1="-58.42" x2="-99.06" y2="-45.72" width="0.1524" layer="91"/>
+<wire x1="-99.06" y1="-45.72" x2="-99.06" y2="-33.02" width="0.1524" layer="91"/>
+<wire x1="-99.06" y1="-33.02" x2="-99.06" y2="-30.48" width="0.1524" layer="91"/>
+<wire x1="-96.52" y1="-58.42" x2="-99.06" y2="-58.42" width="0.1524" layer="91"/>
+<junction x="-99.06" y="-58.42"/>
+<pinref part="R17" gate="G$1" pin="2"/>
+<wire x1="-96.52" y1="-45.72" x2="-99.06" y2="-45.72" width="0.1524" layer="91"/>
+<junction x="-99.06" y="-45.72"/>
+<pinref part="R16" gate="G$1" pin="2"/>
+<wire x1="-96.52" y1="-33.02" x2="-99.06" y2="-33.02" width="0.1524" layer="91"/>
+<junction x="-99.06" y="-33.02"/>
+</segment>
 </net>
 <net name="N$9" class="0">
@@
 </segment>
 </net>
+<net name="SW1" class="0">
+<segment>
+<pinref part="S1" gate="1" pin="P1"/>
+<wire x1="-81.28" y1="-40.64" x2="-83.82" y2="-40.64" width="0.1524" layer="91"/>
+<wire x1="-83.82" y1="-40.64" x2="-83.82" y2="-38.1" width="0.1524" layer="91"/>
+<wire x1="-83.82" y1="-38.1" x2="-86.36" y2="-38.1" width="0.1524" layer="91"/>
+<pinref part="S1" gate="1" pin="P"/>
+<wire x1="-81.28" y1="-38.1" x2="-83.82" y2="-38.1" width="0.1524" layer="91"/>
+<junction x="-83.82" y="-38.1"/>
+<label x="-86.36" y="-38.1" size="1.27" layer="95" rot="R180" xref="yes"/>
+<pinref part="R16" gate="G$1" pin="1"/>
+<wire x1="-86.36" y1="-33.02" x2="-83.82" y2="-33.02" width="0.1524" layer="91"/>
+<wire x1="-83.82" y1="-33.02" x2="-83.82" y2="-38.1" width="0.1524" layer="91"/>
+</segment>
+<segment>
+<pinref part="U$1" gate="G$1" pin="PE8"/>
+<wire x1="-63.5" y1="50.8" x2="-60.96" y2="50.8" width="0.1524" layer="91"/>
+<label x="-63.5" y="50.8" size="1.27" layer="95" rot="R180" xref="yes"/>
+</segment>
+</net>
+<net name="SW2" class="0">
+<segment>
+<pinref part="S2" gate="1" pin="P"/>
+<wire x1="-81.28" y1="-50.8" x2="-83.82" y2="-50.8" width="0.1524" layer="91"/>
+<pinref part="S2" gate="1" pin="P1"/>
+<wire x1="-83.82" y1="-50.8" x2="-86.36" y2="-50.8" width="0.1524" layer="91"/>
+<wire x1="-81.28" y1="-53.34" x2="-83.82" y2="-53.34" width="0.1524" layer="91"/>
+<wire x1="-83.82" y1="-53.34" x2="-83.82" y2="-50.8" width="0.1524" layer="91"/>
+<junction x="-83.82" y="-50.8"/>
+<label x="-86.36" y="-50.8" size="1.27" layer="95" rot="R180" xref="yes"/>
+<pinref part="R17" gate="G$1" pin="1"/>
+<wire x1="-86.36" y1="-45.72" x2="-83.82" y2="-45.72" width="0.1524" layer="91"/>
+<wire x1="-83.82" y1="-45.72" x2="-83.82" y2="-50.8" width="0.1524" layer="91"/>
+</segment>
+<segment>
+<pinref part="U$1" gate="G$1" pin="PE10"/>
+<wire x1="-63.5" y1="48.26" x2="-60.96" y2="48.26" width="0.1524" layer="91"/>
+<label x="-63.5" y="48.26" size="1.27" layer="95" rot="R180" xref="yes"/>
+</segment>
+</net>
+<net name="SW3" class="0">
+<segment>
+<pinref part="S3" gate="1" pin="P"/>
+<wire x1="-81.28" y1="-63.5" x2="-83.82" y2="-63.5" width="0.1524" layer="91"/>
+<pinref part="S3" gate="1" pin="P1"/>
+<wire x1="-83.82" y1="-63.5" x2="-86.36" y2="-63.5" width="0.1524" layer="91"/>
+<wire x1="-81.28" y1="-66.04" x2="-83.82" y2="-66.04" width="0.1524" layer="91"/>
+<wire x1="-83.82" y1="-66.04" x2="-83.82" y2="-63.5" width="0.1524" layer="91"/>
+<junction x="-83.82" y="-63.5"/>
+<label x="-86.36" y="-63.5" size="1.27" layer="95" rot="R180" xref="yes"/>
+<pinref part="R18" gate="G$1" pin="1"/>
+<wire x1="-86.36" y1="-58.42" x2="-83.82" y2="-58.42" width="0.1524" layer="91"/>
+<wire x1="-83.82" y1="-58.42" x2="-83.82" y2="-63.5" width="0.1524" layer="91"/>
+</segment>
+<segment>
+<pinref part="U$1" gate="G$1" pin="PE12"/>
+<wire x1="-63.5" y1="45.72" x2="-60.96" y2="45.72" width="0.1524" layer="91"/>
+<label x="-63.5" y="45.72" size="1.27" layer="95" rot="R180" xref="yes"/>
+</segment>
+</net>
+<net name="SW4" class="0">
+<segment>
+<pinref part="S4" gate="1" pin="P"/>
+<wire x1="-81.28" y1="-76.2" x2="-83.82" y2="-76.2" width="0.1524" layer="91"/>
+<pinref part="S4" gate="1" pin="P1"/>
+<wire x1="-81.28" y1="-78.74" x2="-83.82" y2="-78.74" width="0.1524" layer="91"/>
+<wire x1="-83.82" y1="-78.74" x2="-83.82" y2="-76.2" width="0.1524" layer="91"/>
+<wire x1="-83.82" y1="-76.2" x2="-86.36" y2="-76.2" width="0.1524" layer="91"/>
+<junction x="-83.82" y="-76.2"/>
+<label x="-86.36" y="-76.2" size="1.27" layer="95" rot="R180" xref="yes"/>
+<pinref part="R19" gate="G$1" pin="1"/>
+<wire x1="-86.36" y1="-71.12" x2="-83.82" y2="-71.12" width="0.1524" layer="91"/>
+<wire x1="-83.82" y1="-71.12" x2="-83.82" y2="-76.2" width="0.1524" layer="91"/>
+</segment>
+<segment>
+<pinref part="U$1" gate="G$1" pin="PE14"/>
+<wire x1="-63.5" y1="43.18" x2="-60.96" y2="43.18" width="0.1524" layer="91"/>
+<label x="-63.5" y="43.18" size="1.27" layer="95" rot="R180" xref="yes"/>
+</segment>
+</net>

Commit message: added hardware debounce circuit to buttons
Parts:
- added C10, C11, C12, C13, C14, C15, C16, C17, C18, C19, C20, C21, C22, C23, C24, C9: 100n, microbuilder:CAP_CERAMIC_0603
- added IC2, IC3: 74HC14D, 74xx-eu:74HC14D
- added R20: 500, microbuilder:RESISTOR_0603
- added S5: (no value), switch-omron:10-XX
- R10, R11, R12, R13, R14, R16, R17, R18, R19: device microbuilder:RESISTOR_0805 -> microbuilder:RESISTOR_0603
Connections:
- new net BTN1S: IC2D.O, U$1G$2.PB12
- new net BTN2S: IC2E.O, U$1G$2.PB13
- new net BTN3S: IC2B.O, U$1G$2.PB14
- new net BTN4S: IC2A.O, U$1G$2.PB15
- new net BTN5S: IC2C.O, U$1G$2.PD9
- new net SW1S: IC3D.O, U$1G$1.PE12
- new net SW2S: IC3E.O, U$1G$1.PE14
- new net SW3S: IC3B.O, U$1G$1.PE8
- new net SW4S: IC3A.O, U$1G$1.PE10
- new net SW5: C21.P$2, IC3C.I, R20.1, S5.P, S5.P1
- new net SW5S: IC3C.O, U$1G$1.PB1
- net 3.3V: now also C14.P$1, C15.P$1, C16.P$1, C17.P$1, C18.P$1, C24.P$1, IC2P.VCC, IC3P.VCC, R20.2
- net BTN1: now also C12.P$2, IC2D.I, R13.1, U$42.PIN4; no longer R10.1, U$1G$2.PB12, U$42.PIN2
- net BTN2: now also C13.P$2, IC2E.I, R10.1, U$42.PIN2; no longer R14.1, U$1G$2.PB13, U$42.PIN3
- net BTN3: now also C10.P$2, IC2B.I, R11.1, U$42.PIN6; no longer R13.1, U$1G$2.PB14, U$42.PIN4
- net BTN4: now also C9.P$2, IC2A.I, R14.1, U$42.PIN3; no longer R12.1, U$1G$2.PB15, U$42.PIN5
- net BTN5: now also C11.P$2, IC2C.I, R12.1, U$42.PIN5; no longer R11.1, U$1G$2.PD8, U$42.PIN6
- net GND: now also C10.P$1, C11.P$1, C12.P$1, C13.P$1, C14.P$2, C15.P$2, C16.P$2, C17.P$2, C18.P$2, C19.P$1, C20.P$1, C21.P$1, C22.P$1, C23.P$1, C24.P$2, C9.P$1, IC2F.I, IC2P.GND, IC3F.I, IC3P.GND, S5.S, S5.S1
- net SW1: now also C22.P$2, IC3D.I; no longer U$1G$1.PE8
- net SW2: now also C23.P$2, IC3E.I; no longer U$1G$1.PE10
- net SW3: now also C20.P$2, IC3B.I; no longer U$1G$1.PE12
- net SW4: now also C19.P$2, IC3A.I; no longer U$1G$1.PE14
Other:
- moved on the sheet: R10, R11, R12, R13, R14, R16, R17, R18, R19, S1, S2, S3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
