File: STM32F407 era/Traction control modul/TC board.sch (EAGLE design)
At the start: 49 parts, among them IC1 74HC14D, IC2 lm2575, IC3 74AC08D, IC4 74AC04D, J1 CON1, U1 MAX13052ESA+, U2 MAX232AEWE+, X1 057-006-1

Commit message: fixed CPU board in library
Connections:
- net FUEL1 renamed FUEL-RECIEVE
- net FUEL3 renamed FUEL-SEND
- removed net FUEL2: J1G$3.K
- removed net FUEL4: J1G$4.K
- net 12V: now also J1G$4.K
- net GND: now also J1G$3.K
Changed lines of the file:
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@@
 <pinref part="J1" gate="G$3" pin="B"/>
 <wire x1="401.32" y1="22.86" x2="401.32" y2="20.32" width="0.1524" layer="91"/>
-<wire x1="401.32" y1="20.32" x2="401.32" y2="5.08" width="0.1524" layer="91"/>
+<wire x1="401.32" y1="20.32" x2="401.32" y2="12.7" width="0.1524" layer="91"/>
+<wire x1="401.32" y1="12.7" x2="401.32" y2="5.08" width="0.1524" layer="91"/>
 <wire x1="398.78" y1="33.02" x2="401.32" y2="33.02" width="0.1524" layer="91"/>
 <pinref part="J1" gate="G$3" pin="F"/>
@@
 <wire x1="398.78" y1="20.32" x2="401.32" y2="20.32" width="0.1524" layer="91"/>
 <junction x="401.32" y="20.32"/>
+<pinref part="J1" gate="G$3" pin="K"/>
+<wire x1="398.78" y1="12.7" x2="401.32" y2="12.7" width="0.1524" layer="91"/>
+<junction x="401.32" y="12.7"/>
 </segment>
 <segment>
@@
 <segment>
 <pinref part="U$13" gate="G$1" pin="12V"/>
-<wire x1="439.42" y1="7.62" x2="439.42" y2="22.86" width="0.1524" layer="91"/>
+<wire x1="439.42" y1="7.62" x2="439.42" y2="12.7" width="0.1524" layer="91"/>
 <pinref part="J1" gate="G$4" pin="M"/>
+<wire x1="439.42" y1="12.7" x2="439.42" y2="22.86" width="0.1524" layer="91"/>
 <wire x1="439.42" y1="22.86" x2="439.42" y2="38.1" width="0.1524" layer="91"/>
 <wire x1="431.8" y1="7.62" x2="439.42" y2="7.62" width="0.1524" layer="91"/>
@@
 <wire x1="431.8" y1="22.86" x2="439.42" y2="22.86" width="0.1524" layer="91"/>
 <junction x="439.42" y="22.86"/>
+<pinref part="J1" gate="G$4" pin="K"/>
+<wire x1="431.8" y1="12.7" x2="439.42" y2="12.7" width="0.1524" layer="91"/>
+<junction x="439.42" y="12.7"/>
 </segment>
 <segment>
@@
 </segment>
 </net>
-<net name="FUEL1" class="0">
+<net name="FUEL-RECIEVE" class="0">
 <segment>
 <pinref part="J1" gate="G$3" pin="J"/>
@@
 </segment>
 </net>
-<net name="FUEL2" class="0">
-<segment>
-<pinref part="J1" gate="G$3" pin="K"/>
-<wire x1="403.86" y1="12.7" x2="398.78" y2="12.7" width="0.1524" layer="91"/>
-<label x="403.86" y="12.7" size="1.27" layer="95" xref="yes"/>
-</segment>
-</net>
-<net name="FUEL3" class="0">
+<net name="FUEL-SEND" class="0">
 <segment>
 <pinref part="J1" gate="G$4" pin="J"/>
@@
 </segment>
 </net>
-<net name="FUEL4" class="0">
-<segment>
-<pinref part="J1" gate="G$4" pin="K"/>
-<wire x1="441.96" y1="12.7" x2="431.8" y2="12.7" width="0.1524" layer="91"/>
-<label x="441.96" y="12.7" size="1.27" layer="95" xref="yes"/>
-</segment>
-</net>

Commit message: added CAN bus connections to TC board
Parts:
- added Q4: (no value), microbuilder:TRANSISTOR_NPNWIDE
- added R18: 500, microbuilder:RESISTOR_0603
- added R19: 100k, microbuilder:RESISTOR_0603
- added R20: 178, microbuilder:RESISTOR_0603
- added R21: 604, microbuilder:RESISTOR_0603
Connections:
- new net FUEL-RECIEVEI: R20.2, R21.1, U$1G$4.PC2
- new net FUEL-SENDO: Q4.E, R19.1
- new net N$25: J1G$4.J, R19.2
- new net N$26: Q4.B, R18.1
- net 12V: now also Q4.C
- net 3.3V: no longer J1G$2.D, J1G$3.D
- net CANH: now also J1G$3.D
- net CANL: now also J1G$2.D
- net FUEL-RECIEVE: now also R21.2
- net FUEL-SEND: now also R18.2, U$1G$4.PC1; no longer J1G$4.J
- net GND: now also R20.1
Other:
- note added: "Fuel 12V signal send"

Commit message: finished adding gear feedback circuit
Parts:
- added C13, C14: 100n, microbuilder:CAP_CERAMIC_0603
- added C16: 10u, microbuilder:CAP_CERAMIC_0805
- added C17: 22u, microbuilder:CAP_CERAMIC_0805
- added C18: 33uf pan FC, rcl:CPOL-EUUD-5X5,8
- added IC5: REG1117, burr-brown:REG1117
- added OK1: 4N37, optocoupler:4N37
- added Q5: (no value), microbuilder:TRANSISTOR_NPNWIDE
- added R22, R23: 200, microbuilder:RESISTOR_0603
- added U3: MAX531AESD+, Maxim_By_element14_Batch_1:MAX531AESD+
Connections:
- new net 5.0V: C14.P$1, C17.P$2, IC5.VOUT, U3.VDD
- new net DACCLR: U3.~CLR
- new net DACCS: U3.~CS
- new net DIRASENSE: IC3C.I0, J1G$2.L, U$1G$2.PD12
- new net DIRBSENSE: IC3C.I1, J1G$2.K, U$1G$2.PD14
- new net MISO: U$1G$2.PB14, U3.DOUT
- new net MOSI: U$1G$2.PB15, U3.DIN
- new net N$27: C13.P$2, C14.P$2, U3.AGND, U3.DGND
- new net N$28: C13.P$1, U3.VSS
- new net N$29: OK1.A, R22.1
- new net N$30: IC3C.O, R22.2
- new net N$31: OK1.EMI, R23.2
- new net N$32: Q1.C, Q2.C, Q5.E
- new net N$33: Q5.B, R23.1
- new net REF: C18.+, U3.REFIN, U3.REFOUT
- new net SCK: U$1G$2.PB13, U3.SCLK
- new net VOUT: J1G$2.M, U3.BIPOFF, U3.RFB, U3.VOUT
- net 12V: now also C16.P$2, IC5.VIN, OK1.COL, Q5.C; no longer Q1.C, Q2.C
- net GND: now also C16.P$1, C17.P$1, C18.-, IC5.GND, OK1.C; no longer IC3C.I0, IC3C.I1
Other:
- moved on the sheet: IC3C, Q1, Q2, Q3, Q4, R17, R18, R4, R5, R6, R9
