File: Laptimer/Mixed/Laptimer.sch (EAGLE design)
At the start: 78 parts, among them IC1 MCP73831/OT, IC2 REG1117, IC3 MAX631CPA, IC4 74HC04D, IC5 NE555D, IC6 74HC08D, Q1 8mhz, Q4 PBSS4120T, X1 mini-usb, X2 GLX-S-88M

Commit message: Added RPM leds and constant current IC's
Connections:
- net N$1 renamed 1D+
- net N$27 renamed 1D-
Changed lines of the file:
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@@
 </segment>
 </net>
-<net name="N$1" class="0">
+<net name="1D+" class="0">
 <segment>
 <pinref part="X1" gate="G$1" pin="3"/>
@@
 </segment>
 </net>
-<net name="N$27" class="0">
+<net name="1D-" class="0">
 <segment>
 <pinref part="R8" gate="G$1" pin="2"/>

Commit message: more final board prepping for production
Parts:
- removed JP2: (no value), microbuilder:HEADER-1X2ROUND
- removed JP3: (no value), adafruit:PINHD-1X3
- removed LED1, LED2, LED3, LED4, LED5, LED6, LED7, LED8, LED9: SFH 309, adafruit:LED3MM
Connections:
- removed net INT: JP3.2, LED1.C, LED2.C, LED3.C, LED4.C, LED5.C, LED6.C, LED7.C, LED8.C, LED9.C
- removed net N$10: JP2.1, JP3.1
- removed net N$40: JP2.2, JP3.3, LED1.A, LED2.A, LED3.A, LED4.A, LED5.A, LED6.A, LED7.A, LED8.A, LED9.A
Changed lines of the file:
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@@
 <part name="GND6" library="supply1" deviceset="GND" device=""/>
 <part name="U$4" library="adafruit" deviceset="AVRISP" device="-BOX"/>
-<part name="LED1" library="adafruit" deviceset="LED" device="3MM" value="SFH 309"/>
-<part name="LED2" library="adafruit" deviceset="LED" device="3MM" value="SFH 309"/>
-<part name="LED3" library="adafruit" deviceset="LED" device="3MM" value="SFH 309"/>
-<part name="LED4" library="adafruit" deviceset="LED" device="3MM" value="SFH 309"/>
-<part name="LED5" library="adafruit" deviceset="LED" device="3MM" value="SFH 309"/>
-<part name="LED6" library="adafruit" deviceset="LED" device="3MM" value="SFH 309"/>
-<part name="LED7" library="adafruit" deviceset="LED" device="3MM" value="SFH 309"/>
-<part name="LED8" library="adafruit" deviceset="LED" device="3MM" value="SFH 309"/>
 <part name="IC5" library="linear" deviceset="*555" device="D" technology="NE"/>
 <part name="R18" library="rcl" deviceset="R-EU_" device="R0603" value="1k"/>
@@
 <part name="R7" library="rcl" deviceset="R-EU_" device="R0603" value="220"/>
 <part name="GND8" library="supply1" deviceset="GND" device=""/>
-<part name="LED9" library="adafruit" deviceset="LED" device="3MM" value="SFH 309"/>
-<part name="JP3" library="adafruit" deviceset="PINHD-1X3" device=""/>
-<part name="JP2" library="microbuilder" deviceset="HEADER-1X2" device="ROUND"/>
 <part name="JP1" library="adafruit" deviceset="PINHD-1X3" device=""/>
 <part name="BAT1" library="SparkFun-Electromechanical" deviceset="BATTERY" device="18650"/>
@@
 <instance part="GND6" gate="1" x="137.16" y="53.34"/>
 <instance part="U$4" gate="G$1" x="121.92" y="60.96"/>
-<instance part="LED1" gate="G$1" x="175.26" y="134.62" rot="R90"/>
-<instance part="LED2" gate="G$1" x="175.26" y="127" rot="R90"/>
-<instance part="LED3" gate="G$1" x="175.26" y="119.38" rot="R90"/>
-<instance part="LED4" gate="G$1" x="175.26" y="111.76" rot="R90"/>
-<instance part="LED5" gate="G$1" x="175.26" y="104.14" rot="R90"/>
-<instance part="LED6" gate="G$1" x="175.26" y="96.52" rot="R90"/>
-<instance part="LED7" gate="G$1" x="175.26" y="88.9" rot="R90"/>
-<instance part="LED8" gate="G$1" x="175.26" y="81.28" rot="R90"/>
 <instance part="IC5" gate="A" x="170.18" y="193.04"/>
 <instance part="R18" gate="G$1" x="182.88" y="208.28" rot="R270"/>
@@
 <instance part="R7" gate="G$1" x="25.4" y="213.36"/>
 <instance part="GND8" gate="1" x="43.18" y="208.28"/>
-<instance part="LED9" gate="G$1" x="175.26" y="73.66" rot="R90"/>
-<instance part="JP3" gate="A" x="162.56" y="139.7" rot="MR0"/>
-<instance part="JP2" gate="G$1" x="187.96" y="142.24"/>
 <instance part="JP1" gate="A" x="93.98" y="213.36"/>
 <instance part="BAT1" gate="G$1" x="88.9" y="15.24" rot="R270"/>
@@
 </segment>
 </net>
-<net name="INT" class="0">
-<segment>
-<pinref part="LED1" gate="G$1" pin="C"/>
-<pinref part="LED2" gate="G$1" pin="C"/>
-<wire x1="180.34" y1="134.62" x2="180.34" y2="127" width="0.1524" layer="91"/>
-<pinref part="LED3" gate="G$1" pin="C"/>
-<wire x1="180.34" y1="127" x2="180.34" y2="119.38" width="0.1524" layer="91"/>
-<junction x="180.34" y="127"/>
-<pinref part="LED4" gate="G$1" pin="C"/>
-<wire x1="180.34" y1="119.38" x2="180.34" y2="111.76" width="0.1524" layer="91"/>
-<junction x="180.34" y="119.38"/>
-<pinref part="LED5" gate="G$1" pin="C"/>
-<wire x1="180.34" y1="111.76" x2="180.34" y2="104.14" width="0.1524" layer="91"/>
-<junction x="180.34" y="111.76"/>
-<pinref part="LED6" gate="G$1" pin="C"/>
-<wire x1="180.34" y1="104.14" x2="180.34" y2="96.52" width="0.1524" layer="91"/>
-<junction x="180.34" y="104.14"/>
-<pinref part="LED7" gate="G$1" pin="C"/>
-<wire x1="180.34" y1="96.52" x2="180.34" y2="88.9" width="0.1524" layer="91"/>
-<junction x="180.34" y="96.52"/>
-<pinref part="LED8" gate="G$1" pin="C"/>
-<wire x1="180.34" y1="88.9" x2="180.34" y2="81.28" width="0.1524" layer="91"/>
-<junction x="180.34" y="88.9"/>
-<wire x1="165.1" y1="139.7" x2="180.34" y2="139.7" width="0.1524" layer="91"/>
-<wire x1="180.34" y1="139.7" x2="180.34" y2="134.62" width="0.1524" layer="91"/>
-<junction x="180.34" y="134.62"/>
-<pinref part="LED9" gate="G$1" pin="C"/>
-<wire x1="180.34" y1="81.28" x2="180.34" y2="73.66" width="0.1524" layer="91"/>
-<junction x="180.34" y="81.28"/>
-<pinref part="JP3" gate="A" pin="2"/>
-</segment>
-</net>
-<net name="N$10" class="0">
-<segment>
-<wire x1="165.1" y1="142.24" x2="170.18" y2="142.24" width="0.1524" layer="91"/>
-<pinref part="JP3" gate="A" pin="1"/>
-<pinref part="JP2" gate="G$1" pin="1"/>
-<wire x1="185.42" y1="144.78" x2="170.18" y2="144.78" width="0.1524" layer="91"/>
-<wire x1="170.18" y1="144.78" x2="170.18" y2="142.24" width="0.1524" layer="91"/>
-</segment>
-</net>
 <net name="PT-OUT" class="0">
 <segment>
@@
 </segment>
 </net>
-<net name="N$40" class="0">
-<segment>
-<pinref part="LED6" gate="G$1" pin="A"/>
-<pinref part="LED5" gate="G$1" pin="A"/>
-<wire x1="172.72" y1="96.52" x2="172.72" y2="104.14" width="0.1524" layer="91"/>
-<pinref part="LED4" gate="G$1" pin="A"/>
-<wire x1="172.72" y1="104.14" x2="172.72" y2="111.76" width="0.1524" layer="91"/>
-<junction x="172.72" y="104.14"/>
-<pinref part="LED3" gate="G$1" pin="A"/>
-<wire x1="172.72" y1="111.76" x2="172.72" y2="119.38" width="0.1524" layer="91"/>
-<junction x="172.72" y="111.76"/>
-<pinref part="LED2" gate="G$1" pin="A"/>
-<wire x1="172.72" y1="119.38" x2="172.72" y2="127" width="0.1524" layer="91"/>
-<junction x="172.72" y="119.38"/>
-<pinref part="LED1" gate="G$1" pin="A"/>
-<wire x1="172.72" y1="127" x2="172.72" y2="134.62" width="0.1524" layer="91"/>
-<junction x="172.72" y="127"/>
-<pinref part="LED7" gate="G$1" pin="A"/>
-<wire x1="172.72" y1="96.52" x2="172.72" y2="88.9" width="0.1524" layer="91"/>
-<junction x="172.72" y="96.52"/>
-<pinref part="LED8" gate="G$1" pin="A"/>
-<wire x1="172.72" y1="88.9" x2="172.72" y2="81.28" width="0.1524" layer="91"/>
-<junction x="172.72" y="88.9"/>
-<wire x1="165.1" y1="137.16" x2="172.72" y2="137.16" width="0.1524" layer="91"/>
-<wire x1="172.72" y1="137.16" x2="172.72" y2="134.62" width="0.1524" layer="91"/>
-<junction x="172.72" y="134.62"/>
-<junction x="172.72" y="137.16"/>
-<wire x1="172.72" y1="137.16" x2="172.72" y2="142.24" width="0.1524" layer="91"/>
-<pinref part="LED9" gate="G$1" pin="A"/>
-<wire x1="172.72" y1="81.28" x2="172.72" y2="73.66" width="0.1524" layer="91"/>
-<junction x="172.72" y="81.28"/>
-<pinref part="JP3" gate="A" pin="3"/>
-<pinref part="JP2" gate="G$1" pin="2"/>
-<wire x1="172.72" y1="142.24" x2="185.42" y2="142.24" width="0.1524" layer="91"/>
-</segment>
-</net>
