File: Laptimer/Mixed/remote unit/Laptimer.brd (EAGLE design)
At the start: 100 x 75 mm, 24 parts, among them IC4 74HC04D, IC5 NE555D, X2 GLX-S-88M

Commit message: more final board prepping for production
Parts:
- added JP4: (no value), adafruit:1X03
- added JP5: (no value), microbuilder:1X02_ROUND
- added LED10, LED11, LED12, LED13, LED14, LED15, LED16: SFH 309, adafruit:LED3MM
- moved LED6 79.2 mm to (13.7, 18.0), turned to 225 degrees
- moved LED5 76.1 mm to (11.7, 22.9), turned to 180 degrees
- moved LED9 71.1 mm to (55.9, 22.5), turned to 0 degrees
- moved LED7 70.8 mm to (18.7, 15.9), turned to 270 degrees
- moved LED2 69.3 mm to (23.6, 27.9), turned to 45 degrees
- moved JP2 67.7 mm to (29.2, 22.9)
- moved JP3 67.7 mm to (31.8, 22.9)
- moved LED1 67.1 mm to (25.7, 22.9), turned to 0 degrees
- moved LED8 67.1 mm to (23.7, 17.8), turned to 315 degrees
- moved LED4 66.3 mm to (13.8, 27.6), turned to 135 degrees
- moved LED3 55.9 mm to (18.7, 29.8), turned to 90 degrees
- moved R5 0.32 mm to (63.5, 56.1)
Connections:
- new net INT1: JP4.2, LED10.K, LED11.K, LED12.K, LED13.K, LED14.K, LED15.K, LED16.K, LED9.K
- new net N$7: JP4.1, JP5.1
- new net N$8: JP4.3, JP5.2, LED10.A, LED11.A, LED12.A, LED13.A, LED14.A, LED15.A, LED16.A, LED9.A
- net INT: no longer LED9.K
- net N$40: no longer LED9.A
Routing:
- net INT: track 0.00 -> 52.5 mm
- net INT1: track 0.00 -> 52.4 mm
- net N$40: track 0.00 -> 41.6 mm
- net N$8: track 0.00 -> 41.5 mm, vias 1 -> 0
- net N$7: track 0.00 -> 3.07 mm
- net N$10: track 0.00 -> 3.07 mm
Other:
- outline, holes or cut-outs redrawn
- board text added: "Laptimer Remote unit Version 1"
- board text removed: "Laptimer V1"
