File: STM32F407 era/Telemetry external unit/Rasp Pi Zero model/Version 2/telemetry box.brd (EAGLE design)
At the start: 89.5 x 70.5 mm, 52 parts, among them IC1 MCP73831/OT, IC7 317T, IC8 MCP3202SN, U2 LTC3872ETS8TRMPBF, U3 SI3460DDV-T1-GE3, U4 SC16IS740IPW,112

Commit message: more fixes for V2 as noted on wiki
Parts:
- added S1: TL36WO, switch:TL3XWO
- moved CN2 2.84 mm to (66.4, 7.87)
Connections:
- new net N$1: C24.2, L1.P$2, R11.2, S1.2, U2.1, U2.6
- net VBAT: now also S1.3; no longer C24.2, L1.P$2, R11.2, U2.1, U2.6
Routing:
- net N$1: track 0.00 -> 41.1 mm, vias 0 -> 1
- net VBAT: track 39.2 -> 32.6 mm
Changed lines of the file:
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@@
 <attribute name="VALUE" x="82.8595" y="5.334" size="1.27" layer="27"/>
 </element>
-<element name="CN2" library="adafruit" package="DCJACK_2MM_PTH" value="" x="63.8175" y="6.604" smashed="yes">
-<attribute name="NAME" x="58.7375" y="8.509" size="0.8128" layer="25" rot="R90"/>
-<attribute name="VALUE" x="70.1675" y="6.604" size="1.27" layer="27" rot="R90"/>
+<element name="CN2" library="adafruit" package="DCJACK_2MM_PTH" value="" x="66.3575" y="7.874" smashed="yes">
+<attribute name="NAME" x="61.2775" y="9.779" size="0.8128" layer="25" rot="R90"/>
+<attribute name="VALUE" x="72.7075" y="7.874" size="1.27" layer="27" rot="R90"/>
 </element>
 <element name="PTC1" library="microbuilder" package="1206" value="" x="84.074" y="21.7805" smashed="yes" rot="R270">
@@
 <element name="D2" library="adafruit" package="SMADIODE" value="B320" x="81.5975" y="26.3525"/>
 <element name="D3" library="adafruit" package="SMADIODE" value="B320" x="72.39" y="45.085" rot="R180"/>
+<element name="S1" library="switch" package="TL3XWO" value="TL36WO" x="57.15" y="12.3825" rot="R180"/>
 </elements>
 <signals>
@@
 <vertex x="135.255" y="7.9375"/>
 </polygon>
+<via x="53.9115" y="39.37" extent="1-16" drill="0.381"/>
+<via x="51.3715" y="40.9575" extent="1-16" drill="0.381"/>
+<via x="51.3715" y="38.1" extent="1-16" drill="0.381"/>
 </signal>
 <signal name="5.0V">
@@
 <wire x1="63.0555" y1="30.353" x2="62.5475" y2="29.845" width="0.6096" layer="1"/>
 <wire x1="62.5475" y1="29.845" x2="62.5475" y2="24.4475" width="0.6096" layer="1"/>
-<wire x1="62.5475" y1="24.4475" x2="63.8175" y2="23.1775" width="0.6096" layer="1"/>
-<wire x1="63.8175" y1="23.1775" x2="63.8175" y2="20.204" width="0.6096" layer="1"/>
 <wire x1="68.2625" y1="28.8925" x2="68.2625" y2="29.21" width="0.4064" layer="1"/>
 <wire x1="68.2625" y1="29.21" x2="67.1195" y2="30.353" width="0.4064" layer="1"/>
 <wire x1="67.1195" y1="30.353" x2="64.77" y2="30.353" width="0.4064" layer="1"/>
+<wire x1="66.3575" y1="21.474" x2="65.521" y2="21.474" width="0.6096" layer="1"/>
+<wire x1="65.521" y1="21.474" x2="62.5475" y2="24.4475" width="0.6096" layer="1"/>
 </signal>
 <signal name="N$18">
@@
 </signal>
 <signal name="VBAT">
-<contactref element="U2" pad="1"/>
-<contactref element="U2" pad="6"/>
-<contactref element="R11" pad="2"/>
-<contactref element="L1" pad="P$2"/>
-<contactref element="C24" pad="2"/>
-<wire x1="78.0288" y1="35.2933" x2="78.0288" y2="36.3728" width="0.3048" layer="1"/>
-<wire x1="78.0288" y1="36.3728" x2="78.1685" y2="36.5125" width="0.3048" layer="1"/>
-<wire x1="79.3242" y1="37.7317" x2="79.3242" y2="36.6522" width="0.3048" layer="1"/>
-<wire x1="79.3242" y1="36.6522" x2="79.1845" y2="36.5125" width="0.3048" layer="1"/>
-<wire x1="79.1845" y1="36.5125" x2="78.1685" y2="36.5125" width="0.3048" layer="1"/>
-<wire x1="79.3242" y1="37.7317" x2="79.3242" y2="38.8112" width="0.4064" layer="1"/>
-<wire x1="79.3242" y1="38.8112" x2="79.6925" y2="39.1795" width="0.4064" layer="1"/>
-<wire x1="78.0288" y1="35.2933" x2="76.8223" y2="35.2933" width="0.4064" layer="1"/>
-<wire x1="76.8223" y1="35.2933" x2="73.66" y2="32.131" width="0.4064" layer="1"/>
-<wire x1="73.66" y1="32.131" x2="73.2985" y2="32.131" width="0.4064" layer="1"/>
-<wire x1="73.2985" y1="32.131" x2="73.0885" y2="31.921" width="0.4064" layer="1"/>
-<wire x1="68.7705" y1="33.528" x2="70.3775" y2="31.921" width="0.6096" layer="1"/>
-<wire x1="70.3775" y1="31.921" x2="73.0885" y2="31.921" width="0.6096" layer="1"/>
-<wire x1="72.8345" y1="31.667" x2="73.0885" y2="31.921" width="0.8128" layer="1"/>
 <contactref element="IC1" pad="3"/>
 <contactref element="C5" pad="2"/>
@@
 <wire x1="60.1345" y1="42.7355" x2="60.137" y2="42.7355" width="0.8128" layer="1"/>
 <wire x1="60.137" y1="42.7355" x2="60.137" y2="40.797" width="0.6096" layer="1"/>
-<wire x1="68.7705" y1="33.528" x2="67.1195" y2="33.528" width="0.6096" layer="1"/>
-<wire x1="67.1195" y1="33.528" x2="66.04" y2="34.6075" width="0.6096" layer="1"/>
-<wire x1="66.04" y1="34.6075" x2="66.04" y2="41.5925" width="0.6096" layer="1"/>
-<wire x1="66.04" y1="41.5925" x2="64.897" y2="42.7355" width="0.6096" layer="1"/>
-<wire x1="64.897" y1="42.7355" x2="60.1345" y2="42.7355" width="0.6096" layer="1"/>
+<contactref element="S1" pad="3"/>
+<wire x1="56.7225" y1="40.37" x2="53.705" y2="40.37" width="0.6096" layer="1"/>
+<wire x1="53.705" y1="40.37" x2="53.0225" y2="39.6875" width="0.6096" layer="1"/>
+<wire x1="53.0225" y1="39.6875" x2="53.0225" y2="38.1" width="0.6096" layer="1"/>
+<wire x1="53.0225" y1="38.1" x2="54.61" y2="36.5125" width="0.6096" layer="1"/>
+<wire x1="54.61" y1="36.5125" x2="54.61" y2="17.4625" width="0.6096" layer="1"/>
 </signal>
 <signal name="N$23">
@@
 <contactref element="JP1" pad="11"/>
 </signal>
+<signal name="N$1">
+<contactref element="U2" pad="1"/>
+<contactref element="U2" pad="6"/>
+<contactref element="R11" pad="2"/>
+<contactref element="L1" pad="P$2"/>
+<contactref element="C24" pad="2"/>
+<wire x1="78.0288" y1="35.2933" x2="78.0288" y2="36.3728" width="0.3048" layer="1"/>
+<wire x1="78.0288" y1="36.3728" x2="78.1685" y2="36.5125" width="0.3048" layer="1"/>
+<wire x1="79.3242" y1="37.7317" x2="79.3242" y2="36.6522" width="0.3048" layer="1"/>
+<wire x1="79.3242" y1="36.6522" x2="79.1845" y2="36.5125" width="0.3048" layer="1"/>
+<wire x1="79.1845" y1="36.5125" x2="78.1685" y2="36.5125" width="0.3048" layer="1"/>
+<wire x1="79.3242" y1="37.7317" x2="79.3242" y2="38.8112" width="0.4064" layer="1"/>
+<wire x1="79.3242" y1="38.8112" x2="79.6925" y2="39.1795" width="0.4064" layer="1"/>
+<wire x1="78.0288" y1="35.2933" x2="76.8223" y2="35.2933" width="0.4064" layer="1"/>
+<wire x1="76.8223" y1="35.2933" x2="73.66" y2="32.131" width="0.4064" layer="1"/>
+<wire x1="73.66" y1="32.131" x2="73.2985" y2="32.131" width="0.4064" layer="1"/>
+<wire x1="73.2985" y1="32.131" x2="73.0885" y2="31.921" width="0.4064" layer="1"/>
+<wire x1="68.7705" y1="33.528" x2="70.3775" y2="31.921" width="0.6096" layer="1"/>
+<wire x1="70.3775" y1="31.921" x2="73.0885" y2="31.921" width="0.6096" layer="1"/>
+<wire x1="72.8345" y1="31.667" x2="73.0885" y2="31.921" width="0.8128" layer="1"/>
+<contactref element="S1" pad="2"/>
+<wire x1="57.15" y1="17.4625" x2="57.15" y2="26.9875" width="0.6096" layer="16"/>
+<wire x1="57.15" y1="26.9875" x2="64.135" y2="33.9725" width="0.6096" layer="16"/>
+<via x="64.135" y="33.9725" extent="1-16" drill="0.9"/>
+<wire x1="64.135" y1="33.9725" x2="68.326" y2="33.9725" width="0.6096" layer="1"/>
+<wire x1="68.326" y1="33.9725" x2="68.7705" y2="33.528" width="0.6096" layer="1"/>
+</signal>
 </signals>
+<errors>
+</errors>
 </board>
 </drawing>
