File: STM32F407 era/Telemetry external unit/Rasp Pi Zero model/Version 2/telemetry box.sch (EAGLE design)
At the start: 48 parts, among them IC1 MCP73831/OT, IC7 317T, IC8 MCP3202SN, U2 LTC3872ETS8TRMPBF, U3 SI3460DDV-T1-GE3, U4 SC16IS740IPW,112

Commit message: more fixes for V2 as noted on wiki
Parts:
- added S1: TL36WO, switch:TL36WO
Connections:
- new net N$1: C24.P$2, L1.2, R11.2, S1.P, U2.IPRG, U2.VIN
- net VBAT: now also S1.S; no longer C24.P$2, L1.2, R11.2, U2.IPRG, U2.VIN
Changed lines of the file:
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@@
 <part name="D2" library="adafruit" deviceset="DIODE" device="SMA" value="B320"/>
 <part name="D3" library="adafruit" deviceset="DIODE" device="SMA" value="B320"/>
+<part name="S1" library="switch" deviceset="TL36WO" device=""/>
 </parts>
 <sheets>
@@
 <instance part="C21" gate="G$1" x="-2.54" y="139.7" rot="R90"/>
 <instance part="U$29" gate="G$1" x="-15.24" y="129.54"/>
-<instance part="U$34" gate="G$1" x="25.4" y="154.94"/>
+<instance part="U$34" gate="G$1" x="27.94" y="167.64"/>
 <instance part="R11" gate="G$1" x="15.24" y="139.7" rot="R90"/>
 <instance part="C22" gate="G$1" x="15.24" y="114.3" rot="R180"/>
@@
 <instance part="D2" gate="G$1" x="-160.02" y="182.88"/>
 <instance part="D3" gate="G$1" x="-5.08" y="119.38" rot="R180"/>
+<instance part="S1" gate="BEF1" x="25.4" y="157.48"/>
 </instances>
 <busses>
@@
 </segment>
 <segment>
-<pinref part="U2" gate="A" pin="IPRG"/>
+<pinref part="S1" gate="BEF1" pin="S"/>
 <pinref part="U$34" gate="G$1" pin="VBAT"/>
-<wire x1="27.94" y1="129.54" x2="25.4" y2="129.54" width="0.1524" layer="91"/>
-<wire x1="25.4" y1="129.54" x2="25.4" y2="134.62" width="0.1524" layer="91"/>
-<pinref part="U2" gate="A" pin="VIN"/>
-<wire x1="25.4" y1="134.62" x2="25.4" y2="149.86" width="0.1524" layer="91"/>
-<wire x1="25.4" y1="149.86" x2="25.4" y2="152.4" width="0.1524" layer="91"/>
-<wire x1="27.94" y1="134.62" x2="25.4" y2="134.62" width="0.1524" layer="91"/>
-<junction x="25.4" y="134.62"/>
-<pinref part="R11" gate="G$1" pin="2"/>
-<wire x1="25.4" y1="149.86" x2="20.32" y2="149.86" width="0.1524" layer="91"/>
-<wire x1="20.32" y1="149.86" x2="15.24" y2="149.86" width="0.1524" layer="91"/>
-<wire x1="15.24" y1="149.86" x2="15.24" y2="144.78" width="0.1524" layer="91"/>
-<junction x="25.4" y="149.86"/>
-<pinref part="L1" gate="G$1" pin="2"/>
-<wire x1="20.32" y1="139.7" x2="20.32" y2="149.86" width="0.1524" layer="91"/>
-<junction x="20.32" y="149.86"/>
-<pinref part="C24" gate="G$1" pin="P$2"/>
-<wire x1="25.4" y1="149.86" x2="27.94" y2="149.86" width="0.1524" layer="91"/>
-<wire x1="27.94" y1="149.86" x2="27.94" y2="147.32" width="0.1524" layer="91"/>
+<wire x1="27.94" y1="162.56" x2="27.94" y2="165.1" width="0.1524" layer="91"/>
 </segment>
 </net>
@@
 </segment>
 </net>
+<net name="N$1" class="0">
+<segment>
+<pinref part="U2" gate="A" pin="IPRG"/>
+<wire x1="27.94" y1="129.54" x2="25.4" y2="129.54" width="0.1524" layer="91"/>
+<wire x1="25.4" y1="129.54" x2="25.4" y2="134.62" width="0.1524" layer="91"/>
+<pinref part="U2" gate="A" pin="VIN"/>
+<wire x1="25.4" y1="134.62" x2="25.4" y2="149.86" width="0.1524" layer="91"/>
+<wire x1="27.94" y1="134.62" x2="25.4" y2="134.62" width="0.1524" layer="91"/>
+<junction x="25.4" y="134.62"/>
+<pinref part="R11" gate="G$1" pin="2"/>
+<wire x1="25.4" y1="149.86" x2="20.32" y2="149.86" width="0.1524" layer="91"/>
+<wire x1="20.32" y1="149.86" x2="15.24" y2="149.86" width="0.1524" layer="91"/>
+<wire x1="15.24" y1="149.86" x2="15.24" y2="144.78" width="0.1524" layer="91"/>
+<junction x="25.4" y="149.86"/>
+<pinref part="L1" gate="G$1" pin="2"/>
+<wire x1="20.32" y1="139.7" x2="20.32" y2="149.86" width="0.1524" layer="91"/>
+<junction x="20.32" y="149.86"/>
+<pinref part="C24" gate="G$1" pin="P$2"/>
+<wire x1="25.4" y1="149.86" x2="27.94" y2="149.86" width="0.1524" layer="91"/>
+<wire x1="27.94" y1="149.86" x2="27.94" y2="147.32" width="0.1524" layer="91"/>
+<pinref part="S1" gate="BEF1" pin="P"/>
+<wire x1="25.4" y1="149.86" x2="25.4" y2="152.4" width="0.1524" layer="91"/>
+</segment>
+</net>
