File: STM32F407 era/Traction control modul/Version 1/TC board.sch (EAGLE design)
At the start: 66 parts, among them IC1 74HC14D, IC2 lm2575, IC3 74AC08D, IC5 REG1117, IC6 74AC14D, J1 CON1, J2 CON1, U1 MAX13052ESA+, U2 MAX232AEWE+, U3 MAX531AESD+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

Commit message: Revert "started work on TC V2"
This reverts commit da86986705d51cbc4691d6d7bad1c5aae1ca4806.
Parts:
- removed H6, H7: MOUNT-HOLE3.0, holes:MOUNT-HOLE3.0
- removed J2: CON1, unicorn_v2:AUTOCONNECTOR
- removed U$28: VNH2SP30, SparkFun-PowerIC:VNH2SP30
- added R10, R14, R16, R20: 178, microbuilder:RESISTOR_0603
- added R11, R15, R21, R8: 604, microbuilder:RESISTOR_0603
Connections:
- net BITE: now also R15.2
- net BITEO: now also R15.1, R16.2
- net FUEL-RECIEVE: now also R21.2
- net FUEL-RECIEVEI: now also R20.2, R21.1
- net GND: now also R10.1, R14.1, R16.1, R20.1
- net GSENS: now also R8.2
- net GSENSO: now also R10.2, R8.1
- net YAW: now also R11.2
- net YAWO: now also R11.1, R14.2

Commit message: started work on TC V2
Parts:
- removed R10, R14, R16, R20: 178, microbuilder:RESISTOR_0603
- removed R11, R15, R21, R8: 604, microbuilder:RESISTOR_0603
- added H6, H7: MOUNT-HOLE3.0, holes:MOUNT-HOLE3.0
- added J2: CON1, unicorn_v2:AUTOCONNECTOR
- added U$28: VNH2SP30, SparkFun-PowerIC:VNH2SP30
Connections:
- net BITE: no longer R15.2
- net BITEO: no longer R15.1, R16.2
- net FUEL-RECIEVE: no longer R21.2
- net FUEL-RECIEVEI: no longer R20.2, R21.1
- net GND: no longer R10.1, R14.1, R16.1, R20.1
- net GSENS: no longer R8.2
- net GSENSO: no longer R10.2, R8.1
- net YAW: no longer R11.2
- net YAWO: no longer R11.1, R14.2
