File: Laptimer/Version 3/Mixed/Laptimer.brd (EAGLE design)
At the start: 100 x 75 mm, 74 parts, among them IC1 MCP73831/OT, IC2 REG1117, IC4 74HC04D, IC6 74HC08D, Q1 8mhz, Q4 PBSS4120T, U2 LTC3872ETS8TRMPBF, U3 SI3460DDV-T1-GE3, X1 mini-usb, X2 GLX-S-88M

Commit message: more work on better layout for V3
Parts:
- moved R10 2.54 mm to (84.8, 53.0)
- moved XB1 2.54 mm to (80.9, 59.4)
- moved C2 2.54 mm to (76.2, 65.4)
- moved C9 2.54 mm to (76.2, 67.3)
- moved IC2 2.54 mm to (81.9, 60.6)
- moved Q2 2.54 mm to (81.9, 52.4)
- moved R11 2.54 mm to (78.1, 52.7)
Routing:
- net 5.0V: track 245.3 -> 242.8 mm
- net TX2: track 57.7 -> 55.2 mm
- net RX2: track 86.5 -> 84.0 mm
- net RSSI: track 89.4 -> 86.9 mm
- net ASSOC: track 76.1 -> 73.6 mm
- net 1D-: track 14.3 -> 13.6 mm
