File: Laptimer/Version 3/Lora + XBEE/remote unit/Laptimer.sch (EAGLE design)
At the start: 33 parts, among them IC4 74HC04D, IC5 NE555D, X2 GLX-S-88M

Commit message: laptimer RC done, com node (done) need checkup
Parts:
- removed C13, C17: 100n, rcl:C-EUC0603K
- removed IC4: 74HC04D, 74xx-eu:74HC04D
- removed IC5: NE555D, linear:NE555D
- removed JP2, JP5: (no value), microbuilder:HEADER-1X2ROUND
- removed JP3, JP4: (no value), adafruit:PINHD-1X3
- removed LED1, LED10, LED11, LED12, LED13, LED14, LED15, LED16, LED2, LED3, LED4, LED5, LED6, LED7, LED8, LED9: SFH 309, adafruit:LED3MM
- removed Q3: (no value), microbuilder:TRANSISTOR_NPNWIDE
- removed R15, R16: 220, rcl:R-EU_R0603
- removed R18: 1k, rcl:R-EU_R0603
- removed R19: 100, rcl:R-EU_R0603
- removed U$19: BI-LEVEL-LED-INDICATOR, unicorn_v2:BI-LEVEL-LED-INDICATOR
- removed X2: GLX-S-88M, con-kycon:GLX-S-88M
- added BAT1: (no value), SparkFun-Electromechanical:BATTERY18650
- added C1, C15: 100n, microbuilder:CAP_CERAMIC_0603
- added C10, C11, C2, C24: 10u, microbuilder:CAP_CERAMIC_0805
- added C12: 1n8, microbuilder:CAP_CERAMIC_0603
- added C21: 47p, microbuilder:CAP_CERAMIC_0603
- added C22: 1n, microbuilder:CAP_CERAMIC_0603
- added C23, C25: 100u, microbuilder:CAP_CERAMIC1206
- added C4, C9: 22u, microbuilder:CAP_CERAMIC_0805
- added D1: 3V, microbuilder:DIODE-ZENER
- added D3: B320, adafruit:DIODESMA
- added H1, H2: MOUNT-HOLE3.0, holes:MOUNT-HOLE3.0
- added IC1: MCP73831/OT, adafruit:MCP73831/OT
- added IC2: REG1117, burr-brown:REG1117
- added L1: FDVE0630-H-1R0M, microbuilder:INDUCTORTDK_SLF6045
- added PTC2: (no value), microbuilder:PTC1206
- added Q4: PBSS4120T, microbuilder:TRANSISTOR_NPNWIDE
- added R1, R8: 2k, microbuilder:RESISTOR_0603
- added R17: 34k8, microbuilder:RESISTOR_0603
- added R2: 470, microbuilder:RESISTOR_0603
- added R20: 11k, microbuilder:RESISTOR_0603
- added R21: 17k4, microbuilder:RESISTOR_0603
- added R23: 1m, microbuilder:RESISTOR_0603
- added R3, R4: 1k, microbuilder:RESISTOR_0603
- added R6: 10k, microbuilder:RESISTOR_0603
- added R7: 220, microbuilder:RESISTOR_0603
- added S1: TL36WO, switch:TL36WO
- added U$13, U$14: BI-LEVEL-LED-INDICATOR, unicorn_v2:BI-LEVEL-LED-INDICATOR
- added U$7: GAMMA-868-SO, unicorn_v2:GAMMA-868-SO
- added U1: (no value), microbuilder:LM358
- added U2: LTC3872ETS8TRMPBF, LTC_By_element14_Batch_1:LTC3872ETS8TRMPBF
- added U3: SI3460DDV-T1-GE3, Vishay_By_element14_Batch_1:SI3457CDV-T1-GE3
- added X1: mini-usb, con-cypressindustries:MINI-USB-SCHIELD-32005-301
- R5: device rcl:R-EU_R0603 -> microbuilder:RESISTOR_0603
Connections:
- removed net INT: JP3.2, LED1.C, LED2.C, LED3.C, LED4.C, LED5.C, LED6.C, LED7.C, LED8.C
- removed net INT1: JP4.2, LED10.C, LED11.C, LED12.C, LED13.C, LED14.C, LED15.C, LED16.C, LED9.C
- removed net N$10: JP2.1, JP3.1
- removed net N$22: IC4A.O, X2.5
- removed net N$25: R15.2, U$19.ANODE1
- removed net N$36: C17.1, IC5.DIS, IC5.THR, R18.2, R19.2
- removed net N$40: JP2.2, JP3.3, LED1.A, LED2.A, LED3.A, LED4.A, LED5.A, LED6.A, LED7.A, LED8.A
- removed net N$41: Q3.C, R19.1
- removed net PT-OUT: IC4A.I, IC5.Q, X2.4
- new net +UB: C10.P$2, C15.P$1, IC1.VDD, PTC2.1, R6.1, U$13.ANODE1
- new net 3.3V: C9.P$1, IC2.VOUT, U$7.VCC
- new net BAT-ADC: BAT1.+, C11.P$1, IC1.VBAT, S1.P
- new net CHRG-DONE-LED: R3.1, U$13.ANODE2
- new net CT: U$7.OP1, U$7.OP8
- new net LASER: R4.1, U$7.OP3
- new net MOSD: D3.A, L1.1, U2.SW, U3.D, U3.D_2, U3.D_3, U3.D_4
- new net N$1: R17.2, R20.1, U2.VFB
- new net N$13: C4.P$1, PTC2.2, X1G$1.1
- new net N$14: R2.1, U$13.CATHODE1
- new net N$2: C12.P$2, R21.2
- new net N$27: C21.P$2, R21.1, U2.ITH
- new net N$29: C22.P$2, R23.1, U2.RUN/SS
- new net N$3: IC1.PROG, R1.1
- new net N$4: IC1.STAT, R2.2, R3.2
- new net N$5: JP1.1, Q4.E, R5.1
- new net N$6: Q4.B, R4.2
- new net RLB: U$7.OP6, U1G$1.OUT
- new net VBAT: C24.P$2, L1.2, R23.2, S1.O, U1G$1.+IN, U2.IPRG, U2.VIN
- net 5.0V: now also C1.P$1, C2.P$1, C23.P$1, C25.P$1, D3.C, IC2.VIN, Q4.C, R17.1, R7.1, R8.1, U1G$1.V+; no longer C13.2, IC4P.VCC, IC5.R, IC5.V+, JP1.1, R16.1, R18.1, R5.1, X2.1, X2.2
- net GND: now also BAT1.-, C1.P$2, C10.P$1, C11.P$2, C12.P$1, C15.P$2, C2.P$2, C21.P$1, C22.P$1, C23.P$2, C24.P$1, C25.P$2, C4.P$2, C9.P$2, D1.A, IC1.VSS, IC2.GND, R1.2, R20.2, R6.2, U$13.CATHODE2, U$14.CATHODE1, U$14.CATHODE2, U$7.GND1, U$7.GND2, U$7.OPT1, U1G$1.V-, U2.GND, U3.S, X1G$1.5, X1S.S1, X1S.S2, X1S.S3, X1S.S4; no longer C13.1, C17.2, IC4B.I, IC4C.I, IC4D.I, IC4E.I, IC4F.I, IC4P.GND, IC5.GND, Q3.E, U$19.CATHODE1, U$19.CATHODE2, X2.3, X2.6, X2.7, X2.8, X2.S1, X2.S2
- net N$32: now also R7.2, U$14.ANODE2; no longer R16.2, U$19.ANODE2
- net N$7: now also D1.C, R8.2, U1G$1.-IN; no longer JP4.1, JP5.1
- net N$8: now also U2.NGATE, U3.G; no longer JP4.3, JP5.2, LED10.A, LED11.A, LED12.A, LED13.A, LED14.A, LED15.A, LED16.A, LED9.A
- net PT-IN: now also U$7.OP5; no longer IC5.TR, Q3.B, R15.1
Other:
- note added: "Power Supply + LiPo Charger"
- note added: "USB"
- note removed: "Missing Pulse Detector"
- moved on the sheet: JP1, R5
