File: STM32F407 era/Traction control modul/Version 2/PCB Box/TC board.sch (EAGLE design)
At the start: 144 parts, among them IC2 lm2575, IC5 REG1117, J1 CON1, J2 CON1, U1 MAX13052ESA+, U2 MAX232AEWE+, U3 MAX531AESD+, U5 MAX9926, U6 MAX9926, U7 HEF4049BT

Commit message: continued work with last additions
Parts:
- added C40: 100n, microbuilder:CAP_CERAMIC_0603
- added PTC2: (no value), microbuilder:PTC1812
- added U8: MCP3004-I/ST, Microchip_By_element14_Batch_1:MCP3004-I/ST
Connections:
- new net ADC_CS: U$1G$1.PE9, U8.*CS/SHDN
- new net N$37: C7.+, IC2.IN, PTC2.1
- new net SCL: U$1G$3.PB8
- new net SDA: U$1G$3.PB7
- net 12V: now also PTC2.2; no longer C7.+, IC2.IN
- net 3.3V: now also C40.P$1, U8.VDD, U8.VREF
- net AUX1: no longer U$1G$1.PE9
- net GND: now also C40.P$2, U8.AGND, U8.DGND
- net MISO: now also U8.DOUT
- net MOSI: now also U8.DIN
- net RPM1: now also U$1G$3.PD4; no longer U$1G$3.PD2
- net RPM3: now also U$1G$3.PD2; no longer U$1G$3.PD4
- net SCK: now also U8.CLK
Changed lines of the file:
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@@
 <part name="U$66" library="microbuilder" deviceset="5.0V" device=""/>
 <part name="U$67" library="microbuilder" deviceset="5.0V" device=""/>
+<part name="PTC2" library="microbuilder" deviceset="PTC" device="1812"/>
+<part name="U8" library="Microchip_By_element14_Batch_1" deviceset="MCP3004-I/ST" device=""/>
+<part name="U$68" library="microbuilder" deviceset="3.3V" device=""/>
+<part name="GND13" library="supply1" deviceset="GND" device=""/>
+<part name="C40" library="microbuilder" deviceset="CAP_CERAMIC" device="_0603" value="100n"/>
 </parts>
 <sheets>
@@
 <instance part="U$2" gate="G$1" x="-129.54" y="-12.7"/>
 <instance part="U$3" gate="G$1" x="-99.06" y="-12.7"/>
-<instance part="U$4" gate="G$1" x="-193.04" y="162.56"/>
+<instance part="U$4" gate="G$1" x="-198.12" y="165.1"/>
 <instance part="GND8" gate="1" x="-177.8" y="137.16"/>
 <instance part="IC2" gate="G$1" x="-177.8" y="154.94"/>
@@
 <instance part="U$66" gate="G$1" x="137.16" y="-10.16"/>
 <instance part="U$67" gate="G$1" x="134.62" y="-40.64"/>
+<instance part="PTC2" gate="G$1" x="-193.04" y="157.48"/>
+<instance part="U8" gate="A" x="320.04" y="-7.62"/>
+<instance part="U$68" gate="G$1" x="297.18" y="7.62"/>
+<instance part="GND13" gate="1" x="297.18" y="-30.48"/>
+<instance part="C40" gate="G$1" x="294.64" y="-22.86" rot="MR0"/>
 </instances>
 <busses>
@@
 <wire x1="177.8" y1="-22.86" x2="177.8" y2="-27.94" width="0.1524" layer="91"/>
 </segment>
+<segment>
+<pinref part="U8" gate="A" pin="DGND"/>
+<wire x1="299.72" y1="-22.86" x2="297.18" y2="-22.86" width="0.1524" layer="91"/>
+<pinref part="GND13" gate="1" pin="GND"/>
+<wire x1="297.18" y1="-22.86" x2="297.18" y2="-25.4" width="0.1524" layer="91"/>
+<pinref part="U8" gate="A" pin="AGND"/>
+<wire x1="297.18" y1="-25.4" x2="297.18" y2="-27.94" width="0.1524" layer="91"/>
+<wire x1="299.72" y1="-25.4" x2="297.18" y2="-25.4" width="0.1524" layer="91"/>
+<junction x="297.18" y="-25.4"/>
+<pinref part="C40" gate="G$1" pin="P$2"/>
+<wire x1="294.64" y1="-25.4" x2="297.18" y2="-25.4" width="0.1524" layer="91"/>
+</segment>
 </net>
 <net name="3.3V" class="0">
@@
 <pinref part="U$63" gate="G$1" pin="3.3V"/>
 </segment>
-</net>
-<net name="12V" class="0">
 <segment>
-<pinref part="U$4" gate="G$1" pin="12V"/>
-<wire x1="-187.96" y1="157.48" x2="-193.04" y2="157.48" width="0.1524" layer="91"/>
-<wire x1="-193.04" y1="157.48" x2="-193.04" y2="160.02" width="0.1524" layer="91"/>
-<pinref part="IC2" gate="G$1" pin="IN"/>
-<wire x1="-193.04" y1="152.4" x2="-193.04" y2="157.48" width="0.1524" layer="91"/>
-<junction x="-193.04" y="157.48"/>
-<pinref part="C7" gate="G$1" pin="+"/>
+<pinref part="U8" gate="A" pin="VDD"/>
+<pinref part="U$68" gate="G$1" pin="3.3V"/>
+<wire x1="299.72" y1="-20.32" x2="297.18" y2="-20.32" width="0.1524" layer="91"/>
+<wire x1="297.18" y1="-20.32" x2="297.18" y2="-17.78" width="0.1524" layer="91"/>
+<pinref part="C40" gate="G$1" pin="P$1"/>
+<wire x1="297.18" y1="-17.78" x2="297.18" y2="-15.24" width="0.1524" layer="91"/>
+<wire x1="297.18" y1="-15.24" x2="297.18" y2="5.08" width="0.1524" layer="91"/>
+<wire x1="294.64" y1="-17.78" x2="297.18" y2="-17.78" width="0.1524" layer="91"/>
+<junction x="297.18" y="-17.78"/>
+<pinref part="U8" gate="A" pin="VREF"/>
+<wire x1="299.72" y1="-15.24" x2="297.18" y2="-15.24" width="0.1524" layer="91"/>
+<junction x="297.18" y="-15.24"/>
 </segment>
+</net>
+<net name="12V" class="0">
 <segment>
 <pinref part="IC5" gate="G$1" pin="VIN"/>
@@
 <junction x="167.64" y="106.68"/>
 </segment>
+<segment>
+<pinref part="U$4" gate="G$1" pin="12V"/>
+<wire x1="-198.12" y1="157.48" x2="-198.12" y2="162.56" width="0.1524" layer="91"/>
+<pinref part="PTC2" gate="G$1" pin="2"/>
+</segment>
 </net>
 <net name="N$1" class="0">
@@
 </segment>
 <segment>
-<label x="-48.26" y="-20.32" size="1.27" layer="95" xref="yes"/>
-<pinref part="U$1" gate="G$3" pin="PD2"/>
-<wire x1="-50.8" y1="-20.32" x2="-48.26" y2="-20.32" width="0.1524" layer="91"/>
+<label x="-48.26" y="-22.86" size="1.27" layer="95" xref="yes"/>
+<pinref part="U$1" gate="G$3" pin="PD4"/>
+<wire x1="-50.8" y1="-22.86" x2="-48.26" y2="-22.86" width="0.1524" layer="91"/>
 </segment>
 </net>
@@
 </segment>
 <segment>
-<label x="-48.26" y="-22.86" size="1.27" layer="95" xref="yes"/>
-<pinref part="U$1" gate="G$3" pin="PD4"/>
-<wire x1="-50.8" y1="-22.86" x2="-48.26" y2="-22.86" width="0.1524" layer="91"/>
+<label x="-48.26" y="-20.32" size="1.27" layer="95" xref="yes"/>
+<pinref part="U$1" gate="G$3" pin="PD2"/>
+<wire x1="-50.8" y1="-20.32" x2="-48.26" y2="-20.32" width="0.1524" layer="91"/>
 </segment>
 </net>
@@
 <label x="-96.52" y="-20.32" size="1.27" layer="95" xref="yes"/>
 </segment>
+<segment>
+<pinref part="U8" gate="A" pin="DIN"/>
+<wire x1="294.64" y1="-12.7" x2="299.72" y2="-12.7" width="0.1524" layer="91"/>
+<label x="294.64" y="-12.7" size="1.27" layer="95" rot="R180" xref="yes"/>
+</segment>
 </net>
 <net name="SCK" class="0">
@@
 <label x="-96.52" y="-17.78" size="1.27" layer="95" xref="yes"/>
 </segment>
+<segment>
+<pinref part="U8" gate="A" pin="CLK"/>
+<wire x1="294.64" y1="0" x2="299.72" y2="0" width="0.1524" layer="91"/>
+<label x="294.64" y="0" size="1.27" layer="95" rot="R180" xref="yes"/>
+</segment>
 </net>
 <net name="MISO" class="0">
@@
 <label x="-132.08" y="-20.32" size="1.27" layer="95" rot="R180" xref="yes"/>
 </segment>
+<segment>
+<pinref part="U8" gate="A" pin="DOUT"/>
+<wire x1="342.9" y1="-10.16" x2="340.36" y2="-10.16" width="0.1524" layer="91"/>
+<label x="342.9" y="-10.16" size="1.27" layer="95" xref="yes"/>
+</segment>
 </net>
 <net name="VOUT" class="0">
@@
 <net name="AUX1" class="0">
 <segment>
-<pinref part="U$1" gate="G$1" pin="PE9"/>
-<wire x1="-157.48" y1="-30.48" x2="-160.02" y2="-30.48" width="0.1524" layer="91"/>
-<label x="-157.48" y="-30.48" size="1.27" layer="95" xref="yes"/>
-</segment>
-<segment>
 <pinref part="J1" gate="G$1" pin="D"/>
 <wire x1="73.66" y1="99.06" x2="68.58" y2="99.06" width="0.1524" layer="91"/>
@@
 </segment>
 </net>
+<net name="SDA" class="0">
+<segment>
+<pinref part="U$1" gate="G$3" pin="PB7"/>
+<wire x1="-76.2" y1="-33.02" x2="-73.66" y2="-33.02" width="0.1524" layer="91"/>
+<label x="-76.2" y="-33.02" size="1.27" layer="95" rot="R180" xref="yes"/>
+</segment>
+</net>
+<net name="SCL" class="0">
+<segment>
+<pinref part="U$1" gate="G$3" pin="PB8"/>
+<wire x1="-48.26" y1="-33.02" x2="-50.8" y2="-33.02" width="0.1524" layer="91"/>
+<label x="-48.26" y="-33.02" size="1.27" layer="95" xref="yes"/>
+</segment>
+</net>
+<net name="N$37" class="0">
+<segment>
+<pinref part="IC2" gate="G$1" pin="IN"/>
+<wire x1="-193.04" y1="152.4" x2="-187.96" y2="157.48" width="0.1524" layer="91"/>
+<pinref part="C7" gate="G$1" pin="+"/>
+<pinref part="PTC2" gate="G$1" pin="1"/>
+<junction x="-187.96" y="157.48"/>
+</segment>
+</net>
+<net name="ADC_CS" class="0">
+<segment>
+<pinref part="U8" gate="A" pin="*CS/SHDN"/>
+<wire x1="342.9" y1="0" x2="340.36" y2="0" width="0.1524" layer="91"/>
+<label x="342.9" y="0" size="1.27" layer="95" xref="yes"/>
+</segment>
+<segment>
+<pinref part="U$1" gate="G$1" pin="PE9"/>
+<wire x1="-157.48" y1="-30.48" x2="-160.02" y2="-30.48" width="0.1524" layer="91"/>
+<label x="-157.48" y="-30.48" size="1.27" layer="95" xref="yes"/>
+</segment>
+</net>

Commit message: added switch to select int or ADC for oilp
Parts:
- added C41: 100n, microbuilder:CAP_CERAMIC_0603
- added R54: 499, microbuilder:RESISTOR_0603
- added R55: 976, microbuilder:RESISTOR_0603
- added R56: 10k, microbuilder:RESISTOR_0603
- added S1: (no value), SparkFun-Electromechanical:SWITCH-SPDT-SMD-A
- added U$69: MCP6001T-E/OT, Microchip_By_element14_Batch_1:MCP6001T-E/OT
Connections:
- new net N$42: R54.1, R55.2, U$69.VIN+
- new net N$43: R56.1, U$69.VIN-, U$69.VOUT, U8.CH0
- new net OILPI: S1.O, U$1G$1.PE13
- net 3.3V: now also C41.P$2, R56.2, U$69.VDD
- net GND: now also C41.P$1, R55.1, U$69.VSS
- net OILP: now also S1.P; no longer U$1G$1.PE13
- net YAW: now also R54.2, S1.S
Other:
- moved on the sheet: C40, U8

Commit message: adding last changes to accomendate changes in H-Bridge
Parts:
- removed C13: 330n, microbuilder:CAP_CERAMIC_0603
- removed Q10: (no value), microbuilder:TRANSISTOR_NPNWIDE
- removed R30: 1k5, microbuilder:RESISTOR_0603
- removed R31: 10k, microbuilder:RESISTOR_0603
Connections:
- net HB-EN1 renamed HB1-DIR
- net HB-EN2 renamed HB2-PWM
- net HB-MD renamed HB2-EN
- removed net HB-CS: C13.P$1, R31.1, U$1G$4.PC1
- removed net HB-INA: U$1G$2.PD8, U4.A6
- removed net HB-INB: U$1G$2.PD13, U4.A2
- removed net HB-PWM: U$1G$2.PD11, U4.A4
- removed net N$30: Q10.E, R30.1, R31.2
- new net HB1-EN: U$1G$2.PD11, U4.A6
- new net HB1-PWM: U$1G$2.PD13, U4.A4
- new net HB2-DIR: U$1G$2.PD15, U4.A2
- net 3.3V: no longer Q10.C
- net GND: no longer C13.P$2, R30.2
- net HB-CS-IN: no longer Q10.B
Changed lines of the file:
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@@
 <part name="GND44" library="supply1" deviceset="GND" device=""/>
 <part name="C1" library="microbuilder" deviceset="CAP_CERAMIC" device="_0603" value="100n"/>
-<part name="Q10" library="microbuilder" deviceset="TRANSISTOR_NPN" device="WIDE"/>
-<part name="U$9" library="microbuilder" deviceset="3.3V" device=""/>
-<part name="R30" library="microbuilder" deviceset="RESISTOR" device="_0603" value="1k5"/>
-<part name="R31" library="microbuilder" deviceset="RESISTOR" device="_0603" value="10k"/>
-<part name="C13" library="microbuilder" deviceset="CAP_CERAMIC" device="_0603" value="330n"/>
-<part name="GND33" library="supply1" deviceset="GND" device=""/>
-<part name="GND35" library="supply1" deviceset="GND" device=""/>
 <part name="C15" library="microbuilder" deviceset="CAP_ELECTROLYTIC" device="PANASONIC_D" value="33uf pan FC"/>
 <part name="GND38" library="supply1" deviceset="GND" device=""/>
@@
 <instance part="GND44" gate="1" x="304.8" y="106.68"/>
 <instance part="C1" gate="G$1" x="297.18" y="111.76" rot="MR90"/>
-<instance part="Q10" gate="G$1" x="342.9" y="99.06"/>
-<instance part="U$9" gate="G$1" x="342.9" y="106.68"/>
-<instance part="R30" gate="G$1" x="342.9" y="83.82" rot="R270"/>
-<instance part="R31" gate="G$1" x="350.52" y="91.44" rot="R180"/>
-<instance part="C13" gate="G$1" x="358.14" y="83.82"/>
-<instance part="GND33" gate="1" x="342.9" y="76.2"/>
-<instance part="GND35" gate="1" x="358.14" y="76.2"/>
 <instance part="C15" gate="G$1" x="-139.7" y="104.14"/>
 <instance part="GND38" gate="1" x="71.12" y="73.66"/>
@@
 </segment>
 <segment>
-<pinref part="R30" gate="G$1" pin="2"/>
-<pinref part="GND33" gate="1" pin="GND"/>
-</segment>
-<segment>
-<pinref part="C13" gate="G$1" pin="P$2"/>
-<pinref part="GND35" gate="1" pin="GND"/>
-<wire x1="358.14" y1="78.74" x2="358.14" y2="81.28" width="0.1524" layer="91"/>
-</segment>
-<segment>
 <pinref part="GND36" gate="1" pin="GND"/>
 <pinref part="C15" gate="G$1" pin="-"/>
@@
 </segment>
 <segment>
-<pinref part="Q10" gate="G$1" pin="C"/>
-<pinref part="U$9" gate="G$1" pin="3.3V"/>
-</segment>
-<segment>
 <pinref part="U$24" gate="A" pin="VDD"/>
 <wire x1="33.02" y1="147.32" x2="27.94" y2="147.32" width="0.1524" layer="91"/>
@@
 </segment>
 </net>
-<net name="HB-INA" class="0">
-<segment>
-<label x="-132.08" y="-22.86" size="1.27" layer="95" rot="R180" xref="yes"/>
-<pinref part="U$1" gate="G$2" pin="PD8"/>
-<wire x1="-132.08" y1="-22.86" x2="-124.46" y2="-22.86" width="0.1524" layer="91"/>
-</segment>
-<segment>
-<pinref part="U4" gate="G$1" pin="A6"/>
-<wire x1="271.78" y1="81.28" x2="274.32" y2="81.28" width="0.1524" layer="91"/>
-<label x="271.78" y="81.28" size="1.27" layer="95" font="vector" rot="R180" xref="yes"/>
-</segment>
-</net>
-<net name="HB-EN1" class="0">
-<segment>
-<label x="-132.08" y="-25.4" size="1.27" layer="95" rot="R180" xref="yes"/>
-<pinref part="U$1" gate="G$2" pin="PD10"/>
-<wire x1="-132.08" y1="-25.4" x2="-124.46" y2="-25.4" width="0.1524" layer="91"/>
-</segment>
-<segment>
-<pinref part="U4" gate="G$1" pin="A5"/>
-<wire x1="271.78" y1="83.82" x2="274.32" y2="83.82" width="0.1524" layer="91"/>
-<label x="271.78" y="83.82" size="1.27" layer="95" font="vector" rot="R180" xref="yes"/>
-</segment>
-</net>
-<net name="HB-PWM" class="0">
-<segment>
-<label x="-96.52" y="-25.4" size="1.27" layer="95" xref="yes"/>
-<pinref part="U$1" gate="G$2" pin="PD11"/>
-<wire x1="-96.52" y1="-25.4" x2="-101.6" y2="-25.4" width="0.1524" layer="91"/>
-</segment>
-<segment>
-<pinref part="U4" gate="G$1" pin="A4"/>
-<wire x1="271.78" y1="86.36" x2="274.32" y2="86.36" width="0.1524" layer="91"/>
-<label x="271.78" y="86.36" size="1.27" layer="95" font="vector" rot="R180" xref="yes"/>
-</segment>
-</net>
-<net name="HB-EN2" class="0">
-<segment>
-<label x="-132.08" y="-27.94" size="1.27" layer="95" rot="R180" xref="yes"/>
-<pinref part="U$1" gate="G$2" pin="PD12"/>
-<wire x1="-132.08" y1="-27.94" x2="-124.46" y2="-27.94" width="0.1524" layer="91"/>
-</segment>
-<segment>
-<pinref part="U4" gate="G$1" pin="A3"/>
-<wire x1="271.78" y1="88.9" x2="274.32" y2="88.9" width="0.1524" layer="91"/>
-<label x="271.78" y="88.9" size="1.27" layer="95" font="vector" rot="R180" xref="yes"/>
-</segment>
-</net>
-<net name="HB-INB" class="0">
-<segment>
-<label x="-96.52" y="-27.94" size="1.27" layer="95" xref="yes"/>
-<pinref part="U$1" gate="G$2" pin="PD13"/>
-<wire x1="-96.52" y1="-27.94" x2="-101.6" y2="-27.94" width="0.1524" layer="91"/>
-</segment>
-<segment>
-<pinref part="U4" gate="G$1" pin="A2"/>
-<wire x1="271.78" y1="91.44" x2="274.32" y2="91.44" width="0.1524" layer="91"/>
-<label x="271.78" y="91.44" size="1.27" layer="95" font="vector" rot="R180" xref="yes"/>
-</segment>
-</net>
-<net name="HB-MD" class="0">
-<segment>
-<label x="-132.08" y="-30.48" size="1.27" layer="95" rot="R180" xref="yes"/>
-<pinref part="U$1" gate="G$2" pin="PD14"/>
-<wire x1="-132.08" y1="-30.48" x2="-124.46" y2="-30.48" width="0.1524" layer="91"/>
-</segment>
-<segment>
-<pinref part="U4" gate="G$1" pin="A1"/>
-<wire x1="271.78" y1="93.98" x2="274.32" y2="93.98" width="0.1524" layer="91"/>
-<label x="271.78" y="93.98" size="1.27" layer="95" font="vector" rot="R180" xref="yes"/>
-</segment>
-</net>
 <net name="RPM3IN" class="0">
 <segment>
@@
 </segment>
 </net>
-<net name="N$30" class="0">
-<segment>
-<pinref part="Q10" gate="G$1" pin="E"/>
-<pinref part="R30" gate="G$1" pin="1"/>
-<wire x1="342.9" y1="93.98" x2="342.9" y2="91.44" width="0.1524" layer="91"/>
-<pinref part="R31" gate="G$1" pin="2"/>
-<wire x1="342.9" y1="91.44" x2="342.9" y2="88.9" width="0.1524" layer="91"/>
-<wire x1="345.44" y1="91.44" x2="342.9" y2="91.44" width="0.1524" layer="91"/>
-<junction x="342.9" y="91.44"/>
-</segment>
-</net>
 <net name="HB-CS-IN" class="0">
 <segment>
-<pinref part="Q10" gate="G$1" pin="B"/>
-<wire x1="337.82" y1="99.06" x2="335.28" y2="99.06" width="0.1524" layer="91"/>
-<label x="335.28" y="99.06" size="1.27" layer="95" font="vector" rot="R180" xref="yes"/>
-</segment>
-<segment>
 <pinref part="J1" gate="G$2" pin="H"/>
 <wire x1="104.14" y1="88.9" x2="99.06" y2="88.9" width="0.1524" layer="91"/>
@@
 </segment>
 </net>
-<net name="HB-CS" class="0">
-<segment>
-<pinref part="R31" gate="G$1" pin="1"/>
-<pinref part="C13" gate="G$1" pin="P$1"/>
-<wire x1="355.6" y1="91.44" x2="358.14" y2="91.44" width="0.1524" layer="91"/>
-<wire x1="358.14" y1="91.44" x2="358.14" y2="88.9" width="0.1524" layer="91"/>
-<wire x1="360.68" y1="91.44" x2="358.14" y2="91.44" width="0.1524" layer="91"/>
-<junction x="358.14" y="91.44"/>
-<label x="360.68" y="91.44" size="1.27" layer="95" xref="yes"/>
-</segment>
-<segment>
-<pinref part="U$1" gate="G$4" pin="PC1"/>
-<wire x1="12.7" y1="-27.94" x2="7.62" y2="-27.94" width="0.1524" layer="91"/>
-<label x="12.7" y="-27.94" size="1.27" layer="95" xref="yes"/>
-</segment>
-</net>
 <net name="BITE" class="0">
 <segment>
@@
 </segment>
 </net>
+<net name="HB1-DIR" class="0">
+<segment>
+<label x="-132.08" y="-25.4" size="1.27" layer="95" rot="R180" xref="yes"/>
+<pinref part="U$1" gate="G$2" pin="PD10"/>
+<wire x1="-132.08" y1="-25.4" x2="-124.46" y2="-25.4" width="0.1524" layer="91"/>
+</segment>
+<segment>
+<pinref part="U4" gate="G$1" pin="A5"/>
+<wire x1="271.78" y1="83.82" x2="274.32" y2="83.82" width="0.1524" layer="91"/>
+<label x="271.78" y="83.82" size="1.27" layer="95" font="vector" rot="R180" xref="yes"/>
+</segment>
+</net>
+<net name="HB1-EN" class="0">
+<segment>
+<label x="-96.52" y="-25.4" size="1.27" layer="95" xref="yes"/>
+<pinref part="U$1" gate="G$2" pin="PD11"/>
+<wire x1="-96.52" y1="-25.4" x2="-101.6" y2="-25.4" width="0.1524" layer="91"/>
+</segment>
+<segment>
+<pinref part="U4" gate="G$1" pin="A6"/>
+<wire x1="271.78" y1="81.28" x2="274.32" y2="81.28" width="0.1524" layer="91"/>
+<label x="271.78" y="81.28" size="1.27" layer="95" font="vector" rot="R180" xref="yes"/>
+</segment>
+</net>
+<net name="HB2-DIR" class="0">
+<segment>
+<pinref part="U$1" gate="G$2" pin="PD15"/>
+<wire x1="-96.52" y1="-30.48" x2="-101.6" y2="-30.48" width="0.1524" layer="91"/>
+<label x="-96.52" y="-30.48" size="1.27" layer="95" xref="yes"/>
+</segment>
+<segment>
+<pinref part="U4" gate="G$1" pin="A2"/>
+<wire x1="271.78" y1="91.44" x2="274.32" y2="91.44" width="0.1524" layer="91"/>
+<label x="271.78" y="91.44" size="1.27" layer="95" font="vector" rot="R180" xref="yes"/>
+</segment>
+</net>
+<net name="HB1-PWM" class="0">
+<segment>
+<pinref part="U4" gate="G$1" pin="A4"/>
+<wire x1="271.78" y1="86.36" x2="274.32" y2="86.36" width="0.1524" layer="91"/>
+<label x="271.78" y="86.36" size="1.27" layer="95" font="vector" rot="R180" xref="yes"/>
+</segment>
+<segment>
+<label x="-96.52" y="-27.94" size="1.27" layer="95" xref="yes"/>
+<pinref part="U$1" gate="G$2" pin="PD13"/>
+<wire x1="-96.52" y1="-27.94" x2="-101.6" y2="-27.94" width="0.1524" layer="91"/>
+</segment>
+</net>
+<net name="HB2-PWM" class="0">
+<segment>
+<pinref part="U4" gate="G$1" pin="A3"/>
+<wire x1="271.78" y1="88.9" x2="274.32" y2="88.9" width="0.1524" layer="91"/>
+<label x="271.78" y="88.9" size="1.27" layer="95" font="vector" rot="R180" xref="yes"/>
+</segment>
+<segment>
+<label x="-132.08" y="-27.94" size="1.27" layer="95" rot="R180" xref="yes"/>
+<pinref part="U$1" gate="G$2" pin="PD12"/>
+<wire x1="-132.08" y1="-27.94" x2="-124.46" y2="-27.94" width="0.1524" layer="91"/>
+</segment>
+</net>
+<net name="HB2-EN" class="0">
+<segment>
+<label x="-132.08" y="-30.48" size="1.27" layer="95" rot="R180" xref="yes"/>
+<pinref part="U$1" gate="G$2" pin="PD14"/>
+<wire x1="-132.08" y1="-30.48" x2="-124.46" y2="-30.48" width="0.1524" layer="91"/>
+</segment>
+<segment>
+<pinref part="U4" gate="G$1" pin="A1"/>
+<wire x1="271.78" y1="93.98" x2="274.32" y2="93.98" width="0.1524" layer="91"/>
+<label x="271.78" y="93.98" size="1.27" layer="95" font="vector" rot="R180" xref="yes"/>
+</segment>
+</net>
