File: STM32F407 era/Processor board/Version 3/processor board.sch (EAGLE design)
At the start: 45 parts, among them IC1 REG1117, U2 MAX13052ESA+, X1 MINI-USB-SCHIELD-32005-201, X2 057-010-1, Y1 25 MHz, Y2 32.768KHz

Commit message: added testpoints to power rails and coms, and created new Gerbers for PCB order
Changed lines of the file:
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@@
 <layer number="56" name="wert" color="7" fill="1" visible="no" active="no"/>
 <layer number="57" name="tCAD" color="7" fill="1" visible="no" active="no"/>
+<layer number="90" name="Modules" color="5" fill="1" visible="yes" active="yes"/>
 <layer number="91" name="Nets" color="2" fill="1" visible="yes" active="yes"/>
 <layer number="92" name="Busses" color="1" fill="1" visible="yes" active="yes"/>
@@
 <layer number="251" name="SMDround" color="7" fill="1" visible="yes" active="yes"/>
 <layer number="254" name="cooling" color="7" fill="1" visible="yes" active="yes"/>
+<layer number="255" name="routoute" color="7" fill="1" visible="yes" active="yes"/>
 </layers>
 <schematic xreflabel="%F%N/%S.%C%R" xrefpart="/%S.%C%R">
