File: STM32F407 era/SO-DIMM/Development board/Version 1/Development board.sch (EAGLE design)
At the start: 72 parts, among them IC1 74HC595N, IC2 74HC595N, J3 SO-DIMM-CPU, J4 FTDI_DEVICE, U1 IRF9332PBF, U10 SN65HVD232D, U11 MAX9926, U5 MAX9926, X1 057-014-1

Commit message: more work on debug board silkscreen
Parts:
- R26: value 60 -> 120
Changed lines of the file:
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@@
 <part name="GND25" library="supply1" deviceset="GND" device=""/>
 <part name="SW1" library="microbuilder" deviceset="SWITCH_DPDT" device=""/>
-<part name="R26" library="microbuilder" deviceset="RESISTOR" device="_0603" value="60"/>
+<part name="R26" library="microbuilder" deviceset="RESISTOR" device="_0603" value="120"/>
 <part name="GND16" library="supply1" deviceset="GND" device=""/>
 <part name="U1" library="International_Rectifier_By_element14_Batch_1" deviceset="IRF9332PBF" device=""/>

Commit message: All board V1-RC1 done
all boards ready for inspection
Parts:
- removed C34, C35, C5, C51: 1n, microbuilder:CAP_CERAMIC_0603
- removed C36, C52: 100n, microbuilder:CAP_CERAMIC_0603
- removed H4, H5: MOUNT-HOLE3.0, holes:MOUNT-HOLE3.0
- removed PTC2: (no value), microbuilder:PTC1812
- removed R27, R29, R39, R40, R41, R7, R74: 10k 0W5, microbuilder:RESISTOR_0805
- removed R28, R42, R43, R44, R75, R76: 1k, microbuilder:RESISTOR_0603
- removed U11: MAX9926, AAU-Racing:MAX9926
- added J1: (no value), SparkFun-Connectors:DB9FEMALE
- added J5: AVR_SPI_PRG_6NS, SparkFun-Connectors:AVR_SPI_PRG_6NS
- added LED6, LED7: (no value), microbuilder:LED1206
- added R1: (no value), rcl:R-TRIMM3296W
- added R12, R13, R14, R15, R2: 240, microbuilder:RESISTOR_0603
- added S1, S2, S3, S4: (no value), switch-omron:10-XX
- added S5, S6, S7, S8: (no value), adafruit:EG1218S
- added U$21: MICROFIT4, unicorn:MICROFIT4
- added U4: LoPy, AAU-Racing:LOPY
- added U6: (no value), connector:AUDIO-JACKPTH
- added X2: BN35N61, con-coax:BN35N61
- R3: value 10k 0W5 -> 240; device microbuilder:RESISTOR_0805 -> microbuilder:RESISTOR_0603
- U1: value IRF9332PBF -> ARDUINOR3-DIMENSION; device International_Rectifier_By_element14_Batch_1:IRF9332PBF -> microbuilder:ARDUINOR3-DIMENSION
- U5: value MAX9926 -> (none); device AAU-Racing:MAX9926 -> connector:AUDIO-JACKPTH
Connections:
- removed net BRAKEP2B: J3G$2.PA6
- removed net BRAKEPB: J3G$2.PA5
- removed net CANH: SW1.P2, U10.CANH, X1-7.S
- removed net CANL: SW1.P1, U10.CANL, X1-8.S
- removed net CLUTCH-POTB: J3G$5.PC0
- removed net COMRX: J3G$3.PC7
- removed net COMTX: J3G$3.PC6
- removed net GEARPOSANB: J3G$2.PA7
- removed net GSENSB: J3G$5.PA1
- removed net HB1-DIRA: J3G$5.PE2
- removed net HB1-DIRB: J3G$5.PE3
- removed net HB1-PWM: J3G$5.PE5
- removed net HB2-DIRA: J3G$5.PC13
- removed net HB2-DIRB: J3G$5.PE4
- removed net HB2-PWM: J3G$5.PE6
- removed net N$12: PTC2.2, U1.D, U1.D_2, U1.D_3, U1.D_4
- removed net N$15: C35.P$2, R41.2, U5.IN1-
- removed net N$25: C51.P$1, R29.2, U11.IN1+
- removed net N$26: C5.P$2, R7.2, U11.IN2-
- removed net N$31: R44.1, U5.DIRN
- removed net N$67: R76.1, U11.DIRN
- removed net RPM1: R42.1, U5.COUT1
- removed net RPM1GIN: R39.1
- removed net RPM1IN: R27.1
- removed net RPM2: R43.1, U5.COUT2
- removed net RPM2GIN: R41.1
- removed net RPM2IN: R40.1
- removed net RPM3: R28.1, U11.COUT1
- removed net RPM3GIN: R7.1
- removed net RPM3IN: R3.1
- removed net RPM4: R75.1, U11.COUT2
- removed net RPM4GIN: R74.1
- removed net RPM4IN: R29.1
- removed net SPEEDB: J3G$2.PA3
- removed net TRAVEL1B: J3G$5.PC1
- removed net TRAVEL2B: J3G$5.PC2
- removed net TRAVEL3B: J3G$5.PC3
- removed net TRAVEL4B: J3G$5.PA0
- removed net VCC: U1.S, U1.S_2, U1.S_3
- removed net VOUTUB: J3G$2.PA4
- removed net VTEMP2B: J3G$2.PC5
- removed net VTEMPB: J3G$2.PC4
- removed net YAWB: J3G$5.PA2
- new net 10: J3G$3.PD15, U1.D10
- new net 2: J3G$5.PC0/AN10, U1.D2
- new net 3: J3G$5.PE6, U1.D3
- new net 4: J3G$5.PC13, U1.D4
- new net 5: J3G$5.PE5, U1.D5
- new net 6: J3G$4.PB5, U1.D6
- new net 7: J3G$5.PE4, U1.D7
- new net 8: J3G$5.PE3, U1.D8
- new net 9: J3G$4.PB4, U1.D9
- new net A0: J3G$5.PC1/AN11, U1.A0
- new net A1: J3G$5.PC2/AN12, U1.A1
- new net A2: J3G$5.PC3/AN13, U1.A2
- new net A3: J3G$5.PA0/AN0, U1.A3
- new net A4: J3G$5.PA1/AN1, U1.A4/SDA
- new net A5: J3G$5.PA2/AN2, U1.A5/SCL
- new net CAN_N: J1.2, SW1.P1, U$21.PIN2, U10.CANL, U5.LEFT, U6.LEFT, X1-8.S
- new net CAN_P: J1.7, SW1.P2, U$21.PIN1, U10.CANH, U5.RIGHT, U6.RIGHT, X1-7.S
- new net CTS: J3G$4.PD3, XB1.!CTS!/DIO7
- new net DAC0: J3G$2.PA4/AN4, X2G$1.1
- new net LCD_LATCH: IC1A.RCK, IC2A.RCK, J3G$3.PB12
- new net POT1: J3G$2.PA7/AN7, RV1.S
- new net POT2: J3G$2.PA6/AN6, RV2.S
- new net POT3: J3G$2.PA5/AN5, RV3.S
- new net POT4: J3G$2.PA3/AN3, RV4.S
- new net RTS: J3G$4.PD4, XB1.!RTS!/AD6/DIO6
- new net RX: J3G$4.PB7, U1.D1
- new net SCL1: J3G$4.PB8, U1.SCL
- new net SDA1: J3G$4.PB9, U1.SDA
- new net SW1: J3G$2.PE10, S5.P
- new net SW2: J3G$2.PE9, S6.P
- new net SW3: J3G$2.PE8, S7.P
- new net SW4: J3G$2.PE7, S8.P
- new net SW5: J3G$2.PB1/AN9, R12.1, S1.S, S1.S1
- new net SW6: J3G$2.PB0/AN8, R13.1, S2.S, S2.S1
- new net SW7: J3G$2.PC5/AN15, R14.1, S3.S, S3.S1
- new net SW8: J3G$2.PC4/AN15, R15.1, S4.S, S4.S1
- new net TX: J3G$4.PB6, U1.D0
- net 12V: now also U1.VIN; no longer PTC2.1
- net 3.3V: now also R12.2, R13.2, R14.2, R15.2, S5.O, S6.O, S7.O, S8.O, U1.3V, U1.IOREF, U4.3,3V, XB1.!RESET; no longer R28.2, R42.2, R43.2, R44.2, R75.2, R76.2
- net 5.0V: now also IC1A.SCL, IC2A.SCL, J5.2, R1.E, U1.5V, U4.5V; no longer C36.P$1, C52.P$1, U11.VCC, U5.VCC
- net DBG_RX: now also J3G$3.PC7; no longer J3G$2.PB11
- net DBG_TX: now also J3G$3.PC6; no longer J3G$2.PB10
- net GND: now also IC1A.G, IC2A.G, J1.3, J1.6, J5.6, LED6.C, LED7.C, R1.A, S1.P, S1.P1, S2.P, S2.P1, S3.P, S3.P1, S4.P, S4.P1, S5.S, S6.S, S7.S, S8.S, U$21.PIN3, U$21.PIN4, U1.GND, U1.GND1, U1.GND2, U5.SLEEVE, U6.SLEEVE, X2G$1.GND, XB1.GND; no longer C36.P$2, C52.P$2, U1.G, U11.BIAS1, U11.BIAS2, U11.GND, U11.INT_THRS1, U11.INT_THRS2, U11.ZERO_EN, U5.BIAS1, U5.BIAS2, U5.GND, U5.INT_THRS1, U5.INT_THRS2, U5.ZERO_EN
- net MISO: now also J3G$3.PB14, J5.1, U1.D12
- net MOSI: now also IC1A.SER, J3G$3.PB15, J5.4, U1.D13
- net N$11: now also DIS1.CONTR, R1.S; no longer C34.P$1, R27.2, U5.IN2+
- net N$16: now also LED6.A, R3.1; no longer C5.P$1, R3.2, U11.IN2+
- net N$17: now also R3.2, XB1.ASSOC/AD5/DIO5; no longer C35.P$1, R40.2, U5.IN1+
- net N$18: now also R2.2, XB1.PWM0/RSSI; no longer C34.P$2, R39.2, U5.IN2-
- net N$19: now also LED7.A, R2.1; no longer C51.P$2, R74.2, U11.IN1-
- net SCK: now also IC1A.SCK, IC2A.SCK, J3G$3.PB13, J5.3, U1.D11
- net SCL: now also J3G$2.PB10
- net SDA: now also J3G$2.PB11
- net TELE_RX: now also U4.P0/RX, XB1.DOUT
- net TELE_TX: now also U4.P1/TX, XB1.DIN/!CONFIG
- net ~RESET: now also J3G$2.PE15
Other:
- note removed: "Input"
- note removed: "Interrupt"
- note removed: "Output"
- note removed: "Power protection"
- note removed: "Wheel Speed triggers"
- moved on the sheet: C7, C8, IC1, IC1P, IC2, IC2P, J3G$2, J3G$3, J3G$4, J3G$5, J4, R3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

Commit message: extra ERC check done
Changed lines of the file:
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@@
 <pinref part="S8" gate="1" pin="S"/>
 <wire x1="43.18" y1="-129.54" x2="48.26" y2="-129.54" width="0.1524" layer="91"/>
+<junction x="48.26" y="-129.54"/>
 </segment>
 <segment>
@@
 </segment>
 </net>
-<net name="N$3" class="0">
-<segment>
-<wire x1="289.56" y1="-330.2" x2="289.56" y2="-331.47" width="0.1524" layer="91"/>
-</segment>
-</net>
 <net name="N$10" class="0">
 <segment>
@@
 <wire x1="-55.88" y1="81.28" x2="-55.88" y2="91.44" width="0.1524" layer="91"/>
 <wire x1="-55.88" y1="91.44" x2="-45.72" y2="91.44" width="0.1524" layer="91"/>
-<wire x1="-43.18" y1="91.44" x2="-45.72" y2="91.44" width="0.1524" layer="91"/>
 <pinref part="U$30" gate="G$1" pin="/OUT2"/>
 <pinref part="LED1" gate="G$1" pin="BLUE"/>

Commit message: last end changes on boards
Dev board
- Added 8 LED for ekstra debugging feature
- fixed Tvalue silkscreen
-

COM/TC
- fixed connections om P-channel RPP
- 12V from debug changed to include RPP and fuse

Dash
- fixed connections om P-channel RPP
- 12V from debug changed to include RPP and fuse

debug
- Added "ohm/not ohm to silkscreen
- Added BNC connectors for CAN

and much much more
Parts:
- added C5: 47n, microbuilder:CAP_CERAMIC_0603
- added LED10, LED11, LED12, LED13, LED14, LED15, LED8, LED9: (no value), microbuilder:LED1206
- added R16, R17, R18, R19, R20, R21, R23, R24: 100, microbuilder:RESISTOR_0603
- added R7: 60, microbuilder:RESISTOR_0603
- R26: value 120 -> 60
Connections:
- new net LED1: J3G$3.PA9, R16.2
- new net LED2: J3G$3.PD14, R17.2
- new net LED3: J3G$3.PD13, R18.2
- new net LED4: J3G$3.PD12, R19.2
- new net LED5: J3G$3.PD11, R20.2
- new net LED6: J3G$3.PD10, R21.2
- new net LED7: J3G$3.PD9, R23.2
- new net LED8: J3G$3.PD8, R24.2
- new net N$12: LED8.A, R16.1
- new net N$15: LED9.A, R17.1
- new net N$25: LED10.A, R18.1
- new net N$26: LED11.A, R19.1
- new net N$3: R7.1, SW1.S1
- new net N$31: LED12.A, R20.1
- new net N$41: LED13.A, R21.1
- new net N$42: LED14.A, R23.1
- new net N$43: LED15.A, R24.1
- net GND: now also C5.P$2, LED10.C, LED11.C, LED12.C, LED13.C, LED14.C, LED15.C, LED8.C, LED9.C
- net N$8: now also C5.P$1, R7.2; no longer SW1.S1
Other:
- moved on the sheet: R26, SW1

Commit message: error corrections
Parts:
- added R25: 499, microbuilder:RESISTOR_0603
- added R27: 976, microbuilder:RESISTOR_0603
Connections:
- new net N$46: R25.1, U4.P1/TX
- net 3.3V: no longer U4.3,3V
- net GND: now also R27.2, U4.GND
- net MOSI: now also U1.D11; no longer U1.D13
- net SCK: now also U1.D13; no longer U1.D11
- net TELE_RX: now also R25.2, R27.1; no longer U4.P0/RX
- net TELE_TX: now also U4.P0/RX; no longer U4.P1/TX
Changed lines of the file:
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@@
 <part name="GND12" library="supply1" deviceset="GND" device=""/>
 <part name="U4" library="AAU-Racing" deviceset="LOPY" device="" value="LoPy"/>
-<part name="U$7" library="microbuilder" deviceset="3.3V" device=""/>
 <part name="U$19" library="microbuilder" deviceset="5.0V" device=""/>
 <part name="U5" library="connector" deviceset="AUDIO-JACK" device="PTH"/>
@@
 <part name="LED15" library="microbuilder" deviceset="LED" device="1206"/>
 <part name="GND30" library="supply1" deviceset="GND" device=""/>
+<part name="R25" library="microbuilder" deviceset="RESISTOR" device="_0603" value="499"/>
+<part name="R27" library="microbuilder" deviceset="RESISTOR" device="_0603" value="976"/>
+<part name="GND31" library="supply1" deviceset="GND" device=""/>
+<part name="GND32" library="supply1" deviceset="GND" device=""/>
 </parts>
 <sheets>
@@
 <instance part="GND12" gate="1" x="81.28" y="-401.32"/>
 <instance part="U4" gate="G$1" x="-109.22" y="-200.66"/>
-<instance part="U$7" gate="G$1" x="-106.68" y="-160.02"/>
 <instance part="U$19" gate="G$1" x="-111.76" y="-160.02"/>
 <instance part="U5" gate="G$1" x="220.98" y="-381"/>
@@
 <instance part="LED15" gate="G$1" x="-25.4" y="-342.9"/>
 <instance part="GND30" gate="1" x="-20.32" y="-347.98"/>
+<instance part="R25" gate="G$1" x="-134.62" y="-182.88" rot="R180"/>
+<instance part="R27" gate="G$1" x="-142.24" y="-190.5" rot="R270"/>
+<instance part="GND31" gate="1" x="-109.22" y="-226.06"/>
+<instance part="GND32" gate="1" x="-142.24" y="-198.12"/>
 </instances>
 <busses>
@@
 <junction x="-20.32" y="-297.18"/>
 </segment>
+<segment>
+<pinref part="U4" gate="G$1" pin="GND"/>
+<pinref part="GND31" gate="1" pin="GND"/>
+</segment>
+<segment>
+<pinref part="R27" gate="G$1" pin="2"/>
+<pinref part="GND32" gate="1" pin="GND"/>
+</segment>
 </net>
 <net name="3.3V" class="0">
@@
 </segment>
 <segment>
-<pinref part="U4" gate="G$1" pin="3,3V"/>
-<pinref part="U$7" gate="G$1" pin="3.3V"/>
-<wire x1="-106.68" y1="-165.1" x2="-106.68" y2="-162.56" width="0.1524" layer="91"/>
-</segment>
-<segment>
 <pinref part="U$35" gate="G$1" pin="3.3V"/>
 <pinref part="R12" gate="G$1" pin="2"/>
@@
 </segment>
 <segment>
-<pinref part="U4" gate="G$1" pin="P1/TX"/>
-<wire x1="-121.92" y1="-182.88" x2="-119.38" y2="-182.88" width="0.1524" layer="91"/>
-<label x="-121.92" y="-182.88" size="1.27" layer="95" rot="R180" xref="yes"/>
+<pinref part="U4" gate="G$1" pin="P0/RX"/>
+<wire x1="-121.92" y1="-180.34" x2="-119.38" y2="-180.34" width="0.1524" layer="91"/>
+<label x="-121.92" y="-180.34" size="1.27" layer="95" rot="R180" xref="yes"/>
 </segment>
 </net>
@@
 </segment>
 <segment>
-<pinref part="U4" gate="G$1" pin="P0/RX"/>
-<wire x1="-121.92" y1="-180.34" x2="-119.38" y2="-180.34" width="0.1524" layer="91"/>
-<label x="-121.92" y="-180.34" size="1.27" layer="95" rot="R180" xref="yes"/>
+<pinref part="R25" gate="G$1" pin="2"/>
+<wire x1="-144.78" y1="-182.88" x2="-142.24" y2="-182.88" width="0.1524" layer="91"/>
+<pinref part="R27" gate="G$1" pin="1"/>
+<wire x1="-142.24" y1="-182.88" x2="-139.7" y2="-182.88" width="0.1524" layer="91"/>
+<wire x1="-142.24" y1="-182.88" x2="-142.24" y2="-185.42" width="0.1524" layer="91"/>
+<junction x="-142.24" y="-182.88"/>
+<label x="-144.78" y="-182.88" size="1.27" layer="95" rot="R180" xref="yes"/>
 </segment>
 </net>
@@
 </segment>
 <segment>
+<pinref part="J5" gate="G$1" pin="4"/>
+<wire x1="350.52" y1="-99.06" x2="347.98" y2="-99.06" width="0.1524" layer="91"/>
+<label x="350.52" y="-99.06" size="1.27" layer="95" xref="yes"/>
+</segment>
+<segment>
+<pinref part="U1" gate="G$1" pin="D11"/>
+<wire x1="304.8" y1="-66.04" x2="307.34" y2="-66.04" width="0.1524" layer="91"/>
+<label x="304.8" y="-66.04" size="1.27" layer="95" rot="R180" xref="yes"/>
+</segment>
+</net>
+<net name="SCK" class="0">
+<segment>
+<pinref part="X1" gate="-13" pin="S"/>
+<wire x1="393.7" y1="-251.46" x2="396.24" y2="-251.46" width="0.1524" layer="91"/>
+<label x="393.7" y="-251.46" size="1.27" layer="95" rot="R180" xref="yes"/>
+</segment>
+<segment>
+<pinref part="IC1" gate="A" pin="SCK"/>
+<wire x1="25.4" y1="-353.06" x2="30.48" y2="-353.06" width="0.1524" layer="91"/>
+<label x="25.4" y="-353.06" size="1.27" layer="95" rot="R180" xref="yes"/>
+</segment>
+<segment>
+<pinref part="IC2" gate="A" pin="SCK"/>
+<wire x1="25.4" y1="-388.62" x2="30.48" y2="-388.62" width="0.1524" layer="91"/>
+<label x="25.4" y="-388.62" size="1.27" layer="95" rot="R180" xref="yes"/>
+</segment>
+<segment>
+<pinref part="J3" gate="G$3" pin="PB13"/>
+<wire x1="256.54" y1="-165.1" x2="254" y2="-165.1" width="0.1524" layer="91"/>
+<label x="256.54" y="-165.1" size="1.27" layer="95" xref="yes"/>
+</segment>
+<segment>
+<pinref part="J5" gate="G$1" pin="3"/>
+<wire x1="327.66" y1="-99.06" x2="330.2" y2="-99.06" width="0.1524" layer="91"/>
+<label x="327.66" y="-99.06" size="1.27" layer="95" rot="R180" xref="yes"/>
+</segment>
+<segment>
 <pinref part="U1" gate="G$1" pin="D13"/>
 <wire x1="304.8" y1="-71.12" x2="307.34" y2="-71.12" width="0.1524" layer="91"/>
 <label x="304.8" y="-71.12" size="1.27" layer="95" rot="R180" xref="yes"/>
-</segment>
-<segment>
-<pinref part="J5" gate="G$1" pin="4"/>
-<wire x1="350.52" y1="-99.06" x2="347.98" y2="-99.06" width="0.1524" layer="91"/>
-<label x="350.52" y="-99.06" size="1.27" layer="95" xref="yes"/>
-</segment>
-</net>
-<net name="SCK" class="0">
-<segment>
-<pinref part="X1" gate="-13" pin="S"/>
-<wire x1="393.7" y1="-251.46" x2="396.24" y2="-251.46" width="0.1524" layer="91"/>
-<label x="393.7" y="-251.46" size="1.27" layer="95" rot="R180" xref="yes"/>
-</segment>
-<segment>
-<pinref part="IC1" gate="A" pin="SCK"/>
-<wire x1="25.4" y1="-353.06" x2="30.48" y2="-353.06" width="0.1524" layer="91"/>
-<label x="25.4" y="-353.06" size="1.27" layer="95" rot="R180" xref="yes"/>
-</segment>
-<segment>
-<pinref part="IC2" gate="A" pin="SCK"/>
-<wire x1="25.4" y1="-388.62" x2="30.48" y2="-388.62" width="0.1524" layer="91"/>
-<label x="25.4" y="-388.62" size="1.27" layer="95" rot="R180" xref="yes"/>
-</segment>
-<segment>
-<pinref part="J3" gate="G$3" pin="PB13"/>
-<wire x1="256.54" y1="-165.1" x2="254" y2="-165.1" width="0.1524" layer="91"/>
-<label x="256.54" y="-165.1" size="1.27" layer="95" xref="yes"/>
-</segment>
-<segment>
-<pinref part="U1" gate="G$1" pin="D11"/>
-<wire x1="304.8" y1="-66.04" x2="307.34" y2="-66.04" width="0.1524" layer="91"/>
-<label x="304.8" y="-66.04" size="1.27" layer="95" rot="R180" xref="yes"/>
-</segment>
-<segment>
-<pinref part="J5" gate="G$1" pin="3"/>
-<wire x1="327.66" y1="-99.06" x2="330.2" y2="-99.06" width="0.1524" layer="91"/>
-<label x="327.66" y="-99.06" size="1.27" layer="95" rot="R180" xref="yes"/>
 </segment>
 </net>
@@
 </segment>
 </net>
+<net name="N$46" class="0">
+<segment>
+<pinref part="R25" gate="G$1" pin="1"/>
+<pinref part="U4" gate="G$1" pin="P1/TX"/>
+<wire x1="-129.54" y1="-182.88" x2="-119.38" y2="-182.88" width="0.1524" layer="91"/>
+</segment>
+</net>

Commit message: BOM done
Parts:
- C1, C2, C3, C6: value (none) -> 22u
- U2: value (none) -> 3,3v
- U3: value (none) -> 5,0v
Changed lines of the file:
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@@
 <part name="LED5" library="microbuilder" deviceset="LED_RGB_PLCC4" device=""/>
 <part name="CN2" library="microbuilder" deviceset="DCBARREL" device="PTH"/>
-<part name="U2" library="microbuilder" deviceset="LM1117" device="SOT223-REFLOW"/>
-<part name="U3" library="microbuilder" deviceset="LM1117" device="SOT223-REFLOW"/>
-<part name="C1" library="microbuilder" deviceset="CAP_CERAMIC" device="_0805"/>
-<part name="C2" library="microbuilder" deviceset="CAP_CERAMIC" device="_0805"/>
-<part name="C3" library="microbuilder" deviceset="CAP_CERAMIC" device="_0805"/>
-<part name="C6" library="microbuilder" deviceset="CAP_CERAMIC" device="_0805"/>
+<part name="U2" library="microbuilder" deviceset="LM1117" device="SOT223-REFLOW" value="3,3v"/>
+<part name="U3" library="microbuilder" deviceset="LM1117" device="SOT223-REFLOW" value="5,0v"/>
+<part name="C1" library="microbuilder" deviceset="CAP_CERAMIC" device="_0805" value="22u"/>
+<part name="C2" library="microbuilder" deviceset="CAP_CERAMIC" device="_0805" value="22u"/>
+<part name="C3" library="microbuilder" deviceset="CAP_CERAMIC" device="_0805" value="22u"/>
+<part name="C6" library="microbuilder" deviceset="CAP_CERAMIC" device="_0805" value="22u"/>
 <part name="U$5" library="microbuilder" deviceset="3.3V" device=""/>
 <part name="U$9" library="microbuilder" deviceset="12V" device=""/>
