File: STM32F407 era/SO-DIMM/Telemetry receiver/Version 1/Telemetry receiver.brd (EAGLE design)
At the start: 78.9 x 37.6 mm, 26 parts, among them Q2 12MHz, U7 LoPy

Commit message: last end changes on boards
Dev board
- Added 8 LED for ekstra debugging feature
- fixed Tvalue silkscreen
-

COM/TC
- fixed connections om P-channel RPP
- 12V from debug changed to include RPP and fuse

Dash
- fixed connections om P-channel RPP
- 12V from debug changed to include RPP and fuse

debug
- Added "ohm/not ohm to silkscreen
- Added BNC connectors for CAN

and much much more
Connections:
- net RX: now also U$24.12; no longer U$24.10
- net TX: now also U$24.10; no longer U$24.12
Routing:
- net TX: track 80.2 -> 70.1 mm, vias 2 -> 0
- net RX: track 70.4 -> 80.0 mm
Changed lines of the file:
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@@
 </signal>
 <signal name="RX">
-<contactref element="U$24" pad="10"/>
 <contactref element="XB1" pad="2"/>
 <contactref element="U7" pad="41"/>
@@
 <wire x1="10.63625" y1="9.335" x2="10.63625" y2="18.7325" width="0.3048" layer="1"/>
 <wire x1="40.79875" y1="19.685" x2="40.79875" y2="31.4325" width="0.3048" layer="1"/>
-<wire x1="54.9783" y1="13.81125" x2="46.355" y2="13.81125" width="0.3048" layer="1"/>
-<wire x1="46.355" y1="13.81125" x2="41.5925" y2="18.57375" width="0.3048" layer="1"/>
-<via x="41.5925" y="18.57375" extent="1-16" drill="0.3302"/>
-<wire x1="41.5925" y1="18.57375" x2="40.64" y2="19.52625" width="0.3048" layer="16"/>
 <via x="40.64" y="19.52625" extent="1-16" drill="0.3302"/>
+<contactref element="U$24" pad="12"/>
+<wire x1="65.0367" y1="15.08125" x2="63.34125" y2="15.08125" width="0.3048" layer="1"/>
+<via x="63.34125" y="15.08125" extent="1-16" drill="0.3302"/>
+<wire x1="63.34125" y1="15.08125" x2="46.0375" y2="15.08125" width="0.3048" layer="16"/>
+<wire x1="46.0375" y1="15.08125" x2="41.5925" y2="19.52625" width="0.3048" layer="16"/>
+<wire x1="41.5925" y1="19.52625" x2="40.64" y2="19.52625" width="0.3048" layer="16"/>
 </signal>
 <signal name="TX">
-<contactref element="U$24" pad="12"/>
 <contactref element="XB1" pad="3"/>
 <contactref element="U7" pad="40"/>
 <wire x1="11.1925" y1="7.89125" x2="11.1925" y2="18.495" width="0.3048" layer="1"/>
 <wire x1="11.1925" y1="18.495" x2="11.58875" y2="18.89125" width="0.3048" layer="1"/>
-<wire x1="11.58875" y1="18.89125" x2="40.9575" y2="18.89125" width="0.3048" layer="1"/>
-<wire x1="41.275" y1="19.20875" x2="40.9575" y2="18.89125" width="0.3048" layer="1"/>
-<wire x1="41.275" y1="19.20875" x2="41.275" y2="29.36875" width="0.3048" layer="1"/>
 <wire x1="41.275" y1="29.36875" x2="43.33875" y2="31.4325" width="0.3048" layer="1"/>
-<wire x1="65.0367" y1="15.08125" x2="63.5" y2="15.08125" width="0.3048" layer="1"/>
-<via x="63.5" y="15.08125" extent="1-16" drill="0.3302"/>
-<wire x1="63.5" y1="15.08125" x2="61.595" y2="15.08125" width="0.3048" layer="16"/>
-<via x="61.595" y="15.08125" extent="1-16" drill="0.3302"/>
-<wire x1="61.595" y1="15.08125" x2="60.96" y2="14.44625" width="0.3048" layer="1"/>
-<wire x1="46.51375" y1="14.44625" x2="42.38625" y2="18.57375" width="0.3048" layer="1"/>
-<wire x1="42.38625" y1="18.57375" x2="42.38625" y2="18.7325" width="0.3048" layer="1"/>
-<wire x1="42.38625" y1="18.7325" x2="41.91" y2="19.20875" width="0.3048" layer="1"/>
-<wire x1="41.91" y1="19.20875" x2="41.275" y2="19.20875" width="0.3048" layer="1"/>
-<wire x1="60.96" y1="14.44625" x2="46.51375" y2="14.44625" width="0.3048" layer="1"/>
+<contactref element="U$24" pad="10"/>
+<wire x1="41.275" y1="18.89125" x2="11.58875" y2="18.89125" width="0.3048" layer="1"/>
+<wire x1="41.275" y1="18.89125" x2="41.275" y2="29.36875" width="0.3048" layer="1"/>
+<wire x1="54.9783" y1="13.81125" x2="46.355" y2="13.81125" width="0.3048" layer="1"/>
+<wire x1="46.355" y1="13.81125" x2="41.275" y2="18.89125" width="0.3048" layer="1"/>
 </signal>
 <signal name="N$26">

Commit message: error corrections
Parts:
- added R2: 499, microbuilder:_0603
- added R3: 976, microbuilder:_0603
Connections:
- new net N$7: R2.1, U7.41
- net 3.3V: no longer U7.3,3V
- net GND: now also R3.1
- net RX: now also R2.2, R3.2; no longer U7.41
Routing:
- net RX: track 80.0 -> 68.2 mm
- net 3.3V: track 102.5 -> 95.4 mm
Changed lines of the file:
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@@
 <attribute name="VALUE" x="7.55645" y="5.3975" size="0.4064" layer="27" ratio="10" rot="R270"/>
 </element>
+<element name="R2" library="microbuilder" package="_0603" value="499" x="0.47625" y="-2.38125"/>
+<element name="R3" library="microbuilder" package="_0603" value="976" x="0.47625" y="-6.50875"/>
 </elements>
 <signals>
@@
 <contactref element="R1" pad="2"/>
 <contactref element="R8" pad="1"/>
+<contactref element="R3" pad="1"/>
+<wire x1="64.8675" y1="32.7025" x2="61.24575" y2="34.29" width="0" layer="19" extent="1-1"/>
+<wire x1="64.8675" y1="31.115" x2="64.8675" y2="32.7025" width="0" layer="19" extent="1-1"/>
+<wire x1="65.0367" y1="25.24125" x2="64.8675" y2="31.115" width="0" layer="19" extent="1-1"/>
+<wire x1="70.70725" y1="20.49125" x2="65.0367" y2="25.24125" width="0" layer="19" extent="1-1"/>
+<wire x1="55.08625" y1="28.3845" x2="61.24575" y2="34.29" width="0" layer="19" extent="1-1"/>
+<wire x1="47.78375" y1="24.3205" x2="55.08625" y2="28.3845" width="0" layer="19" extent="1-1"/>
+<wire x1="47.78375" y1="22.352" x2="47.78375" y2="24.3205" width="0" layer="19" extent="1-1"/>
+<wire x1="43.33875" y1="11.1125" x2="47.78375" y2="22.352" width="0" layer="19" extent="1-1"/>
+<wire x1="55.08625" y1="9.906" x2="43.33875" y2="11.1125" width="0" layer="19" extent="1-1"/>
+<wire x1="56.35625" y1="5.87375" x2="55.08625" y2="9.906" width="0" layer="19" extent="1-1"/>
+<wire x1="57.54875" y1="5.84" x2="56.35625" y2="5.87375" width="0" layer="19" extent="1-1"/>
+<wire x1="57.62625" y1="4.60375" x2="57.54875" y2="5.84" width="0" layer="19" extent="1-1"/>
+<wire x1="64.61125" y1="9.906" x2="57.54875" y2="5.84" width="0" layer="19" extent="1-1"/>
+<wire x1="25.1925" y1="7.89125" x2="43.33875" y2="11.1125" width="0" layer="19" extent="1-1"/>
+<wire x1="9.04875" y1="3.3655" x2="25.1925" y2="7.89125" width="0" layer="19" extent="1-1"/>
+<wire x1="-0.28575" y1="-6.50875" x2="9.04875" y2="3.3655" width="0" layer="19" extent="1-1"/>
+<wire x1="9.04875" y1="32.73425" x2="9.04875" y2="3.3655" width="0" layer="19" extent="1-1"/>
 </signal>
 <signal name="3.3V">
@@
 <contactref element="U2" pad="2"/>
 <contactref element="C2" pad="1"/>
-<contactref element="U7" pad="3,3V"/>
 <contactref element="XB1" pad="1"/>
 <contactref element="XB1" pad="5"/>
@@
 <wire x1="62.5475" y1="22.5425" x2="61.9125" y2="21.9075" width="0.3048" layer="1"/>
 <wire x1="55.08625" y1="7.874" x2="44.03725" y2="7.874" width="0.6096" layer="1"/>
-<wire x1="40.79875" y1="11.1125" x2="44.03725" y2="7.874" width="0.6096" layer="1"/>
 <wire x1="7.1925" y1="7.89125" x2="8.8925" y2="6.19125" width="0.6096" layer="1"/>
 <wire x1="13.4925" y1="6.19125" x2="15.1925" y2="7.89125" width="0.6096" layer="1"/>
 <wire x1="8.8925" y1="6.19125" x2="13.4925" y2="6.19125" width="0.6096" layer="1"/>
 <wire x1="15.1925" y1="7.89125" x2="16.6675" y2="9.36625" width="0.6096" layer="1"/>
-<wire x1="39.0525" y1="9.36625" x2="40.79875" y2="11.1125" width="0.6096" layer="1"/>
 <wire x1="16.6675" y1="9.36625" x2="39.0525" y2="9.36625" width="0.6096" layer="1"/>
 <wire x1="55.08625" y1="26.8605" x2="55.08625" y2="25.3492" width="0.6096" layer="1"/>
 <wire x1="55.08625" y1="25.3492" x2="54.9783" y2="25.24125" width="0.6096" layer="1"/>
+<wire x1="39.0525" y1="9.36625" x2="44.03725" y2="7.874" width="0" layer="19" extent="1-1"/>
 </signal>
 <signal name="RX">
 <contactref element="XB1" pad="2"/>
-<contactref element="U7" pad="41"/>
 <wire x1="9.1925" y1="7.89125" x2="10.63625" y2="9.335" width="0.3048" layer="1"/>
 <wire x1="10.63625" y1="18.7325" x2="11.27125" y2="19.3675" width="0.3048" layer="1"/>
@@
 <wire x1="40.64" y1="19.52625" x2="40.79875" y2="19.685" width="0.3048" layer="1"/>
 <wire x1="10.63625" y1="9.335" x2="10.63625" y2="18.7325" width="0.3048" layer="1"/>
-<wire x1="40.79875" y1="19.685" x2="40.79875" y2="31.4325" width="0.3048" layer="1"/>
 <via x="40.64" y="19.52625" extent="1-16" drill="0.3302"/>
 <contactref element="U$24" pad="12"/>
@@
 <wire x1="46.0375" y1="15.08125" x2="41.5925" y2="19.52625" width="0.3048" layer="16"/>
 <wire x1="41.5925" y1="19.52625" x2="40.64" y2="19.52625" width="0.3048" layer="16"/>
+<contactref element="R2" pad="2"/>
+<contactref element="R3" pad="2"/>
+<wire x1="1.23825" y1="-2.38125" x2="9.1925" y2="7.89125" width="0" layer="19" extent="1-1"/>
+<wire x1="1.23825" y1="-6.50875" x2="1.23825" y2="-2.38125" width="0" layer="19" extent="1-1"/>
 </signal>
 <signal name="TX">
@@
 <wire x1="24.92375" y1="20.955" x2="23.1925" y2="22.68625" width="0.3048" layer="16"/>
 </signal>
+<signal name="N$7">
+<contactref element="R2" pad="1"/>
+<contactref element="U7" pad="41"/>
+<wire x1="-0.28575" y1="-2.38125" x2="40.79875" y2="31.4325" width="0" layer="19" extent="1-1"/>
+</signal>
 </signals>

Commit message: final changes
Parts:
- removed R2: 499, microbuilder:_0603
- removed R3: 976, microbuilder:_0603
Connections:
- removed net N$7: R2.1, U7.41
- net GND: no longer R3.1
- net RX: now also U7.41; no longer R2.2, R3.2
Routing:
- net RX: track 68.2 -> 80.0 mm
- net 3.3V: track 95.4 -> 102.5 mm
- net N$43: track 19.2 -> 18.1 mm
- net N$36: track 17.3 -> 16.4 mm
Other:
- board text removed: "<Assoc"
- board text removed: "<RSSI"
- board text removed: "RX"
- board text removed: "TX"

Commit message: BOM done
Parts:
- U2: value (none) -> 3,3v
Changed lines of the file:
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@@
 <attribute name="NAME" x="59.15025" y="26.2255" size="1.27" layer="25" font="vector" ratio="10"/>
 </element>
-<element name="U2" library="microbuilder" package="SOT223-R" value="" x="59.84875" y="8.89" smashed="yes">
+<element name="U2" library="microbuilder" package="SOT223-R" value="3,3v" x="59.84875" y="8.89" smashed="yes">
 <attribute name="NAME" x="58.3565" y="12.2555" size="1.27" layer="25" font="vector" ratio="10" rot="R180"/>
 <attribute name="VALUE" x="57.05475" y="8.255" size="0.4064" layer="27" ratio="10"/>
