File: STM32F407 era/SO-DIMM/CPU Board/Version 2/CPU Board.brd (EAGLE design)
At the start: 67.6 x 35 mm, 30 parts, among them U2 TPS3825-33DBVR, Y1 24 MHz, Y2 32.768KHz

Commit message: added vias for better ground stitching
Routing:
- net GND: vias 20 -> 63
Changed lines of the file:
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@@
 <via x="17.62125" y="14.9225" extent="1-16" drill="0.3"/>
 <via x="23.65375" y="14.44625" extent="1-16" drill="0.3"/>
+<via x="13.0175" y="23.65375" extent="1-16" drill="0.3"/>
+<via x="12.22375" y="23.65375" extent="1-16" drill="0.3"/>
+<via x="11.43" y="23.65375" extent="1-16" drill="0.3"/>
+<via x="11.43" y="24.4475" extent="1-16" drill="0.3"/>
+<via x="12.22375" y="24.4475" extent="1-16" drill="0.3"/>
+<via x="13.0175" y="24.4475" extent="1-16" drill="0.3"/>
+<via x="13.0175" y="22.86" extent="1-16" drill="0.3"/>
+<via x="12.22375" y="22.86" extent="1-16" drill="0.3"/>
+<via x="11.43" y="22.86" extent="1-16" drill="0.3"/>
+<via x="29.5275" y="33.9725" extent="1-16" drill="0.3"/>
+<via x="30.32125" y="33.9725" extent="1-16" drill="0.3"/>
+<via x="31.115" y="33.9725" extent="1-16" drill="0.3"/>
+<via x="31.90875" y="33.9725" extent="1-16" drill="0.3"/>
+<via x="32.7025" y="33.9725" extent="1-16" drill="0.3"/>
+<via x="33.49625" y="33.9725" extent="1-16" drill="0.3"/>
+<via x="34.29" y="33.9725" extent="1-16" drill="0.3"/>
+<via x="59.055" y="21.2725" extent="1-16" drill="0.3"/>
+<via x="59.69" y="21.9075" extent="1-16" drill="0.3"/>
+<via x="60.325" y="22.5425" extent="1-16" drill="0.3"/>
+<via x="60.96" y="23.1775" extent="1-16" drill="0.3"/>
+<via x="61.595" y="23.8125" extent="1-16" drill="0.3"/>
+<via x="53.34" y="11.58875" extent="1-16" drill="0.3"/>
+<via x="53.975" y="10.95375" extent="1-16" drill="0.3"/>
+<via x="54.61" y="10.31875" extent="1-16" drill="0.3"/>
+<via x="55.245" y="9.68375" extent="1-16" drill="0.3"/>
+<via x="55.245" y="8.89" extent="1-16" drill="0.3"/>
+<via x="55.245" y="8.09625" extent="1-16" drill="0.3"/>
+<via x="55.245" y="7.3025" extent="1-16" drill="0.3"/>
+<via x="55.245" y="6.50875" extent="1-16" drill="0.3"/>
+<via x="22.86" y="14.44625" extent="1-16" drill="0.3"/>
+<via x="22.06625" y="14.44625" extent="1-16" drill="0.3"/>
+<via x="23.65375" y="13.6525" extent="1-16" drill="0.3"/>
+<via x="23.65375" y="12.85875" extent="1-16" drill="0.3"/>
+<via x="24.4475" y="14.44625" extent="1-16" drill="0.3"/>
+<via x="25.24125" y="14.44625" extent="1-16" drill="0.3"/>
+<via x="22.06625" y="12.85875" extent="1-16" drill="0.3"/>
+<via x="22.06625" y="13.6525" extent="1-16" drill="0.3"/>
+<via x="22.86" y="13.6525" extent="1-16" drill="0.3"/>
+<via x="22.86" y="12.85875" extent="1-16" drill="0.3"/>
+<via x="24.4475" y="12.85875" extent="1-16" drill="0.3"/>
+<via x="24.4475" y="13.6525" extent="1-16" drill="0.3"/>
+<via x="25.24125" y="13.6525" extent="1-16" drill="0.3"/>
+<via x="25.24125" y="12.85875" extent="1-16" drill="0.3"/>
 </signal>
 <signal name="3.3V">

Commit message: created Gerbers
Parts:
- moved R2 0.16 mm to (42.5, 22.2)
- moved U2 0.16 mm to (42.5, 19.8)
Routing:
- net 3.3V: track 114.9 -> 115.8 mm
